File: K9HZ_LFP_Module/K9HZ_LPF_V1.00_KiCad/K9HZ_100W_11band_LPF-Filter/K9HZ_100W_11band_LPF-Filter.kicad_sch (KiCad schematic)
At the start: 169 parts, among them J17 RF interconnect, J22 RF interconnect, J26 LPF CTRL LOW, J27 LPF CTRL HI, K10 HF41F/12-ZS, K11 HF41F/12-ZS, K12 HF41F/12-ZS, K13 HF41F/12-ZS, K14 HF41F/12-ZS, K15 HF41F/12-ZS, K16 HF41F/12-ZS, K17 HF41F/12-ZS, K18 HF41F/12-ZS, K19 HF41F/12-ZS, K20 HF41F/12-ZS, K21 HF41F/12-ZS, K22 HF41F/12-ZS, K23 HF41F/12-ZS, K24 HF41F/12-ZS, K25 HF41F/12-ZS, K26 HF41F/12-ZS, K27 HF41F/12-ZS, K28 HF41F/12-ZS, K29 HF41F/12-ZS, K32 HF41F/12-ZS, K33 HF41F/12-ZS, K8 HF41F/12-ZS, K9 HF41F/12-ZS

Commit message: Corrected typo on band code for no-filter option
Other:
- note added: "NO FILT [1111]"
- note removed: "NO FILT [1011]"
Changed lines of the file:
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@@
   (title_block
     (title "K9HZ 100W 11 Band LPF: Filter board")
-    (date "2024-01-14")
+    (date "2024-01-17")
     (rev "V1.00")
     (comment 1 "Layout by OG King-KI3P")
@@
     (effects (font (size 1.27 1.27) bold) (justify left bottom))
   )
-  (text "NO FILT [1011]" (at 396.24 200.66 0)
+  (text "NO FILT [1111]" (at 396.24 200.66 0)
     (effects (font (size 1.27 1.27) bold) (justify left bottom))
   )
