File: K9HZ_LFP_Module/K9HZ_LPF_V1.00_KiCad/K9HZ_100W_11band_LPF-Filter/K9HZ_100W_11band_LPF-Filter.kicad_pcb (KiCad board)
At the start: 4 copper layers, 100 x 100 mm, 169 parts, among them J17 RF interconnect, J22 RF interconnect, J26 LPF CTRL LOW, J27 LPF CTRL HI, K10 HF41F/12-ZS, K11 HF41F/12-ZS, K12 HF41F/12-ZS, K13 HF41F/12-ZS, K14 HF41F/12-ZS, K15 HF41F/12-ZS, K16 HF41F/12-ZS, K17 HF41F/12-ZS, K18 HF41F/12-ZS, K19 HF41F/12-ZS, K20 HF41F/12-ZS, K21 HF41F/12-ZS, K22 HF41F/12-ZS, K23 HF41F/12-ZS, K24 HF41F/12-ZS, K25 HF41F/12-ZS, K26 HF41F/12-ZS, K27 HF41F/12-ZS, K28 HF41F/12-ZS, K29 HF41F/12-ZS, K32 HF41F/12-ZS, K33 HF41F/12-ZS, K8 HF41F/12-ZS, K9 HF41F/12-ZS

Commit message: Fixed silkscreen label placements on LPF filter board
Parts:
- moved C115 0.08 mm to (248.3, 77.5)
Other:
- board text added: "K9HZ 100W 11 Band LPF Filter board Designed by K9HZ Layout by KI3P 2024-02-03"
- board text removed: "K9HZ 100W 11 Band LPF Filter board Designed by K9HZ Layout by KI3P 2024-01-14"
