File: K9HZ_LFP_Module/K9HZ_LPF_V1.00_KiCad/K9HZ_100W_11band_LPF-TR-carrier/K9HZ_100W_11band_LPF-TR-carrier.kicad_pcb (KiCad board)
At the start: 4 copper layers, 40.6 x 25.4 mm, 12 parts, among them J22.1 ANTENNA, J22.2 TRANSMIT, J23.1 RECEIVE, J23.2 TR CTL, K1 HF41F/12-ZS, K2 HF41F/12-ZS, Q1 BS170

Commit message: Fixed stackup ambiguity in LPF relay carrier board. It is a 2 layer board but KiCad stackup contained two unused inner copper layers
Other:
- copper layers 4 -> 2
Changed lines of the file:
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@@
   (layers
     (0 "F.Cu" signal)
-    (1 "In1.Cu" signal)
-    (2 "In2.Cu" signal)
     (31 "B.Cu" signal)
     (32 "B.Adhes" user "B.Adhesive")
@@
       (layer "F.Mask" (type "Top Solder Mask") (thickness 0.01))
       (layer "F.Cu" (type "copper") (thickness 0.035))
-      (layer "dielectric 1" (type "prepreg") (thickness 0.2104) (material "FR4") (epsilon_r 4.5) (loss_tangent 0.02))
-      (layer "In1.Cu" (type "copper") (thickness 0.035))
-      (layer "dielectric 2" (type "core") (thickness 1.065) (material "FR4") (epsilon_r 4.5) (loss_tangent 0.02))
-      (layer "In2.Cu" (type "copper") (thickness 0.035))
-      (layer "dielectric 3" (type "prepreg") (thickness 0.2104) (material "FR4") (epsilon_r 4.5) (loss_tangent 0.02))
+      (layer "dielectric 1" (type "core") (thickness 1.5558) (material "FR4") (epsilon_r 4.5) (loss_tangent 0.02))
       (layer "B.Cu" (type "copper") (thickness 0.035))
       (layer "B.Mask" (type "Bottom Solder Mask") (thickness 0.01))
