File: T41_V012_Files_01-15-24/T41_V012_KiCad/T41-RF-board-V012/T41-RF-board-V012.kicad_sch (KiCad schematic)
At the start: 224 parts, among them J1 IQ_Out, J2 RF_IN, J3 RFControl, J4 12-13.8V, J5 IQ_In, J6 RF_OUT, Q1 BS170, U1 74CBTLV3253DR, U10 SN74LVC1G04DCK, U106 MC33078, U107 MC33078, U11 Si5351A-B-GT, U12 PE4312, U13 MAR-3SM+, U14 LM7805CT, U15 LM1117T-3.3, U16 MC33078, U17 LM317L, U18 SN74LVC1G04DCK, U19 MASWSS0179, U2 PSA-8A+, U20 MASWSS0179, U21 MCP23017_SO, U22 HMC434E, U23 HMC434E, U3 PE4312, U4 74CBTLV3253DR, U5 SN74LVC1G04DCK, U6 MC33078, U7 MASWSS0179, U8 MC33078, U9 MASWSS0179, Y1 ECS-TX053-S3, Y2 25MHz

Commit message: Recreate these
Parts:
- added JP1: SolderJumper_2_Open, Jumper:SolderJumper-2_P1.3mm_Open_TrianglePad1.0x1.5mm, symbol Jumper:SolderJumper_2_Open
- added JP2: SolderJumper_2_Bridged, Jumper:SolderJumper-2_P1.3mm_Bridged_RoundedPad1.0x1.5mm, symbol Jumper:SolderJumper_2_Bridged
Connections:
- net +3V3: now also JP2.2 (B); no longer C6.2, L1.1, R15.1
- net +5V: now also JP1.2 (B)
- net at L1.2, U1.16 (VCC): now also C6.2
- new net: JP1.1 (A), JP2.1 (A), L1.1, R15.1
Other:
- note added: "MiniCircuits ADT1-1+"
- note added: "MiniCircuits ADT2-1T+"
- note added: "Select 5V if needed for large signal operation."
- note removed: "T37-43 (yellow) Toroid 10T Bifial #28 or MiniCircuits ADT1-1+"
- note removed: "T37-43 (yellow) Toroid Primary: 12T Bifilar #28 Secondary: 24T #28 or MiniCircuits ADT2-1T+"
- moved on the sheet: C6

Commit message: Added ground test points and pad, silkscreen edits
Parts:
- added G1, G2, G3: TestPoint, Connector_PinHeader_2.54mm:PinHeader_1x01_P2.54mm_Vertical, symbol Connector:TestPoint
- added H1: ~, MountingHole:MountingHole_3.2mm_M3_Pad, symbol Mechanical:MountingHole_Pad
Connections:
- net GND: now also G1.1, G2.1, G3.1, H1.1
Changed lines of the file:
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@@
   (title_block
     (title "T41 RF Board")
-    (date "2024-01-26")
+    (date "2024-02-17")
     (rev "V012.6")
     (comment 1 "        Transcribed to KiCAD by OG King-KI3P")
     (comment 2 "By Al Peter-AC8GY, Revised by WJ Schmidt-K9HZ")
     (comment 3 "Change log: switched the order of attenuator and amp in receive chain")
+    (comment 4 "  - Added ground test points & pad, silkscreen edits")
   )
   (junction (at 266.7 256.54) (diameter 0) (color 0 0 0 0)
@@
   (junction (at 322.58 77.47) (diameter 0) (color 0 0 0 0)
   )
+  (junction (at 142.24 60.96) (diameter 0) (color 0 0 0 0)
+  )
   (junction (at 114.3 85.09) (diameter 0) (color 0 0 0 0)
   )
@@
   (junction (at 269.24 133.35) (diameter 0) (color 0 0 0 0)
   )
+  (junction (at 142.24 55.88) (diameter 0) (color 0 0 0 0)
+  )
   (junction (at 185.42 210.82) (diameter 0) (color 0 0 0 0)
   )
@@
     (stroke (width 0) (type default))
   )
+  (wire (pts (xy 139.7 60.96) (xy 142.24 60.96))
+    (stroke (width 0) (type default))
+  )
   (wire (pts (xy 339.09 181.61) (xy 339.09 215.9))
     (stroke (width 0) (type default))
@@
     (stroke (width 0) (type default))
   )
+  (wire (pts (xy 142.24 55.88) (xy 142.24 53.34))
+    (stroke (width 0) (type default))
+  )
   (wire (pts (xy 342.9 66.04) (xy 344.17 66.04))
     (stroke (width 0) (type default))
@@
     (stroke (width 0) (type default))
   )
+  (wire (pts (xy 142.24 60.96) (xy 146.05 60.96))
+    (stroke (width 0) (type default))
+  )
   (wire (pts (xy 210.82 218.44) (xy 218.44 218.44))
     (stroke (width 0) (type default))
@@
     (stroke (width 0) (type default))
   )
+  (wire (pts (xy 142.24 55.88) (xy 142.24 60.96))
+    (stroke (width 0) (type default))
+  )
   (wire (pts (xy 163.83 275.59) (xy 168.91 275.59))
     (stroke (width 0) (type default))
@@
     (stroke (width 0) (type default))
   )
+  (wire (pts (xy 139.7 55.88) (xy 142.24 55.88))
+    (stroke (width 0) (type default))
+  )
   (wire (pts (xy 312.42 161.29) (xy 298.45 161.29))
     (stroke (width 0) (type default))
@@
     (effects (font (size 1.27 1.27) (thickness 0.254) bold) (justify right top))
   )
+  (text_box "Misc. holes"
+    (at 133.35 33.02 0) (size 19.05 33.02)
+    (stroke (width 0) (type default))
+    (fill (type none))
+    (effects (font (size 1.27 1.27) (thickness 0.254) bold) (justify left top))
+  )
   (text_box "CW envelope shaping"
     (at 241.3 231.14 0) (size 55.88 40.64)
@@
     )
   )
+  (symbol (lib_id "power:GND") (at 140.97 38.1 0) (unit 1)
+    (in_bom yes) (on_board yes) (dnp no) (fields_autoplaced)
+    (property "Reference" "#PWR022" (at 140.97 44.45 0)
+      (effects (font (size 1.27 1.27)) hide)
+    )
+    (property "Value" "GND" (at 140.97 42.2331 0)
+      (effects (font (size 1.27 1.27)))
+    )
+    (property "Footprint" "" (at 140.97 38.1 0)
+      (effects (font (size 1.27 1.27)) hide)
+    )
+    (property "Datasheet" "" (at 140.97 38.1 0)
+      (effects (font (size 1.27 1.27)) hide)
+    )
+    (pin "1")
+    (instances
+      (project "T41-RF-board-V012"
+        (path "/3c4b9d3b-a516-4fd7-b325-b74c836dee65"
+          (reference "#PWR022") (unit 1)
+        )
+      )
+    )
+  )
   (symbol (lib_id "Device:C") (at 309.88 33.02 0) (mirror x) (unit 1)
     (in_bom yes) (on_board yes) (dnp no)
@@
     )
   )
+  (symbol (lib_id "Connector:TestPoint") (at 139.7 60.96 90) (unit 1)
+    (in_bom yes) (on_board yes) (dnp no)
+    (property "Reference" "G3" (at 135.89 58.42 90)
+      (effects (font (size 1.27 1.27)))
+    )
+    (property "Value" "TestPoint" (at 139.7 63.5 90)
+      (effects (font (size 1.27 1.27)))
+    )
+    (property "Footprint" "Connector_PinHeader_2.54mm:PinHeader_1x01_P2.54mm_Vertical" (at 139.7 55.88 0)
+      (effects (font (size 1.27 1.27)) hide)
+    )
+    (property "Datasheet" "~" (at 139.7 55.88 0)
+      (effects (font (size 1.27 1.27)) hide)
+    )
+    (property "Mouser Part Number" "" (at 139.7 60.96 0)
+      (effects (font (size 1.27 1.27)) hide)
+    )
+    (pin "1")
+    (instances
+      (project "T41-RF-board-V012"
+        (path "/3c4b9d3b-a516-4fd7-b325-b74c836dee65"
+          (reference "G3") (unit 1)
+        )
+      )
+    )
+  )
   (symbol (lib_id "Oscillator:Si5351A-B-GT") (at 325.12 156.21 0) (mirror y) (unit 1)
     (in_bom yes) (on_board yes) (dnp no)
@@
     )
   )
+  (symbol (lib_id "Connector:TestPoint") (at 142.24 53.34 0) (unit 1)
+    (in_bom yes) (on_board yes) (dnp no)
+    (property "Reference" "G1" (at 143.51 49.53 0)
+      (effects (font (size 1.27 1.27)) (justify left))
+    )
+    (property "Value" "TestPoint" (at 142.24 52.07 0)
+      (effects (font (size 1.27 1.27)) (justify left))
+    )
+    (property "Footprint" "Connector_PinHeader_2.54mm:PinHeader_1x01_P2.54mm_Vertical" (at 147.32 53.34 0)
+      (effects (font (size 1.27 1.27)) hide)
+    )
+    (property "Datasheet" "~" (at 147.32 53.34 0)
+      (effects (font (size 1.27 1.27)) hide)
+    )
+    (property "Mouser Part Number" "" (at 142.24 53.34 0)
+      (effects (font (size 1.27 1.27)) hide)
+    )
+    (pin "1")
+    (instances
+      (project "T41-RF-board-V012"
+        (path "/3c4b9d3b-a516-4fd7-b325-b74c836dee65"
+          (reference "G1") (unit 1)
+        )
+      )
+    )
+  )
   (symbol (lib_id "Device:C") (at 38.1 236.22 270) (mirror x) (unit 1)
     (in_bom yes) (on_board yes) (dnp no)
@@
     )
   )
+  (symbol (lib_id "Mechanical:MountingHole_Pad") (at 143.51 38.1 270) (unit 1)
+    (in_bom no) (on_board yes) (dnp no) (fields_autoplaced)
+    (property "Reference" "H1" (at 147.32 38.1 90)
+      (effects (font (size 1.27 1.27)) (justify left))
+    )
+    (property "Value" "~" (at 147.32 39.3121 90)
+      (effects (font (size 1.27 1.27)) (justify left))
+    )
+    (property "Footprint" "MountingHole:MountingHole_3.2mm_M3_Pad" (at 143.51 38.1 0)
+      (effects (font (size 1.27 1.27)) hide)
+    )
+    (property "Datasheet" "~" (at 143.51 38.1 0)
+      (effects (font (size 1.27 1.27)) hide)
+    )
+    (property "Mouser Part Number" "" (at 143.51 38.1 0)
+      (effects (font (size 1.27 1.27)) hide)
+    )
+    (pin "1")
+    (instances
+      (project "T41-RF-board-V012"
+        (path "/3c4b9d3b-a516-4fd7-b325-b74c836dee65"
+          (reference "H1") (unit 1)
+        )
+      )
+    )
+  )
   (symbol (lib_id "Device:R") (at 281.94 109.22 0) (mirror y) (unit 1)
     (in_bom yes) (on_board yes) (dnp no)
@@
     )
   )
+  (symbol (lib_id "power:GND") (at 146.05 60.96 0) (unit 1)
+    (in_bom yes) (on_board yes) (dnp no) (fields_autoplaced)
+    (property "Reference" "#PWR098" (at 146.05 67.31 0)
+      (effects (font (size 1.27 1.27)) hide)
+    )
+    (property "Value" "GND" (at 146.05 65.0931 0)
+      (effects (font (size 1.27 1.27)))
+    )
+    (property "Footprint" "" (at 146.05 60.96 0)
+      (effects (font (size 1.27 1.27)) hide)
+    )
+    (property "Datasheet" "" (at 146.05 60.96 0)
+      (effects (font (size 1.27 1.27)) hide)
+    )
+    (pin "1")
+    (instances
+      (project "T41-RF-board-V012"
+        (path "/3c4b9d3b-a516-4fd7-b325-b74c836dee65"
+          (reference "#PWR098") (unit 1)
+        )
+      )
+    )
+  )
   (symbol (lib_id "power:GND") (at 273.05 201.93 0) (unit 1)
     (in_bom yes) (on_board yes) (dnp no)
@@
         )
       )
+    )
+  )
+  (symbol (lib_id "Connector:TestPoint") (at 139.7 55.88 90) (unit 1)
+    (in_bom yes) (on_board yes) (dnp no)
+    (property "Reference" "G2" (at 135.89 53.34 90)
+      (effects (font (size 1.27 1.27)))
+    )
+    (property "Value" "TestPoint" (at 142.24 57.15 90)
+      (effects (font (size 1.27 1.27)))
+    )
+    (property "Footprint" "Connector_PinHeader_2.54mm:PinHeader_1x01_P2.54mm_Vertical" (at 139.7 50.8 0)
+      (effects (font (size 1.27 1.27)) hide)
+    )
+    (property "Datasheet" "~" (at 139.7 50.8 0)
+      (effects (font (size 1.27 1.27)) hide)
+    )
+    (property "Mouser Part Number" "" (at 139.7 55.88 0)
+      (effects (font (size 1.27 1.27)) hide)
+    )
+    (pin "1")
+    (instances
+      (project "T41-RF-board-V012"
+        (path "/3c4b9d3b-a516-4fd7-b325-b74c836dee65"
+          (reference "G2") (unit 1)
+        )
+      )

Commit message: Fixed errata in KI3P RF board test report
Parts:
- added H2, H3: ~, MountingHole:MountingHole_3mm_Pad, symbol Mechanical:MountingHole
- U16: value MC33078 -> LM358B
- U17: symbol Regulator_Linear:LM317L_TO92 -> Regulator_Linear:LM317L_SO8
Connections:
- net +12V: now also U17.1 (VI); no longer U17.3 (VI)
- net at R56.1, R57.2, U16.1: now also U17.4 (ADJ); no longer U17.1 (ADJ)
- net at R54.2, R57.1, U17.2 (VO): now also U17.3 (VO), U17.6 (VO), U17.7 (VO)
Changed lines of the file:
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@@
   (title_block
     (title "T41 RF Board")
-    (date "2024-02-17")
+    (date "2024-02-25")
     (rev "V012.6")
     (comment 1 "        Transcribed to KiCAD by OG King-KI3P")
@@
     )
   )
+  (symbol (lib_id "Mechanical:MountingHole") (at 137.16 45.72 0) (unit 1)
+    (in_bom yes) (on_board yes) (dnp no)
+    (property "Reference" "H2" (at 137.16 40.64 90)
+      (effects (font (size 1.27 1.27)))
+    )
+    (property "Value" "~" (at 139.7 46.9321 0)
+      (effects (font (size 1.27 1.27)) (justify left))
+    )
+    (property "Footprint" "MountingHole:MountingHole_3mm_Pad" (at 137.16 45.72 0)
+      (effects (font (size 1.27 1.27)) hide)
+    )
+    (property "Datasheet" "~" (at 137.16 45.72 0)
+      (effects (font (size 1.27 1.27)) hide)
+    )
+    (property "Mouser" "" (at 137.16 45.72 0)
+      (effects (font (size 1.27 1.27)) hide)
+    )
+    (property "Tayda" "" (at 137.16 45.72 0)
+      (effects (font (size 1.27 1.27)) hide)
+    )
+    (property "PJRC.com" "" (at 137.16 45.72 0)
+      (effects (font (size 1.27 1.27)) hide)
+    )
+    (instances
+      (project "T41-RF-board-V012"
+        (path "/3c4b9d3b-a516-4fd7-b325-b74c836dee65"
+          (reference "H2") (unit 1)
+        )
+      )
+    )
+  )
   (symbol (lib_id "T41_Library:ECS-TX053-S3") (at 368.3 147.32 0) (mirror y) (unit 1)
     (in_bom yes) (on_board yes) (dnp no)
@@
     )
   )
+  (symbol (lib_id "Mechanical:MountingHole") (at 142.24 45.72 270) (unit 1)
+    (in_bom yes) (on_board yes) (dnp no)
+    (property "Reference" "H3" (at 147.32 45.72 90)
+      (effects (font (size 1.27 1.27)))
+    )
+    (property "Value" "~" (at 141.0279 48.26 0)
+      (effects (font (size 1.27 1.27)) (justify left))
+    )
+    (property "Footprint" "MountingHole:MountingHole_3mm_Pad" (at 142.24 45.72 0)
+      (effects (font (size 1.27 1.27)) hide)
+    )
+    (property "Datasheet" "~" (at 142.24 45.72 0)
+      (effects (font (size 1.27 1.27)) hide)
+    )
+    (property "Mouser" "" (at 142.24 45.72 0)
+      (effects (font (size 1.27 1.27)) hide)
+    )
+    (property "Tayda" "" (at 142.24 45.72 0)
+      (effects (font (size 1.27 1.27)) hide)
+    )
+    (property "PJRC.com" "" (at 142.24 45.72 0)
+      (effects (font (size 1.27 1.27)) hide)
+    )
+    (instances
+      (project "T41-RF-board-V012"
+        (path "/3c4b9d3b-a516-4fd7-b325-b74c836dee65"
+          (reference "H3") (unit 1)
+        )
+      )
+    )
+  )
   (symbol (lib_id "Device:L") (at 171.45 191.77 0) (mirror y) (unit 1)
     (in_bom yes) (on_board yes) (dnp no) (fields_autoplaced)
@@
     )
   )
-  (symbol (lib_id "Regulator_Linear:LM317L_TO92") (at 289.56 251.46 270) (mirror x) (unit 1)
+  (symbol (lib_id "Regulator_Linear:LM317L_SO8") (at 289.56 251.46 270) (mirror x) (unit 1)
     (in_bom yes) (on_board yes) (dnp no)
     (property "Reference" "U17" (at 292.227 252.6721 90)
@@
       (effects (font (size 1.27 1.27)) (justify left))
     )
-    (property "Footprint" "Package_SO:SOIC-8_3.9x4.9mm_P1.27mm" (at 295.275 251.46 0)
+    (property "Footprint" "Package_SO:SOIC-8_3.9x4.9mm_P1.27mm" (at 294.64 251.46 0)
       (effects (font (size 1.27 1.27) italic) hide)
     )
-    (property "Datasheet" "http://www.ti.com/lit/ds/snvs775k/snvs775k.pdf" (at 289.56 251.46 0)
+    (property "Datasheet" "http://www.ti.com/lit/ds/snvs775k/snvs775k.pdf" (at 284.48 251.46 0)
       (effects (font (size 1.27 1.27)) hide)
     )
@@
     (pin "1")
     (pin "3")
+    (pin "7")
+    (pin "6")
+    (pin "8")
+    (pin "4")
+    (pin "5")
     (instances
       (project "T41-RF-board-V012"
@@
       (effects (font (size 1.27 1.27)))
     )
-    (property "Value" "MC33078" (at 279.4 263.8369 90)
+    (property "Value" "LM358B" (at 279.4 263.8369 90)
       (effects (font (size 1.27 1.27)))
     )
@@
   (symbol (lib_id "Amplifier_Operational:MC33078") (at 274.32 250.19 0) (unit 1)
     (in_bom yes) (on_board yes) (dnp no) (fields_autoplaced)
-    (property "Reference" "U16" (at 274.32 240.9657 0)
+    (property "Reference" "U16" (at 274.32 240.03 0)
       (effects (font (size 1.27 1.27)))
     )
-    (property "Value" "MC33078" (at 274.32 243.3899 0)
+    (property "Value" "LM358B" (at 274.32 242.57 0)
       (effects (font (size 1.27 1.27)))
     )

Commit message: Added heatsink model to RF board to confirm component fit. Tweaked locations of a few components.
Parts:
- removed H2, H3: ~, MountingHole:MountingHole_3mm_Pad, symbol Mechanical:MountingHole
- added H4: EA-T220-38E, EAT22038E, symbol T41_Library:EA-T220-38E
Connections:
- no-connect marks 12 -> 14
Other:
- moved on the sheet: H1
Changed lines of the file:
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@@
   )
   (no_connect (at 26.67 220.98))
+  (no_connect (at 135.89 43.18))
   (no_connect (at 93.98 144.78))
   (no_connect (at 93.98 167.64))
@@
   (no_connect (at 393.7 66.04))
   (no_connect (at 393.7 71.12))
+  (no_connect (at 135.89 40.64))
   (no_connect (at 156.21 156.21))
   (no_connect (at 93.98 147.32))
@@
   )
   (text_box "Misc. holes"
-    (at 133.35 33.02 0) (size 19.05 33.02)
+    (at 133.35 29.21 0) (size 24.13 40.64)
     (stroke (width 0) (type default))
     (fill (type none))
@@
   )
   (text_box "Board mounting holes"
-    (at 133.35 12.7 0) (size 19.05 17.78)
+    (at 133.35 12.7 0) (size 24.13 16.51)
     (stroke (width 0) (type default))
     (fill (type none))
@@
     )
   )
-  (symbol (lib_id "Mechanical:MountingHole") (at 137.16 45.72 0) (unit 1)
-    (in_bom yes) (on_board yes) (dnp no)
-    (property "Reference" "H2" (at 137.16 40.64 90)
-      (effects (font (size 1.27 1.27)))
-    )
-    (property "Value" "~" (at 139.7 46.9321 0)
-      (effects (font (size 1.27 1.27)) (justify left))
-    )
-    (property "Footprint" "MountingHole:MountingHole_3mm_Pad" (at 137.16 45.72 0)
-      (effects (font (size 1.27 1.27)) hide)
-    )
-    (property "Datasheet" "~" (at 137.16 45.72 0)
-      (effects (font (size 1.27 1.27)) hide)
-    )
-    (property "Mouser" "" (at 137.16 45.72 0)
-      (effects (font (size 1.27 1.27)) hide)
-    )
-    (property "Tayda" "" (at 137.16 45.72 0)
-      (effects (font (size 1.27 1.27)) hide)
-    )
-    (property "PJRC.com" "" (at 137.16 45.72 0)
-      (effects (font (size 1.27 1.27)) hide)
-    )
-    (instances
-      (project "T41-RF-board-V012"
-        (path "/3c4b9d3b-a516-4fd7-b325-b74c836dee65"
-          (reference "H2") (unit 1)
-        )
-      )
-    )
-  )
   (symbol (lib_id "T41_Library:ECS-TX053-S3") (at 368.3 147.32 0) (mirror y) (unit 1)
     (in_bom yes) (on_board yes) (dnp no)
@@
     )
   )
-  (symbol (lib_id "Mechanical:MountingHole") (at 142.24 45.72 270) (unit 1)
-    (in_bom yes) (on_board yes) (dnp no)
-    (property "Reference" "H3" (at 147.32 45.72 90)
-      (effects (font (size 1.27 1.27)))
-    )
-    (property "Value" "~" (at 141.0279 48.26 0)
-      (effects (font (size 1.27 1.27)) (justify left))
-    )
-    (property "Footprint" "MountingHole:MountingHole_3mm_Pad" (at 142.24 45.72 0)
-      (effects (font (size 1.27 1.27)) hide)
-    )
-    (property "Datasheet" "~" (at 142.24 45.72 0)
-      (effects (font (size 1.27 1.27)) hide)
-    )
-    (property "Mouser" "" (at 142.24 45.72 0)
-      (effects (font (size 1.27 1.27)) hide)
-    )
-    (property "Tayda" "" (at 142.24 45.72 0)
-      (effects (font (size 1.27 1.27)) hide)
-    )
-    (property "PJRC.com" "" (at 142.24 45.72 0)
-      (effects (font (size 1.27 1.27)) hide)
-    )
-    (instances
-      (project "T41-RF-board-V012"
-        (path "/3c4b9d3b-a516-4fd7-b325-b74c836dee65"
-          (reference "H3") (unit 1)
-        )
-      )
-    )
-  )
   (symbol (lib_id "Device:L") (at 171.45 191.77 0) (mirror y) (unit 1)
     (in_bom yes) (on_board yes) (dnp no) (fields_autoplaced)
@@
     )
   )
-  (symbol (lib_id "power:GND") (at 140.97 38.1 0) (unit 1)
+  (symbol (lib_id "power:GND") (at 149.86 57.15 0) (unit 1)
     (in_bom yes) (on_board yes) (dnp no) (fields_autoplaced)
-    (property "Reference" "#PWR022" (at 140.97 44.45 0)
+    (property "Reference" "#PWR022" (at 149.86 63.5 0)
       (effects (font (size 1.27 1.27)) hide)
     )
-    (property "Value" "GND" (at 140.97 42.2331 0)
+    (property "Value" "GND" (at 149.86 61.2831 0)
       (effects (font (size 1.27 1.27)))
     )
-    (property "Footprint" "" (at 140.97 38.1 0)
+    (property "Footprint" "" (at 149.86 57.15 0)
       (effects (font (size 1.27 1.27)) hide)
     )
-    (property "Datasheet" "" (at 140.97 38.1 0)
+    (property "Datasheet" "" (at 149.86 57.15 0)
       (effects (font (size 1.27 1.27)) hide)
     )
@@
     )
   )
+  (symbol (lib_id "T41_Library:EA-T220-38E") (at 135.89 40.64 0) (unit 1)
+    (in_bom yes) (on_board yes) (dnp no)
+    (property "Reference" "H4" (at 144.78 34.29 0)
+      (effects (font (size 1.27 1.27)) (justify left))
+    )
+    (property "Value" "EA-T220-38E" (at 139.7 36.83 0)
+      (effects (font (size 1.27 1.27)) (justify left))
+    )
+    (property "Footprint" "EAT22038E" (at 152.4 135.56 0)
+      (effects (font (size 1.27 1.27)) (justify left top) hide)
+    )
+    (property "Datasheet" "https://www.ohmite.com/assets/docs/sink_e.pdf?r=false" (at 152.4 235.56 0)
+      (effects (font (size 1.27 1.27)) (justify left top) hide)
+    )
+    (property "Height" "38.35" (at 152.4 435.56 0)
+      (effects (font (size 1.27 1.27)) (justify left top) hide)
+    )
+    (property "Mouser Part Number" "588-EA-T220-38E" (at 152.4 535.56 0)
+      (effects (font (size 1.27 1.27)) (justify left top) hide)
+    )
+    (property "Mouser Price/Stock" "https://www.mouser.co.uk/ProductDetail/Ohmite/EA-T220-38E?qs=6weo7U0lPxCX9kcQhGcuZQ%3D%3D" (at 152.4 635.56 0)
+      (effects (font (size 1.27 1.27)) (justify left top) hide)
+    )
+    (property "Manufacturer_Name" "Ohmite" (at 152.4 735.56 0)
+      (effects (font (size 1.27 1.27)) (justify left top) hide)
+    )
+    (property "Manufacturer_Part_Number" "EA-T220-38E" (at 152.4 835.56 0)
+      (effects (font (size 1.27 1.27)) (justify left top) hide)
+    )
+    (pin "1")
+    (pin "2")
+    (instances
+      (project "T41-RF-board-V012"
+        (path "/3c4b9d3b-a516-4fd7-b325-b74c836dee65"
+          (reference "H4") (unit 1)
+        )
+      )
+    )
+  )
   (symbol (lib_id "Amplifier_Operational:MC33078") (at 99.06 205.74 0) (mirror x) (unit 2)
     (in_bom yes) (on_board yes) (dnp no)
@@
     )
   )
-  (symbol (lib_id "Mechanical:MountingHole_Pad") (at 143.51 38.1 270) (unit 1)
+  (symbol (lib_id "Mechanical:MountingHole_Pad") (at 152.4 57.15 270) (unit 1)
     (in_bom no) (on_board yes) (dnp no) (fields_autoplaced)
-    (property "Reference" "H1" (at 147.32 38.1 90)
+    (property "Reference" "H1" (at 156.21 57.15 90)
       (effects (font (size 1.27 1.27)) (justify left))
     )
-    (property "Value" "~" (at 147.32 39.3121 90)
+    (property "Value" "~" (at 156.21 58.3621 90)
       (effects (font (size 1.27 1.27)) (justify left))
     )
-    (property "Footprint" "MountingHole:MountingHole_3.2mm_M3_Pad" (at 143.51 38.1 0)
+    (property "Footprint" "MountingHole:MountingHole_3.2mm_M3_Pad" (at 152.4 57.15 0)
       (effects (font (size 1.27 1.27)) hide)
     )
-    (property "Datasheet" "~" (at 143.51 38.1 0)
+    (property "Datasheet" "~" (at 152.4 57.15 0)
       (effects (font (size 1.27 1.27)) hide)
     )
-    (property "Mouser Part Number" "" (at 143.51 38.1 0)
+    (property "Mouser Part Number" "" (at 152.4 57.15 0)
       (effects (font (size 1.27 1.27)) hide)
     )

Commit message: Added CAL isolation jumper to RF board to improve Bode plot measurement
Parts:
- added JP4: CAL isolation, Connector_PinHeader_2.54mm:PinHeader_1x02_P2.54mm_Vertical, symbol Jumper:Jumper_2_Open
Connections:
- net RFIN: now also JP4.1 (A); no longer C16.1, J2.1 (In)
- new net: C16.1, J2.1 (In), JP4.2 (B)
