File: T41_V012_Files_01-15-24/T41_V012_KiCad/T41-RF-board-V012/T41-RF-board-V012.kicad_sch (KiCad schematic)
At the start: 232 parts, among them J1 IQ_Out, J2 RF_IN, J3 RFControl, J4 12-13.8V, J5 IQ_In, J6 RF_OUT, Q1 BS170, U1 74CBTLV3253DR, U10 SN74LVC1G04DCK, U106 MC33078, U107 MC33078, U11 Si5351A-B-GT, U12 PE4312, U13 MAR-3SM+, U14 LM7805CT, U15 LM1117T-3.3, U16 LM358B, U17 LM317L, U18 SN74LVC1G04DCK, U19 MASWSS0179, U2 PSA-8A+, U20 MASWSS0179, U21 MCP23017_SO, U22 HMC434E, U23 HMC434E, U3 PE4312, U4 74CBTLV3253DR, U5 SN74LVC1G04DCK, U6 MC33078, U7 MASWSS0179, U8 MC33078, U9 MASWSS0179, Y1 ECS-TX053-S3, Y2 25MHz

Commit message: Added R73 to RF board to adjust off ramp time
Parts:
- added R73: 100k, Resistor_SMD:R_1206_3216Metric, symbol Device:R
Connections:
- net GND: now also R73.2
- net at C73.2, R58.1, U16.3 (+): now also R73.1
Other:
- note added: "R73 stacked on top of C73"
Changed lines of the file:
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@@
 	(title_block
 		(title "T41 RF Board")
-		(date "2024-04-08")
+		(date "2024-07-18")
 		(rev "V012.6")
 		(comment 1 "        Transcribed to KiCAD by OG King-KI3P")
 		(comment 2 "By Al Peter-AC8GY, Revised by WJ Schmidt-K9HZ")
-		(comment 3 "Change log: switched the order of attenuator and amp in receive chain")
-		(comment 4 "  - Added ground test points & pad, silkscreen edits")
-		(comment 5 "  - Added JP4 for electrical disconnect of CAL signal (4/8/24)")
+		(comment 3 "Change log: Added R73 to schematic")
 	)
 	(junction
@@
 	)
 	(junction
+		(at 260.35 251.46)
+		(diameter 0)
+		(color 0 0 0 0)
+	)
+	(junction
 		(at 106.68 241.3)
 		(diameter 0)
@@
 	)
 	(junction
+		(at 260.35 259.08)
+		(diameter 0)
+		(color 0 0 0 0)
+	)
+	(junction
 		(at 78.74 96.52)
 		(diameter 0)
@@
 	(wire
 		(pts
+			(xy 251.46 259.08) (xy 260.35 259.08)
+		)
+		(stroke
+			(width 0)
+			(type default)
+		)
+	)
+	(wire
+		(pts
 			(xy 177.8 62.23) (xy 177.8 63.5)
 		)
@@
 	(wire
 		(pts
+			(xy 251.46 251.46) (xy 260.35 251.46)
+		)
+		(stroke
+			(width 0)
+			(type default)
+		)
+	)
+	(wire
+		(pts
 			(xy 85.09 99.06) (xy 87.63 99.06)
 		)
@@
 		)
 	)
+	(text "R73 stacked \non top of C73"
+		(exclude_from_sim no)
+		(at 251.46 262.89 0)
+		(effects
+			(font
+				(size 1.27 1.27)
+			)
+		)
+	)
 	(text "10T"
 		(exclude_from_sim no)
@@
 	)
 	(symbol
+		(lib_id "Device:R")
+		(at 251.46 255.27 0)
+		(mirror y)
+		(unit 1)
+		(exclude_from_sim no)
+		(in_bom yes)
+		(on_board no)
+		(dnp no)
+		(property "Reference" "R73"
+			(at 248.92 254.3697 0)
+			(effects
+				(font
+					(size 1.27 1.27)
+				)
+				(justify left)
+			)
+		)
+		(property "Value" "100k"
+			(at 248.92 256.794 0)
+			(effects
+				(font
+					(size 1.27 1.27)
+				)
+				(justify left)
+			)
+		)
+		(property "Footprint" "Resistor_SMD:R_1206_3216Metric"
+			(at 253.238 255.27 90)
+			(effects
+				(font
+					(size 1.27 1.27)
+				)
+				(hide yes)
+			)
+		)
+		(property "Datasheet" "~"
+			(at 251.46 255.27 0)
+			(effects
+				(font
+					(size 1.27 1.27)
+				)
+				(hide yes)
+			)
+		)
+		(property "Description" ""
+			(at 251.46 255.27 0)
+			(effects
+				(font
+					(size 1.27 1.27)
+				)
+				(hide yes)
+			)
+		)
+		(property "Mouser Part Number" ""
+			(at 251.46 255.27 0)
+			(effects
+				(font
+					(size 1.27 1.27)
+				)
+				(hide yes)
+			)
+		)
+		(pin "2"
+		)
+		(pin "1"
+		)
+		(instances
+			(project "T41-RF-board-V012"
+				(path "/3c4b9d3b-a516-4fd7-b325-b74c836dee65"
+					(reference "R73")
+					(unit 1)
+				)
+			)
+		)
+	)
+	(symbol
 		(lib_id "power:GND")
 		(at 278.13 66.04 0)
@@
 		)
 		(property "Value" "0.1uF 50V"
-			(at 254 257.81 0)
+			(at 259.334 257.81 0)
 			(effects
 				(font

Commit message: Updated C5,C8,C19,C21 values per Al
Parts:
- C19, C8: value 68pF 50V -> 180pF 50V
- C21, C5: value 68pF 50V -> 105pF 50V
Changed lines of the file:
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@@
 		(comment 1 "        Transcribed to KiCAD by OG King-KI3P")
 		(comment 2 "By Al Peter-AC8GY, Revised by WJ Schmidt-K9HZ")
-		(comment 3 "Change log: Added R73 to schematic")
+		(comment 3 "Change log: Added R73 to schematic, updated C5,C8,C19,C21")
 	)
 	(junction
@@
 			)
 		)
-		(property "Value" "68pF 50V"
+		(property "Value" "180pF 50V"
 			(at 319.659 49.4721 0)
 			(effects
@@
 			)
 		)
-		(property "Value" "68pF 50V"
+		(property "Value" "105pF 50V"
 			(at 326.39 111.76 90)
 			(effects
@@
 			)
 		)
-		(property "Value" "68pF 50V"
+		(property "Value" "105pF 50V"
 			(at 326.39 63.5 90)
 			(effects
@@
 			)
 		)
-		(property "Value" "68pF 50V"
+		(property "Value" "180pF 50V"
 			(at 319.659 97.7321 0)
 			(effects

Commit message: Correct R35 and R37 to 0R on the RF board
Parts:
- R35, R37: value 3k3 -> 0
Changed lines of the file:
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@@
 	(title_block
 		(title "T41 RF Board")
-		(date "2024-07-18")
+		(date "2024-09-07")
 		(rev "V012.6")
 		(comment 1 "        Transcribed to KiCAD by OG King-KI3P")
 		(comment 2 "By Al Peter-AC8GY, Revised by WJ Schmidt-K9HZ")
-		(comment 3 "Change log: Added R73 to schematic, updated C5,C8,C19,C21")
+		(comment 3 "Change log: Changed R35&R37 to 0R")
 	)
 	(junction
@@
 			)
 		)
-		(property "Value" "3k3"
+		(property "Value" "0"
 			(at 205.74 144.9761 90)
 			(effects
@@
 			)
 		)
-		(property "Value" "3k3"
+		(property "Value" "0"
 			(at 205.74 165.2961 90)
 			(effects
