File: T41_V012_Files_01-15-24/T41_V012_KiCad/T41-RF-board-V012/T41-RF-board-V012.kicad_sch (KiCad schematic)
At the start: 233 parts, among them J1 IQ_Out, J2 RF_IN, J3 RFControl, J4 12-13.8V, J5 IQ_In, J6 RF_OUT, Q1 BS170, U1 74CBTLV3253DR, U10 SN74LVC1G04DCK, U106 MC33078, U107 MC33078, U11 Si5351A-B-GT, U12 PE4312, U13 MAR-3SM+, U14 LM7805CT, U15 LM1117T-3.3, U16 LM358B, U17 LM317L, U18 SN74LVC1G04DCK, U19 MASWSS0179, U2 PSA-8A+, U20 MASWSS0179, U21 MCP23017_SO, U22 HMC434E, U23 HMC434E, U3 PE4312, U4 74CBTLV3253DR, U5 SN74LVC1G04DCK, U6 MC33078, U7 MASWSS0179, U8 MC33078, U9 MASWSS0179, Y1 ECS-TX053-S3, Y2 25MHz

Commit message: RF board updates: removed clock divider, replaces IQ output caps with 0R, added cap to FB for TCXO
Parts:
- removed C14, C3: 10uF 50V, Capacitor_SMD:C_1206_3216Metric, symbol Device:C
- removed C74, C75, C77, C79, C83, C84: 0.1uF 50V, Capacitor_SMD:C_1206_3216Metric, symbol Device:C
- removed C76, C78, C81, C82: 100pF, Capacitor_SMD:C_1206_3216Metric, symbol Device:C
- removed JP18, JP19: PrescalarBypass, Connector_PinHeader_2.54mm:PinHeader_1x02_P2.54mm_Vertical, symbol Jumper:Jumper_2_Open
- removed U18: SN74LVC1G04DCK, T41_Library:SOT-SC70, symbol 74xGxx:74LVC1G04
- removed U19, U20: MASWSS0179, T41_Library:MASWSS0179-SOT-26, symbol RF_Switch:MASWSS0179
- removed U22, U23: HMC434E, Package_TO_SOT_SMD:SOT-23-6, symbol T41_Library:HMC434E
- added C85: 0.1uF 50V, Capacitor_SMD:C_1206_3216Metric, symbol Device:C
- added R64, R65: 0, Resistor_SMD:R_1206_3216Metric, symbol Device:R
Connections:
- net GND: now also C85.1
- net I_out: now also R65.2
- net Q_out: now also R64.2
- net at R35.2, R40.2, TP15.1: now also U11.10 (CLK0)
- net at C21.1, R11.2, U107.7: now also R65.1
- net at C5.1, R2.2, U107.1: now also R64.1
- net at R37.2, R42.2, TP16.1: now also U11.9 (CLK1)
- net at L7.1, Y1.9 (VDD): now also C85.2
- net MF/HF: no longer names the net of U21.28 (GPA7)
- no-connect marks 14 -> 15
Other:
- note removed: "<- CLOCK GENERATION AND CONTROL"
- note removed: "Divide by 8"
- note removed: "Prescalar Divide-By-8 and relays only required for MF (160m operation). Bypass using JP18 & JP19 if not needed."
- moved on the sheet: C49, C52, L107, L7, U11, Y1, Y2

Commit message: Added bypass capacitor to TCXO, removed clock divider circuit, replaced I/Q output DC blocking capacitors with 0R resistors
Parts:
- added G4, G5, G6: TestPoint, Connector_PinHeader_2.54mm:PinHeader_1x01_P2.54mm_Vertical, symbol Connector:TestPoint
- added JP5: CLK0, Connector_PinHeader_2.54mm:PinHeader_1x02_P2.54mm_Vertical, symbol Jumper:Jumper_2_Open
- added JP6: CLK1, Connector_PinHeader_2.54mm:PinHeader_1x02_P2.54mm_Vertical, symbol Jumper:Jumper_2_Open
- U106: value MC33078 -> AD8599
- U107: value MC33078 -> OPA2209
Connections:
- net GND: now also G4.1, G5.1, G6.1
- net at R35.2, R40.2, TP15.1: now also JP5.1 (A); no longer U11.10 (CLK0)
- net at R37.2, R42.2, TP16.1: now also JP6.1 (A); no longer U11.9 (CLK1)
- new net: JP6.2 (B), U11.9 (CLK1)
- new net: JP5.2 (B), U11.10 (CLK0)
