File: T41_V012_Files_01-15-24/T41_V012_KiCad/T41-RF-board-V012/T41-RF-board-V012.kicad_pcb (KiCad board)
At the start: 4 copper layers, 100 x 100 mm, 224 parts, among them J1 IQ_Out, J2 RF_IN, J3 RFControl, J4 12-13.8V, J5 IQ_In, J6 RF_OUT, Q1 BS170, U1 74CBTLV3253DR, U10 SN74LVC1G04DCK, U106 MC33078, U107 MC33078, U11 Si5351A-B-GT, U12 PE4312, U13 MAR-3SM+, U14 LM7805CT, U15 LM1117T-3.3, U16 MC33078, U17 LM317L, U18 SN74LVC1G04DCK, U19 MASWSS0179, U2 PSA-8A+, U20 MASWSS0179, U21 MCP23017_SO, U22 HMC434E, U23 HMC434E, U3 PE4312, U4 74CBTLV3253DR, U5 SN74LVC1G04DCK, U6 MC33078, U7 MASWSS0179, U8 MC33078, U9 MASWSS0179, Y1 ECS-TX053-S3, Y2 25MHz

Commit message: Switched order of attenuator and amplifier in receive chain. Now attenuator is before amplifier
Parts:
- moved C12 18.6 mm to (71.6, 74.6), turned to 0 degrees
- moved R14 15.8 mm to (75.7, 73.1), turned to 90 degrees
- moved U2 15.1 mm to (67.1, 69.0), turned to 0 degrees
- moved R24 14.7 mm to (65.8, 57.0)
- moved C29 14.1 mm to (63.1, 69.3), turned to -90 degrees
- moved C13 13.9 mm to (71.6, 71.1), turned to 0 degrees
- moved R28 13.7 mm to (73.5, 57.8), turned to 90 degrees
- moved JP3 11.7 mm to (64.5, 60.3), turned to 0 degrees
- moved L4 9.33 mm to (75.7, 68.5), turned to 90 degrees
- moved U3 8.24 mm to (69.2, 61.7), turned to -90 degrees
- moved C27 8.13 mm to (71.6, 66.5), turned to 0 degrees
Connections:
- C22 pad 2: Net-(U2-IN) -> Net-(JP3-A)
- C27 pad 2: Net-(JP3-A) -> Net-(U1-1A)
- R20 pad 2: Net-(JP3-B) -> Net-(U1-1A)
- TP6 pad 1: Net-(JP3-B) -> Net-(U1-1A)
- U1 pad 7: Net-(JP3-B) -> Net-(U1-1A)
- U1 pad 9: Net-(JP3-B) -> Net-(U1-1A)
- U2 pad 3: Net-(U2-IN) -> Net-(JP3-B)
Routing:
- net Net-(U1-1A): track 0.00 -> 32.9 mm
- net +5V: track 244.0 -> 218.1 mm
- net Net-(JP3-B): track 34.3 -> 13.0 mm
- net /RC16: track 41.7 -> 55.4 mm
- net /RC8: track 54.6 -> 44.4 mm
- net +3V3: track 368.9 -> 377.7 mm, vias 16 -> 17
- net /RC0.5: track 36.7 -> 44.8 mm
- net /RC4: track 50.9 -> 44.4 mm
- net Net-(JP3-A): track 23.8 -> 19.1 mm
- net Net-(U3-RF2): track 4.06 -> 8.58 mm
- net /RC1: track 40.7 -> 44.3 mm
- net Net-(U2-IN): track 3.11 -> 0.00 mm
- net /RC2: track 47.0 -> 44.0 mm
- net Net-(U3-Data): track 4.54 -> 3.57 mm
- net GND: track 47.2 -> 46.5 mm
Other:
- board text added: "T41 RF Board: V12.06 Designed by AC8GY/K9HZ Layout by KI3P 4 layer, 2024/01/25"
- board text removed: "T41 RF Board: V12.06 Designed by AC8GY/K9HZ Layout by KI3P 4 layer, 2024/01/14"

Commit message: Restored silkscreen registration dot on U2 of RF board to its rightful place
Routing:
- net GND: track 46.5 -> 52.4 mm
Changed lines of the file:
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@@
     (property "ki_keywords" "R res resistor")
     (attr smd)
-    (fp_text reference "R28" (at 0 -2.032 90) (layer "F.SilkS")
+    (fp_text reference "R28" (at 0.077 1.867 90) (layer "F.SilkS")
         (effects (font (size 1 1) (thickness 0.15)))
     )
@@
   (gr_line (start 136.525 145.034) (end 136.525 148.844)
     (stroke (width 0.15) (type default)) (layer "F.SilkS"))
-  (gr_circle (center 68.58 67.056) (end 68.834 67.056)
+  (gr_circle (center 71.4 59) (end 71.654 59)
     (stroke (width 0.15) (type solid)) (fill solid) (layer "F.SilkS"))
   (gr_line (start 123.952 120.269) (end 123.952 116.84)
@@
   (segment (start 126.484 138.676) (end 125.984 138.176) (width 0.2) (layer "F.Cu") (net 1))
   (segment (start 68.711 62.218) (end 69.211 61.718) (width 0.2) (layer "F.Cu") (net 1))
+  (segment (start 68.363 64.516) (end 66.675 64.516) (width 0.2) (layer "F.Cu") (net 1))
+  (segment (start 69.211 63.668) (end 68.211 63.668) (width 0.2) (layer "F.Cu") (net 1))
   (segment (start 113.284 95.885) (end 113.538 96.139) (width 0.2) (layer "F.Cu") (net 1))
   (segment (start 113.742 143.956) (end 112.079 143.956) (width 0.2) (layer "F.Cu") (net 1))
   (segment (start 127.934 139.176) (end 126.984 139.176) (width 0.2) (layer "F.Cu") (net 1))
+  (segment (start 69.211 63.668) (end 68.363 64.516) (width 0.2) (layer "F.Cu") (net 1))
+  (segment (start 66.675 63.304) (end 66.675 64.516) (width 0.2) (layer "F.Cu") (net 1))
   (segment (start 71.793047 61.718) (end 72.555047 62.48) (width 0.2) (layer "F.Cu") (net 1))
   (segment (start 92.837 87.884) (end 91.948 86.995) (width 0.2) (layer "F.Cu") (net 1))
@@
   (segment (start 69.211 63.668) (end 69.211 61.718) (width 0.2) (layer "F.Cu") (net 1))
   (segment (start 103.124 90.0375) (end 103.124 90.772994) (width 0.2) (layer "F.Cu") (net 1))
+  (segment (start 67.261 62.718) (end 66.675 63.304) (width 0.2) (layer "F.Cu") (net 1))
   (segment (start 112.079 143.956) (end 111.252 143.129) (width 0.2) (layer "F.Cu") (net 1))
   (segment (start 113.792 143.906) (end 113.742 143.956) (width 0.2) (layer "F.Cu") (net 1))

Commit message: Recreate these
Parts:
- added JP1: SolderJumper_2_Open, Jumper:SolderJumper-2_P1.3mm_Open_TrianglePad1.0x1.5mm, F.Cu at (82.1, 63.1)
- added JP2: SolderJumper_2_Bridged, Jumper:SolderJumper-2_P1.3mm_Bridged_RoundedPad1.0x1.5mm, F.Cu at (82.1, 60.6)
- moved L1 5.34 mm to (82.8, 66.8), turned to -90 degrees
- moved C6 3.15 mm to (84.0, 70.8), turned to 180 degrees
Connections:
- C6 pad 2: +3V3 -> Net-(U1-VCC)
- L1 pad 1: +3V3 -> Net-(JP1-A)
- R15 pad 1: +3V3 -> Net-(JP1-A)
Routing:
- net +5V: track 218.1 -> 232.6 mm, vias 5 -> 6
- net Net-(U1-1A): track 32.9 -> 43.5 mm
- net Net-(JP1-A): track 0.00 -> 9.29 mm
- net Net-(U1-S0): track 13.4 -> 16.7 mm
- net +3V3: track 377.7 -> 375.3 mm, vias 17 -> 15
- net Net-(U1-VCC): track 3.72 -> 5.38 mm
- net GND: track 52.4 -> 52.6 mm, vias 234 -> 232
Other:
- board text added: "3V3"
- board text added: "5V"
- board text added: "A0"
- board text added: "A1"
- board text added: "A2"
- board text added: "T41 RF Board: V12.06 Designed by AC8GY/K9HZ Layout by KI3P 4 layer, 2024/02/12"
- board text removed: "T41 RF Board: V12.06 Designed by AC8GY/K9HZ Layout by KI3P 4 layer, 2024/01/25"
