File: T41_V012_Files_01-15-24/T41_V012_KiCad/T41-RF-board-V012/T41-RF-board-V012.kicad_pcb (KiCad board)
At the start: 4 copper layers, 100 x 100 mm, 225 parts, among them J1 IQ_Out, J2 RF_IN, J3 RFControl, J4 12-13.8V, J5 IQ_In, J6 RF_OUT, Q1 BS170, U1 74CBTLV3253DR, U10 SN74LVC1G04DCK, U106 MC33078, U107 MC33078, U11 Si5351A-B-GT, U12 PE4312, U13 MAR-3SM+, U14 LM7805CT, U15 LM1117T-3.3, U16 MC33078, U17 LM317L, U18 SN74LVC1G04DCK, U19 MASWSS0179, U2 PSA-8A+, U20 MASWSS0179, U21 MCP23017_SO, U22 HMC434E, U23 HMC434E, U3 PE4312, U4 74CBTLV3253DR, U5 SN74LVC1G04DCK, U6 MC33078, U7 MASWSS0179, U8 MC33078, U9 MASWSS0179, Y1 ECS-TX053-S3, Y2 25MHz

Commit message: Added ground test points and pad, silkscreen edits
Parts:
- added C2: 1uF 50V, Capacitor_SMD:C_1206_3216Metric, F.Cu at (99.5, 55.9)
- added G1: TestPoint, Connector_PinHeader_2.54mm:PinHeader_1x01_P2.54mm_Vertical, F.Cu at (97.5, 52.8)
- added G2: TestPoint, Connector_PinHeader_2.54mm:PinHeader_1x01_P2.54mm_Vertical, F.Cu at (93.9, 144.8)
- added G3: TestPoint, Connector_PinHeader_2.54mm:PinHeader_1x01_P2.54mm_Vertical, F.Cu at (116.7, 113.8)
- added H1: ~, MountingHole:MountingHole_3.2mm_M3_Pad, F.Cu at (81.2, 82.0)
Routing:
- net GND: vias 232 -> 229
Other:
- board text added: "T41 RF Board: V12.06 Designed by AC8GY/K9HZ Layout by KI3P 4 layer, 2024/02/17"
- board text removed: "T41 RF Board: V12.06 Designed by AC8GY/K9HZ Layout by KI3P 4 layer, 2024/02/12"

Commit message: Corrected footprint for TCXO Y1
Parts:
- moved L7 5.06 mm to (111.3, 80.5)
- moved Y1 2.19 mm to (110.4, 84.0)
Routing:
- net +3V3: track 375.3 -> 369.9 mm
- net GND: vias 229 -> 227

Commit message: Fixed errata in KI3P RF board test report
Parts:
- added H2: ~, MountingHole:MountingHole_3mm_Pad, F.Cu at (129.2, 112.2)
- added H3: ~, MountingHole:MountingHole_3mm_Pad, F.Cu at (129.2, 86.8)
- U16: value MC33078 -> LM358B
- moved TP17 31.5 mm to (147.9, 72.9)
- moved L12 27.2 mm to (146.0, 79.2), turned to 90 degrees
- moved C70 26.5 mm to (147.6, 98.4)
- moved J4 26.1 mm to (143.7, 116.2)
- moved L13 22.1 mm to (146.2, 104.5), turned to 90 degrees
- moved U15 17.3 mm to (132.7, 102.0), turned to 90 degrees
- moved C68 16.8 mm to (147.6, 91.0)
- moved C67 14.7 mm to (136.9, 86.9)
- moved C69 14.0 mm to (138.4, 94.8), turned to 0 degrees
- moved L11 12.7 mm to (138.6, 104.6), turned to 90 degrees
- moved U14 10.0 mm to (146.3, 85.0)
- moved C71 5.86 mm to (137.9, 115.6), turned to -90 degrees
- moved TP18 4.28 mm to (120.5, 107.8)
- moved G3 1.27 mm to (115.8, 112.9)
- moved C72 0.24 mm to (137.9, 110.8)
Connections:
- R54 pad 2: Net-(U17-VO) -> Net-(R54-Pad2)
- R57 pad 1: Net-(U17-VO) -> Net-(R54-Pad2)
- U17 pad 1: Net-(U17-ADJ) -> +12V
- U17 pad 2: Net-(U17-VO) -> Net-(R54-Pad2)
- U17 pad 3: +12V -> Net-(R54-Pad2)
- U17 pad 4: (no net) -> Net-(U17-ADJ)
- U17 pad 5: (no net) -> unconnected-(U17-NC-Pad5)
- U17 pad 6: (no net) -> Net-(R54-Pad2)
- U17 pad 7: (no net) -> Net-(R54-Pad2)
- U17 pad 8: (no net) -> unconnected-(U17-NC-Pad8)
Routing:
- net Net-(R54-Pad2): track 0.00 -> 19.0 mm
- net +3V3: track 369.9 -> 386.0 mm, vias 15 -> 16
- net +12V: track 85.6 -> 98.9 mm, vias 2 -> 3
- net Net-(U15-VO): track 14.3 -> 27.5 mm
- net /RFIN: track 148.3 -> 136.4 mm
- net Net-(U17-VO): track 11.3 -> 0.00 mm
- net Net-(U14-VO): track 13.1 -> 20.0 mm, vias 0 -> 1
- net Net-(U17-ADJ): track 19.9 -> 23.9 mm
- net Net-(J4-Pin_1): track 10.4 -> 11.4 mm
- net GND: vias 227 -> 205
Other:
- board text added: "+12V"
- board text added: "Anti-alias filters"
- board text added: "GND"
- board text added: "T41 RF Board: V12.06 Designed by AC8GY/K9HZ Layout by KI3P 4 layer, 2024/02/25"
- board text removed: "Anti- alias filters"
- board text removed: "T41 RF Board: V12.06 Designed by AC8GY/K9HZ Layout by KI3P 4 layer, 2024/02/17"
- board text removed: "Transmit"
