File: T41_V012_Files_01-15-24/T41_V012_KiCad/T41-RF-board-V012/T41-RF-board-V012.kicad_pcb (KiCad board)
At the start: 4 copper layers, 100 x 100 mm, 232 parts, among them J1 IQ_Out, J2 RF_IN, J3 RFControl, J4 12-13.8V, J5 IQ_In, J6 RF_OUT, Q1 BS170, U1 74CBTLV3253DR, U10 SN74LVC1G04DCK, U106 MC33078, U107 MC33078, U11 Si5351A-B-GT, U12 PE4312, U13 MAR-3SM+, U14 LM7805CT, U15 LM1117T-3.3, U16 LM358B, U17 LM317L, U18 SN74LVC1G04DCK, U19 MASWSS0179, U2 PSA-8A+, U20 MASWSS0179, U21 MCP23017_SO, U22 HMC434E, U23 HMC434E, U3 PE4312, U4 74CBTLV3253DR, U5 SN74LVC1G04DCK, U6 MC33078, U7 MASWSS0179, U8 MC33078, U9 MASWSS0179, Y1 ECS-TX053-S3, Y2 25MHz

Commit message: Added heatsink model to RF board to confirm component fit. Tweaked locations of a few components.
Parts:
- removed H2, H3: ~, MountingHole:MountingHole_3mm_Pad
- added H4: EA-T220-38E, T41_Library:EAT22038E, F.Cu at (129.2, 112.2)
- moved Y2 0.74 mm to (119.2, 92.3)
- moved TP18 0.64 mm to (119.9, 107.6)
- moved C67 0.57 mm to (137.3, 86.5)
- moved L11 0.32 mm to (138.9, 104.5)
- moved R58 0.21 mm to (128.0, 118.6)
- moved C73 0.19 mm to (133.7, 118.5)
Routing:
- net GND: track 52.6 -> 53.6 mm, vias 205 -> 204
- net +3V3: track 386.0 -> 386.7 mm
- net Net-(U14-VO): track 20.0 -> 19.4 mm

Commit message: Added CAL isolation jumper to RF board to improve Bode plot measurement
Parts:
- added JP4: CAL isolation, Connector_PinHeader_2.54mm:PinHeader_1x02_P2.54mm_Vertical, F.Cu at (57.2, 84.6)
Connections:
- C16 pad 1: /RFIN -> Net-(J2-In)
- J2 pad 1: /RFIN -> Net-(J2-In)
Routing:
- net Net-(J2-In): track 0.00 -> 14.6 mm
- net /RFIN: track 136.4 -> 131.7 mm
Other:
- board text added: "CAL Isolation"
- board text added: "Receive RF IN"
- board text added: "T41 RF Board: V12.06 Designed by AC8GY/K9HZ Layout by KI3P 4 layer, 2024/04/08"
- board text removed: "RF IN"
- board text removed: "Receive"
- board text removed: "T41 RF Board: V12.06 Designed by AC8GY/K9HZ Layout by KI3P 4 layer, 2024/02/25"

Commit message: Updated silkscreen for RF Board Y1 to put indicator dot in the correct location
Other:
- board text added: "T41 RF Board: V12.06 Designed by AC8GY/K9HZ Layout by KI3P 4 layer, 2024/06/30"
- board text removed: "T41 RF Board: V12.06 Designed by AC8GY/K9HZ Layout by KI3P 4 layer, 2024/04/08"

Commit message: Added ground pad hole for digital attenuators on RF board
Routing:
- net /TC2: track 128.5 -> 129.4 mm
- net /TC8: track 132.0 -> 132.7 mm
- net /RC16: track 55.4 -> 55.9 mm
Other:
- board text added: "T41 RF Board: V12.06 Designed by AC8GY/K9HZ Layout by KI3P 4 layer, 2024/08/07"
- board text removed: "T41 RF Board: V12.06 Designed by AC8GY/K9HZ Layout by KI3P 4 layer, 2024/06/30"
