File: T41_V012_Files_01-15-24/T41_V012_KiCad/T41-RF-board-V012/T41-RF-board-V012_WJS.kicad_sch (KiCad schematic)
At the start: 219 parts, among them J1 IQ_Out, J2 RF_IN, J3 RFControl, J4 12-13.8V, J5 IQ_In, J6 RF_OUT, Q1 BS170, U1 74CBTLV3253DR, U10 SN74LVC1G04DCK, U106 AD8599, U107 OPA2209, U11 Si5351A-B-GT, U12 PE4312, U13 MAR-3SM+, U14 LM7805CT, U15 LM1117T-3.3, U16 LM358B, U17 LM317L, U2 PSA-8A+, U21 MCP23017_SO, U3 PE4312, U4 74CBTLV3253DR, U5 SN74LVC1G04DCK, U6 MC33078, U7 MASWSS0179, U8 MC33078, U9 MASWSS0179, Y1 ECS-TX053-S3, Y2 25MHz

Commit message: Update Boards
Update Boards
Parts:
- removed C74: 0.1uF 50V, Capacitor_SMD:C_1206_3216Metric, symbol Device:C
- JP1: value SolderJumper_2_Bridged -> SolderJumper_2_Open; footprint Jumper:SolderJumper-2_P1.3mm_Bridged_TrianglePad1.0x1.5mm -> Jumper:SolderJumper-2_P1.3mm_Open_TrianglePad1.0x1.5mm; symbol Jumper:SolderJumper_2_Bridged -> Jumper:SolderJumper_2_Open
- JP2: value SolderJumper_2_Open -> SolderJumper_2_Bridged; footprint Jumper:SolderJumper-2_P1.3mm_Open_RoundedPad1.0x1.5mm -> Jumper:SolderJumper-2_P1.3mm_Bridged_RoundedPad1.0x1.5mm; symbol Jumper:SolderJumper_2_Open -> Jumper:SolderJumper_2_Bridged; now in the parts list
- U106: value AD8599 -> MC33078
- U107: value OPA2209 -> MC33078
Other:
- note added: "Select 5V if needed for large signal operation."
- note removed: "Optional 3.3V Tap"
- moved on the sheet: JP1
Changed lines of the file:
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@@
 	)
 	(junction
-		(at 363.22 137.16)
-		(diameter 0)
-		(color 0 0 0 0)
-	)
-	(junction
 		(at 172.72 275.59)
 		(diameter 0)
@@
 	(wire
 		(pts
-			(xy 370.84 134.62) (xy 373.38 134.62)
-		)
-		(stroke
-			(width 0)
-			(type default)
-		)
-	)
-	(wire
-		(pts
 			(xy 289.56 109.22) (xy 289.56 114.3)
 		)
@@
 	(wire
 		(pts
-			(xy 363.22 137.16) (xy 370.84 137.16)
-		)
-		(stroke
-			(width 0)
-			(type default)
-		)
-	)
-	(wire
-		(pts
 			(xy 106.68 205.74) (xy 109.22 205.74)
 		)
@@
 	(wire
 		(pts
-			(xy 361.95 137.16) (xy 363.22 137.16)
+			(xy 361.95 137.16) (xy 370.84 137.16)
 		)
 		(stroke
@@
 	(wire
 		(pts
-			(xy 363.22 134.62) (xy 363.22 137.16)
-		)
-		(stroke
-			(width 0)
-			(type default)
-		)
-	)
-	(wire
-		(pts
 			(xy 341.63 29.21) (xy 341.63 41.91)
 		)
@@
 	(wire
 		(pts
-			(xy 373.38 134.62) (xy 373.38 135.89)
-		)
-		(stroke
-			(width 0)
-			(type default)
-		)
-	)
-	(wire
-		(pts
 			(xy 280.67 44.45) (xy 300.99 44.45)
 		)
@@
 		)
 	)
-	(text "Optional 3.3V Tap"
+	(text "Select 5V if needed for large \nsignal operation."
 		(exclude_from_sim no)
 		(at 171.45 46.99 0)
@@
 			)
 		)
-		(property "Value" "AD8599"
+		(property "Value" "MC33078"
 			(at 271.78 51.2501 0)
 			(effects
@@
 			)
 		)
-		(property "Value" "OPA2209"
+		(property "Value" "MC33078"
 			(at 332.74 96.9701 0)
 			(effects
@@
 	(symbol
 		(lib_id "power:GND")
+		(at 240.03 173.99 0)
+		(unit 1)
+		(exclude_from_sim no)
+		(in_bom yes)
+		(on_board yes)
+		(dnp no)
+		(property "Reference" "#PWR085"
+			(at 240.03 180.34 0)
+			(effects
+				(font
+					(size 1.27 1.27)
+				)
+				(hide yes)
+			)
+		)
+		(property "Value" "GND"
+			(at 242.57 175.26 90)
+			(effects
+				(font
+					(size 1.27 1.27)
+				)
+			)
+		)
+		(property "Footprint" ""
+			(at 240.03 173.99 0)
+			(effects
+				(font
+					(size 1.27 1.27)
+				)
+				(hide yes)
+			)
+		)
+		(property "Datasheet" ""
+			(at 240.03 173.99 0)
+			(effects
+				(font
+					(size 1.27 1.27)
+				)
+				(hide yes)
+			)
+		)
+		(property "Description" ""
+			(at 240.03 173.99 0)
+			(effects
+				(font
+					(size 1.27 1.27)
+				)
+				(hide yes)
+			)
+		)
+		(pin "1"
+		)
+		(instances
+			(project "T41-RF-board-V012"
+				(path "/3c4b9d3b-a516-4fd7-b325-b74c836dee65"
+					(reference "#PWR085")
+					(unit 1)
+				)
+			)
+		)
+	)
+	(symbol
+		(lib_id "power:GND")
 		(at 140.97 91.44 0)
 		(unit 1)
@@
 	)
 	(symbol
-		(lib_id "Jumper:SolderJumper_2_Bridged")
+		(lib_id "Jumper:SolderJumper_2_Open")
 		(at 177.8 58.42 90)
 		(unit 1)
-		(exclude_from_sim yes)
+		(exclude_from_sim no)
 		(in_bom no)
 		(on_board yes)
 		(dnp no)
+		(fields_autoplaced yes)
 		(property "Reference" "JP1"
-			(at 171.196 58.42 90)
+			(at 180.34 58.42 90)
 			(effects
 				(font
@@
 			)
 		)
-		(property "Value" "SolderJumper_2_Bridged"
+		(property "Value" "SolderJumper_2_Open"
 			(at 175.1909 58.42 0)
 			(effects
@@
 			)
 		)
-		(property "Footprint" "Jumper:SolderJumper-2_P1.3mm_Bridged_TrianglePad1.0x1.5mm"
+		(property "Footprint" "Jumper:SolderJumper-2_P1.3mm_Open_TrianglePad1.0x1.5mm"
 			(at 177.8 58.42 0)
 			(effects
@@
 			)
 		)
-		(property "Description" "Solder Jumper, 2-pole, closed"
+		(property "Description" ""
 			(at 177.8 58.42 0)
 			(effects
@@
 	)
 	(symbol
-		(lib_name "SolderJumper_2_Open_1")
-		(lib_id "Jumper:SolderJumper_2_Open")
+		(lib_id "Jumper:SolderJumper_2_Bridged")
 		(at 185.42 58.42 90)
 		(unit 1)
-		(exclude_from_sim yes)
-		(in_bom no)
+		(exclude_from_sim no)
+		(in_bom yes)
 		(on_board yes)
 		(dnp no)
 		(fields_autoplaced yes)
 		(property "Reference" "JP2"
-			(at 187.96 58.4199 90)
+			(at 187.96 57.15 90)
 			(effects
 				(font
@@
 			)
 		)
-		(property "Value" "SolderJumper_2_Open"
+		(property "Value" "SolderJumper_2_Bridged"
 			(at 187.96 59.69 90)
 			(effects
@@
 			)
 		)
-		(property "Footprint" "Jumper:SolderJumper-2_P1.3mm_Open_RoundedPad1.0x1.5mm"
+		(property "Footprint" "Jumper:SolderJumper-2_P1.3mm_Bridged_RoundedPad1.0x1.5mm"
 			(at 185.42 58.42 0)
 			(effects
@@
 			)
 		)
-		(property "Description" "Solder Jumper, 2-pole, open"
+		(property "Description" ""
 			(at 185.42 58.42 0)
 			(effects
@@
 	)
 	(symbol
-		(lib_id "Device:C")
-		(at 367.03 134.62 90)
-		(unit 1)
-		(exclude_from_sim no)
-		(in_bom yes)
-		(on_board yes)
-		(dnp no)
-		(property "Reference" "C74"
-			(at 361.95 133.35 90)
-			(effects
-				(font
-					(size 1.27 1.27)
-				)
-				(justify right)
-			)
-		)
-		(property "Value" "0.1uF 50V"
-			(at 369.57 133.35 90)
-			(effects
-				(font
-					(size 1.27 1.27)
-				)
-				(justify right)
-			)
-		)
-		(property "Footprint" "Capacitor_SMD:C_1206_3216Metric"
-			(at 370.84 133.6548 0)
-			(effects
-				(font
-					(size 1.27 1.27)
-				)
-				(hide yes)
-			)
-		)
-		(property "Datasheet" "~"
-			(at 367.03 134.62 0)
-			(effects
-				(font
-					(size 1.27 1.27)
-				)
-				(hide yes)
-			)
-		)
-		(property "Description" ""
-			(at 367.03 134.62 0)
-			(effects
-				(font
-					(size 1.27 1.27)
-				)
-				(hide yes)
-			)
-		)
-		(property "Mouser Part Number" ""
-			(at 367.03 134.62 0)
-			(effects
-				(font
-					(size 1.27 1.27)
-				)
-				(hide yes)
-			)
-		)
-		(pin "2"
-		)
-		(pin "1"
-		)
-		(instances
-			(project "T41-RF-board-V012"
-				(path "/3c4b9d3b-a516-4fd7-b325-b74c836dee65"
-					(reference "C74")
-					(unit 1)
-				)
-			)
-		)
-	)
-	(symbol
 		(lib_id "Device:L")
 		(at 171.45 191.77 0)
@@
 			)
 		)
-		(property "Value" "AD8599"
+		(property "Value" "MC33078"
 			(at 270.51 99.5101 0)
 			(effects
@@
 			)
 		)
-		(property "Value" "OPA2209"
+		(property "Value" "MC33078"
 			(at 335.28 64.4469 90)
 			(effects
@@
 			)
 		)
-		(property "Value" "AD8599"
+		(property "Value" "MC33078"
 			(at 275.59 73.3369 90)
 			(effects
@@
 	)
 	(symbol
-		(lib_id "power:GND")
-		(at 373.38 135.89 0)
-		(unit 1)
-		(exclude_from_sim no)
-		(in_bom yes)
-		(on_board yes)
-		(dnp no)
-		(property "Reference" "#PWR058"
-			(at 373.38 142.24 0)
-			(effects
-				(font
-					(size 1.27 1.27)
-				)
-				(hide yes)
-			)
-		)
-		(property "Value" "GND"
-			(at 375.92 137.16 90)
-			(effects
-				(font
-					(size 1.27 1.27)
-				)
-			)
-		)
-		(property "Footprint" ""
-			(at 373.38 135.89 0)
-			(effects
-				(font
-					(size 1.27 1.27)
-				)
-				(hide yes)
-			)
-		)
-		(property "Datasheet" ""
-			(at 373.38 135.89 0)
-			(effects
-				(font
-					(size 1.27 1.27)
-				)
-				(hide yes)
-			)
-		)
-		(property "Description" ""
-			(at 373.38 135.89 0)
-			(effects
-				(font
-					(size 1.27 1.27)
-				)
-				(hide yes)
-			)
-		)
-		(pin "1"
-		)
-		(instances
-			(project "T41-RF-board-V012"
-				(path "/3c4b9d3b-a516-4fd7-b325-b74c836dee65"
-					(reference "#PWR058")
-					(unit 1)
-				)
-			)
-		)
-	)
-	(symbol
 		(lib_id "Connector:TestPoint")
 		(at 67.31 102.87 0)
@@
 			)
 		)
-		(property "Value" "OPA2209"
+		(property "Value" "MC33078"
 			(at 332.74 48.7101 0)
 			(effects
