File: K9HZ_LFP_Module/K9HZ_LPF_V1.00_KiCad/K9HZ_100W_11band_LPF-Control/K9HZ_100W_11band_LPF-Control.kicad_sch (KiCad schematic)
At the start: 156 parts, among them J1 LPF ACC Control, J10 FROM 100W PA, J11 ANT-1, J12 ANT-2, J13 ANT-3, J14 ANT-4, J15 TO BPF, J16 TO LPF, J16.1 ANTENNA, J16.2 TRANSMIT, J17.1 RECEIVE, J17.2 TR CTL, J18 FROM BPF, J19 KEY OUT, J2 TO_RECEIVER, J20 12-13.8V, J21 Bands, J23 FROM LPF, J24 LPF CTRL HI, J25 LPF CTRL LOW, J3 FROM TX, J4 TO ATTN, J5 FROM ATTN, J6 TO XVTR, J7 TO 20W PA, J8 FROM 20W PA, J9 TO 100W PA, K2 HF41F/12-ZS, K3 HF41F/12-ZS, K4 HF41F/12-ZS, K5 HF41F/12-ZS, K6 HF41F/12-ZS, K7 HF41F/12-ZS, Q1 IRF630, Q2 2N7000, U1 MASWSS0179, U10 ULN2803, U11 LM7805CT, U12 CD74HC4514M96, U13 L7808, U14 AD8307, U15 MCP23017_SO, U16 LM1117T-3.3, U17 REF3440IDBVR, U18 TC4428, U19 AD8307, U2 74HC237, U20 AD7991YRJZ, U21 MASWSS0179, U22 SN74LVC1G04DCK, U3 MASWSS0179, U4 ULN2803, U5 SN74LVC1G04DCK, U6 SN74LVC1G04DCK, U7 MASWSS0179, U8 MASWSS0179, U9 ULN2803

Commit message: Recreate these
Parts:
- L38, L40, L42, L43: value 22uH -> 22nH; Mouser Part Number 70-ILSB1206ER220K -> (none)
- Q2: footprint Package_TO_SOT_THT:TO-92 -> Package_TO_SOT_THT:TO-92_Inline; symbol Transistor_FET:2N7002 -> Transistor_FET:2N7000
Connections:
- net 8R ~{TX}: now also Q2.2 (G); no longer Q2.1 (G)
- net GND: now also Q2.1 (S); no longer Q2.2 (S)
Other:
- note added: "20W: N = 10 100W: N = 20 R17,R22 = 498 Ohms R16,R18,R24,R25 = 55.2 Ohms"
- note removed: "20W: N = 9 100W: N = 20 R17,R22 = 498 Ohms R16,R18,R24,R25 = 55.2 Ohms"
Changed lines of the file:
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@@
   (title_block
     (title "K9HZ 100W 11 Band LPF: Control board")
-    (date "2024-01-14")
+    (date "2024-02-14")
     (rev "V1.00")
     (comment 1 "Layout by OG King-KI3P")
@@
     (effects (font (size 1.27 1.27)) (justify left bottom))
   )
-  (text "20W: N = 9\n100W: N = 20\nR17,R22 = 498 Ohms\nR16,R18,R24,R25 = 55.2 Ohms"
+  (text "20W: N = 10\n100W: N = 20\nR17,R22 = 498 Ohms\nR16,R18,R24,R25 = 55.2 Ohms"
     (at 365.76 180.34 0)
     (effects (font (size 1.27 1.27)) (justify left bottom))
@@
       (effects (font (size 1.27 1.27)) (justify left))
     )
-    (property "Value" "22uH" (at 231.1373 238.7021 0)
+    (property "Value" "22nH" (at 231.1373 238.7021 0)
       (effects (font (size 1.27 1.27)) (justify left))
     )
@@
       (effects (font (size 1.27 1.27)) hide)
     )
-    (property "Mouser Part Number" "70-ILSB1206ER220K" (at 229.87 237.49 0)
+    (property "Mouser Part Number" "" (at 229.87 237.49 0)
       (effects (font (size 1.27 1.27)) hide)
     )
@@
       (effects (font (size 1.27 1.27)) (justify left))
     )
-    (property "Value" "22uH" (at 231.1372 195.5221 0)
+    (property "Value" "22nH" (at 231.1372 195.5221 0)
       (effects (font (size 1.27 1.27)) (justify left))
     )
@@
       (effects (font (size 1.27 1.27)) hide)
     )
-    (property "Mouser Part Number" "70-ILSB1206ER220K" (at 229.87 194.31 0)
+    (property "Mouser Part Number" "" (at 229.87 194.31 0)
       (effects (font (size 1.27 1.27)) hide)
     )
@@
       (effects (font (size 1.27 1.27)) (justify left))
     )
-    (property "Value" "22uH" (at 223.5172 195.5221 0)
+    (property "Value" "22nH" (at 223.5172 195.5221 0)
       (effects (font (size 1.27 1.27)) (justify left))
     )
@@
       (effects (font (size 1.27 1.27)) hide)
     )
-    (property "Mouser Part Number" "70-ILSB1206ER220K" (at 222.25 194.31 0)
+    (property "Mouser Part Number" "" (at 222.25 194.31 0)
       (effects (font (size 1.27 1.27)) hide)
     )
@@
     )
   )
-  (symbol (lib_id "Transistor_FET:2N7002") (at 321.31 129.54 0) (unit 1)
+  (symbol (lib_id "Transistor_FET:2N7000") (at 321.31 129.54 0) (unit 1)
     (in_bom yes) (on_board yes) (dnp no)
     (property "Reference" "Q2" (at 326.517 128.3279 0)
@@
       (effects (font (size 1.27 1.27)) (justify left))
     )
-    (property "Footprint" "Package_TO_SOT_THT:TO-92" (at 326.39 131.445 0)
+    (property "Footprint" "Package_TO_SOT_THT:TO-92_Inline" (at 326.39 131.445 0)
       (effects (font (size 1.27 1.27) italic) (justify left) hide)
     )
-    (property "Datasheet" "https://www.onsemi.com/pub/Collateral/NDS7002A-D.PDF" (at 326.39 133.35 0)
+    (property "Datasheet" "https://www.vishay.com/docs/70226/70226.pdf" (at 326.39 133.35 0)
       (effects (font (size 1.27 1.27)) (justify left) hide)
     )
@@
       (effects (font (size 1.27 1.27)) (justify left))
     )
-    (property "Value" "22uH" (at 223.5173 238.7021 0)
+    (property "Value" "22nH" (at 223.5173 238.7021 0)
       (effects (font (size 1.27 1.27)) (justify left))
     )
@@
       (effects (font (size 1.27 1.27)) hide)
     )
-    (property "Mouser Part Number" "70-ILSB1206ER220K" (at 222.25 237.49 0)
+    (property "Mouser Part Number" "" (at 222.25 237.49 0)
       (effects (font (size 1.27 1.27)) hide)
     )
