File: K9HZ_LFP_Module/K9HZ_LPF_V1.00_KiCad/K9HZ_100W_11band_LPF-Control/K9HZ_100W_11band_LPF-Control.kicad_sch (KiCad schematic)
At the start: 156 parts, among them J1 LPF ACC Control, J10 FROM 100W PA, J11 ANT-1, J12 ANT-2, J13 ANT-3, J14 ANT-4, J15 TO BPF, J16 TO LPF, J16.1 ANTENNA, J16.2 TRANSMIT, J17.1 RECEIVE, J17.2 TR CTL, J18 FROM BPF, J19 KEY OUT, J2 TO_RECEIVER, J20 12-13.8V, J21 Bands, J23 FROM LPF, J24 LPF CTRL HI, J25 LPF CTRL LOW, J3 FROM TX, J4 TO ATTN, J5 FROM ATTN, J6 TO XVTR, J7 TO 20W PA, J8 FROM 20W PA, J9 TO 100W PA, K2 HF41F/12-ZS, K3 HF41F/12-ZS, K4 HF41F/12-ZS, K5 HF41F/12-ZS, K6 HF41F/12-ZS, K7 HF41F/12-ZS, Q1 IRF630, Q2 2N7000, U1 MASWSS0179, U10 ULN2803, U11 LM7805CT, U12 CD74HC4514M96, U13 L7808, U14 AD8307, U15 MCP23017_SO, U16 LM1117T-3.3, U17 REF3440IDBVR, U18 TC4428, U19 AD8307, U2 74HC237, U20 AD7991YRJZ, U21 MASWSS0179, U22 SN74LVC1G04DCK, U3 MASWSS0179, U4 ULN2803, U5 SN74LVC1G04DCK, U6 SN74LVC1G04DCK, U7 MASWSS0179, U8 MASWSS0179, U9 ULN2803

Commit message: Fixes to LPF as part of checkout
Parts:
- removed C9: 0.1uF 50V, Capacitor_SMD:C_1206_3216Metric, symbol Device:C
- removed U10, U4, U9: ULN2803, Package_SO:SOIC-20W_7.5x12.8mm_P1.27mm, symbol Transistor_Array:ULN2803A
- added U10, U4, U9: ULN2803C, Package_SO:SOIC-20W_7.5x12.8mm_P1.27mm, symbol T41_Library:ULN2803C
Connections:
- net +12V: now also U10.12 (COM), U4.12 (COM), U9.12 (COM)
- net 100W_PA_SEL: now also U4.16 (O5)
- net 10M: now also U10.17 (O4)
- net 12M: now also U10.18 (O3)
- net 15M: now also U10.19 (O2)
- net 160M: now also U9.20 (O1)
- net 17M: now also U10.20 (O1)
- net 20M: now also U9.15 (O6)
- net 30M: now also U9.16 (O5)
- net 40M: now also U9.17 (O4)
- net 60M: now also U9.18 (O3)
- net 6M: now also U10.16 (O5)
- net 80M: now also U9.19 (O2)
- net ANT1_SEL: now also U4.20 (O1)
- net ANT2_SEL: now also U4.19 (O2)
- net ANT3_SEL: now also U4.18 (O3)
- net ANT4_SEL: now also U4.17 (O4)
- net GND: now also U10.7 (I7), U10.8 (I8), U10.9 (GND), U4.6 (I6), U4.7 (I7), U4.8 (I8), U4.9 (GND), U9.7 (I7), U9.8 (I8), U9.9 (GND)
- net NF: now also U10.15 (O6)
- net XVTR_SEL: now also J1.3 (Pin_3), U15.7 (GPB6)
- net at U12.9 (Y1): now also U9.1 (I1)
- net at U12.10 (Y2): now also U9.2 (I2)
- net at U12.11 (Y0): now also U9.3 (I3)
- net at U12.8 (Y3): now also U9.4 (I4)
- net at U12.7 (Y4): now also U9.5 (I5)
- net at U12.6 (Y5): now also U9.6 (I6)
- net at U2.12 (Y3): now also U4.4 (I4)
- net at U2.13 (Y2): now also U4.3 (I3)
- net at U2.14 (Y1): now also U4.2 (I2)
- net at U2.15 (Y0): now also U4.1 (I1)
- net at J1.4 (Pin_4), U15.8 (GPB7): now also U4.5 (I5)
- net at U12.15 (Y15): now also U10.6 (I6)
- net at U12.17 (Y9): now also U10.4 (I4)
- net at U12.18 (Y8): now also U10.3 (I3)
- net at U12.20 (Y10): now also U10.5 (I5)
- net at U12.4 (Y7): now also U10.2 (I2)
- net at U12.5 (Y6): now also U10.1 (I1)
- no-connect marks 36 -> 43
Other:
- note added: "20W: N = 9 100W: N = 20 26 dB attenuation: R17,R22 = 498 Ohms R16,R18,R24,R25 = 55.2 Ohms"
- note removed: "20W: N = 9 100W: N = 20 R17,R22 = 498 Ohms R16,R18,R24,R25 = 55.2 Ohms"
- moved on the sheet: C11, C129

Commit message: Fixes to LPF control board based on KI3P testing
Parts:
- L38, L40, L42, L43: value 22uH -> 22nH; Mouser Part Number 70-ILSB1206ER220K -> (none)
- Q2: footprint Package_TO_SOT_THT:TO-92 -> Package_TO_SOT_THT:TO-92_Inline; symbol Transistor_FET:2N7002 -> Transistor_FET:2N7000
Connections:
- net 8R ~{TX}: now also Q2.2 (G); no longer Q2.1 (G)
- net GND: now also Q2.1 (S); no longer Q2.2 (S)
Other:
- note added: "20W: N = 10 100W: N = 20 26 dB attenuation: R17,R22 = 498 Ohms R16,R18,R24,R25 = 55.2 Ohms"
- note removed: "20W: N = 9 100W: N = 20 26 dB attenuation: R17,R22 = 498 Ohms R16,R18,R24,R25 = 55.2 Ohms"
Changed lines of the file:
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@@
   (title_block
     (title "K9HZ 100W 11 Band LPF: Control board")
-    (date "2024-02-11")
+    (date "2024-02-14")
     (rev "V1.1")
     (comment 1 "Layout by OG King-KI3P")
@@
     (effects (font (size 1.27 1.27)) (justify left bottom))
   )
-  (text "20W: N = 9\n100W: N = 20\n26 dB attenuation:\n    R17,R22 = 498 Ohms\n    R16,R18,R24,R25 = 55.2 Ohms"
+  (text "20W: N = 10\n100W: N = 20\n26 dB attenuation:\n    R17,R22 = 498 Ohms\n    R16,R18,R24,R25 = 55.2 Ohms"
     (at 365.76 180.34 0)
     (effects (font (size 1.27 1.27)) (justify left bottom))
@@
       (effects (font (size 1.27 1.27)) (justify left))
     )
-    (property "Value" "22uH" (at 231.1373 238.7021 0)
+    (property "Value" "22nH" (at 231.1373 238.7021 0)
       (effects (font (size 1.27 1.27)) (justify left))
     )
@@
       (effects (font (size 1.27 1.27)) hide)
     )
-    (property "Mouser Part Number" "70-ILSB1206ER220K" (at 229.87 237.49 0)
+    (property "Mouser Part Number" "" (at 229.87 237.49 0)
       (effects (font (size 1.27 1.27)) hide)
     )
@@
       (effects (font (size 1.27 1.27)) (justify left))
     )
-    (property "Value" "22uH" (at 231.1372 195.5221 0)
+    (property "Value" "22nH" (at 231.1372 195.5221 0)
       (effects (font (size 1.27 1.27)) (justify left))
     )
@@
       (effects (font (size 1.27 1.27)) hide)
     )
-    (property "Mouser Part Number" "70-ILSB1206ER220K" (at 229.87 194.31 0)
+    (property "Mouser Part Number" "" (at 229.87 194.31 0)
       (effects (font (size 1.27 1.27)) hide)
     )
@@
       (effects (font (size 1.27 1.27)) (justify left))
     )
-    (property "Value" "22uH" (at 223.5172 195.5221 0)
+    (property "Value" "22nH" (at 223.5172 195.5221 0)
       (effects (font (size 1.27 1.27)) (justify left))
     )
@@
       (effects (font (size 1.27 1.27)) hide)
     )
-    (property "Mouser Part Number" "70-ILSB1206ER220K" (at 222.25 194.31 0)
+    (property "Mouser Part Number" "" (at 222.25 194.31 0)
       (effects (font (size 1.27 1.27)) hide)
     )
@@
     )
   )
-  (symbol (lib_id "Transistor_FET:2N7002") (at 321.31 129.54 0) (unit 1)
+  (symbol (lib_id "Transistor_FET:2N7000") (at 321.31 129.54 0) (unit 1)
     (in_bom yes) (on_board yes) (dnp no)
     (property "Reference" "Q2" (at 326.517 128.3279 0)
@@
       (effects (font (size 1.27 1.27)) (justify left))
     )
-    (property "Footprint" "Package_TO_SOT_THT:TO-92" (at 326.39 131.445 0)
+    (property "Footprint" "Package_TO_SOT_THT:TO-92_Inline" (at 326.39 131.445 0)
       (effects (font (size 1.27 1.27) italic) (justify left) hide)
     )
-    (property "Datasheet" "https://www.onsemi.com/pub/Collateral/NDS7002A-D.PDF" (at 326.39 133.35 0)
+    (property "Datasheet" "https://www.vishay.com/docs/70226/70226.pdf" (at 326.39 133.35 0)
       (effects (font (size 1.27 1.27)) (justify left) hide)
     )
@@
       (effects (font (size 1.27 1.27)) (justify left))
     )
-    (property "Value" "22uH" (at 223.5173 238.7021 0)
+    (property "Value" "22nH" (at 223.5173 238.7021 0)
       (effects (font (size 1.27 1.27)) (justify left))
     )
@@
       (effects (font (size 1.27 1.27)) hide)
     )
-    (property "Mouser Part Number" "70-ILSB1206ER220K" (at 222.25 237.49 0)
+    (property "Mouser Part Number" "" (at 222.25 237.49 0)
       (effects (font (size 1.27 1.27)) hide)
     )
