File: T41_V012_Files_01-15-24/T41_V012_KiCad/T41-main-board-V012/T41-main-board-V012.kicad_pcb (KiCad board)
At the start: 4 copper layers, 100 x 100 mm, 103 parts, among them J1 +12V, J10 Conn_01x02, J11 ENCODER, J12 BANDS, J13 Header, J14 Rec_Out, J15 Rec_In, J16 Mic_In, J17 Ex_Out, J18 Conn_01x02, J19 Conn_01x01, J2 Fan1, J20 Conn_01x01, J21 Conn_01x01, J22 Header, J23 Ethernet, J24 USBHost, J3 Acc, J4 12-13.8V, J5 Front Panel, J6 RF CONTROL, J7 Display, J8 Display Voltage, J9 Keys/PTT, Q1 IRF4905, Q2 2N7000, Q3 2N7000, SW1 ON-OFF BUTTON, U1 LM7805CT, U10 LM1117T-3.3, U2 AP7384-50V, U3 LM1117T-3.3, U4 ATtiny85-20S, U5 PCM5102, U6 PCM1808PW, U8 Teensy4.1, U9 LM7805CT

Commit message: Fixed incorrect grounding of heatsink feet on main board
Connections:
- H1 pad 1: GND -> (no net)
- H2 pad 1: GND -> (no net)
- H3 pad 1: GND -> (no net)
- H4 pad 1: GND -> (no net)
Other:
- board text added: "T41 Main+, V012.6 Design by AC8GY/W8TEE/K9HZ KiCad Layout by KI3P 4 layer, 2024-02-03"
- board text removed: "T41 Main+, V012.6 Design by AC8GY/W8TEE/K9HZ KiCad Layout by KI3P 4 layer, 2024-01-14"

Commit message: Moved heatsink up slightly on main board to avoid board edge
Parts:
- moved H1 0.76 mm to (98.6, 119.6)
- moved H2 0.76 mm to (98.6, 145.0)
- moved U1 0.76 mm to (102.0, 134.9)
- moved U9 0.76 mm to (95.2, 134.9)
Routing:
- net +12V: track 167.3 -> 162.7 mm
- net /BAND1 (40m): vias 0 -> 1
- net /BAND0 (80m): vias 0 -> 1

Commit message: Changed Q1 of main board to correct part FQP47P06
Parts:
- Q1: value IRF4905 -> FQP47P06
Changed lines of the file:
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@@
     (descr "TO-220-3, Vertical, RM 2.54mm, see https://www.vishay.com/docs/66542/to-220-1.pdf")
     (tags "TO-220-3 Vertical RM 2.54mm")
-    (property "Mouser" "942-IRF4905PBF")
+    (property "Mouser" "")
     (property "PJRC.com" "")
     (property "Sheetfile" "T41-main-board-V012.kicad_sch")
@@
         (effects (font (size 1 1) (thickness 0.15)))
     )
-    (fp_text value "IRF4905" (at 2.54 2.5 90) (layer "F.Fab")
+    (fp_text value "FQP47P06" (at 2.54 2.5 90) (layer "F.Fab")
         (effects (font (size 1 1) (thickness 0.15)))
     )
