File: T41_V012_Files_01-15-24/T41_V012_KiCad/T41-main-board-V012/T41-main-board-V012.kicad_pcb (KiCad board)
At the start: 4 copper layers, 100 x 100 mm, 103 parts, among them J1 +12V, J10 Conn_01x02, J11 ENCODER, J12 BANDS, J13 Header, J14 Rec_Out, J15 Rec_In, J16 Mic_In, J17 Ex_Out, J18 Conn_01x02, J19 Conn_01x01, J2 Fan1, J20 Conn_01x01, J21 Conn_01x01, J22 Header, J23 Ethernet, J24 USBHost, J3 Acc, J4 12-13.8V, J5 Front Panel, J6 RF CONTROL, J7 Display, J8 Display Voltage, J9 Keys/PTT, Q1 FQP47P06, Q2 2N7000, Q3 2N7000, SW1 ON-OFF BUTTON, U1 LM7805CT, U10 LM1117T-3.3, U2 AP7384-50V, U3 LM1117T-3.3, U4 ATtiny85-20S, U5 PCM5102, U6 PCM1808PW, U8 Teensy4.1, U9 LM7805CT

Commit message: Changed orientation of Q1 and D5 for reverse protection
Parts:
- removed H1, H2, H3, H4: ~, MountingHole:MountingHole_3mm_Pad
- added H7: EA-T220-38E, T41_Library:EAT22038E, F.Cu at (98.6, 145.0)
- added H8: EA-T220-38E, T41_Library:EAT22038E, F.Cu at (127.3, 145.0)
- Q1: value FQP47P06 -> SUP90P06-09L
Connections:
- D5 pad 1: Net-(D1-A) -> +12V
- Q1 pad 2: +12V -> Net-(D1-A)
- Q1 pad 3: Net-(D1-A) -> +12V
Routing:
- net +12V: track 162.7 -> 170.1 mm, vias 0 -> 1
- net Net-(D1-A): track 28.1 -> 23.7 mm, vias 1 -> 0
Other:
- board text added: "T41 Main+, V012.6 Design by AC8GY/W8TEE/K9HZ KiCad Layout by KI3P 4 layer, 2024-02-26"
- board text removed: "T41 Main+, V012.6 Design by AC8GY/W8TEE/K9HZ KiCad Layout by KI3P 4 layer, 2024-02-03"

Commit message: Incorporate final QC changes from Bill: add altenative MOSFET switch footprint for voltage reversal protection
Parts:
- added Q4: SUP90P06-09L, Package_TO_SOT_THT:TO-220-3_Vertical, F.Cu at (74.7, 138.6)
- Q1: moved to B.Cu
- moved Q1 9.87 mm to (69.8, 130.9), turned to -90 degrees
- moved L2 1.32 mm to (65.2, 133.3)
- moved C2 0.25 mm to (118.6, 143.8)
Routing:
- net Net-(D5-A): track 26.6 -> 48.8 mm, vias 0 -> 1
- net Net-(D1-A): track 23.7 -> 20.3 mm
- net +12V: track 170.1 -> 168.0 mm, vias 1 -> 0
- net +12P: track 8.59 -> 7.28 mm
Other:
- board text added: "12V OUT"
- board text added: "T41 Main+, V012.6 Design by AC8GY/W8TEE/K9HZ KiCad Layout by KI3P 4 layer, 2024-04-26"
- board text removed: "T41 Main+, V012.6 Design by AC8GY/W8TEE/K9HZ KiCad Layout by KI3P 4 layer, 2024-02-26"
