File: T41_V012_Files_01-15-24/T41_V012_KiCad/T41-main-board-V012/T41-main-board-V012.kicad_sch (KiCad schematic)
At the start: 105 parts, among them J1 +12V, J10 Conn_01x02, J11 ENCODER, J12 BANDS, J13 Header, J14 Rec_Out, J15 Rec_In, J16 Mic_In, J17 Ex_Out, J18 Conn_01x02, J19 Conn_01x01, J2 Fan1, J20 Conn_01x01, J21 Conn_01x01, J22 Header, J23 Ethernet, J24 USBHost, J3 Acc, J4 12-13.8V, J5 Front Panel, J6 RF CONTROL, J7 Display, J8 Display Voltage, J9 Keys/PTT, M1 Fan, Q1 IRF4905, Q2 2N7000, Q3 2N7000, SW1 ON-OFF BUTTON, U1 LM7805CT, U10 LM1117T-3.3, U2 AP7384-50V, U3 LM1117T-3.3, U4 ATtiny85-20S, U5 PCM5102, U6 PCM1808PW, U7 Teensy_Audio_Adaptor, U8 Teensy4.1, U9 LM7805CT

Commit message: Fixed incorrect grounding of heatsink feet on main board
Parts:
- H1, H2, H3, H4: symbol Mechanical:MountingHole_Pad -> Mechanical:MountingHole; now in the parts list
Connections:
- net GND: no longer H1.1, H2.1, H3.1, H4.1
Changed lines of the file:
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@@
   (title_block
     (title "T41 Main Board")
-    (date "2024-01-14")
+    (date "2024-02-03")
     (rev "V012.6")
     (comment 1 "         Transcribed to KiCAD by OG King-KI3P")
@@
   (junction (at 205.74 209.55) (diameter 0) (color 0 0 0 0)
   )
-  (junction (at 361.95 43.18) (diameter 0) (color 0 0 0 0)
-  )
   (junction (at 236.22 240.03) (diameter 0) (color 0 0 0 0)
   )
@@
   (junction (at 222.25 251.46) (diameter 0) (color 0 0 0 0)
   )
-  (junction (at 363.22 43.18) (diameter 0) (color 0 0 0 0)
-  )
   (junction (at 50.8 236.22) (diameter 0) (color 0 0 0 0)
   )
@@
   (junction (at 82.55 238.76) (diameter 0) (color 0 0 0 0)
   )
-  (junction (at 361.95 38.1) (diameter 0) (color 0 0 0 0)
-  )
   (junction (at 82.55 53.34) (diameter 0) (color 0 0 0 0)
   )
@@
     (stroke (width 0) (type default))
   )
-  (wire (pts (xy 363.22 43.18) (xy 364.49 43.18))
-    (stroke (width 0) (type default))
-  )
   (wire (pts (xy 222.25 20.32) (xy 222.25 38.1))
     (stroke (width 0) (type default))
@@
     (stroke (width 0) (type default))
   )
-  (wire (pts (xy 361.95 43.18) (xy 363.22 43.18))
-    (stroke (width 0) (type default))
-  )
   (wire (pts (xy 41.91 161.29) (xy 38.1 161.29))
     (stroke (width 0) (type default))
@@
     (stroke (width 0) (type default))
   )
-  (wire (pts (xy 361.95 38.1) (xy 361.95 43.18))
-    (stroke (width 0) (type default))
-  )
   (wire (pts (xy 43.18 111.76) (xy 39.37 111.76))
     (stroke (width 0) (type default))
@@
     (stroke (width 0) (type default))
   )
-  (wire (pts (xy 361.95 38.1) (xy 364.49 38.1))
-    (stroke (width 0) (type default))
-  )
   (wire (pts (xy 138.43 54.61) (xy 140.97 54.61))
     (stroke (width 0) (type default))
@@
     )
   )
-  (symbol (lib_id "Mechanical:MountingHole_Pad") (at 359.41 43.18 90) (unit 1)
-    (in_bom no) (on_board yes) (dnp no)
+  (symbol (lib_id "Mechanical:MountingHole") (at 359.41 43.18 90) (unit 1)
+    (in_bom yes) (on_board yes) (dnp no)
     (property "Reference" "H2" (at 354.33 43.18 90)
       (effects (font (size 1.27 1.27)))
@@
       (effects (font (size 1.27 1.27)) hide)
     )
-    (pin "1")
     (instances
       (project "T41-main-board-V012"
@@
     )
   )
-  (symbol (lib_id "Mechanical:MountingHole_Pad") (at 367.03 43.18 270) (unit 1)
-    (in_bom no) (on_board yes) (dnp no) (fields_autoplaced)
-    (property "Reference" "H4" (at 370.84 43.18 90)
+  (symbol (lib_id "Mechanical:MountingHole") (at 367.03 43.18 270) (unit 1)
+    (in_bom yes) (on_board yes) (dnp no) (fields_autoplaced)
+    (property "Reference" "H4" (at 369.57 43.18 90)
       (effects (font (size 1.27 1.27)) (justify left))
     )
@@
       (effects (font (size 1.27 1.27)) hide)
     )
-    (pin "1")
     (instances
       (project "T41-main-board-V012"
@@
     )
   )
-  (symbol (lib_id "power:GND") (at 363.22 43.18 0) (unit 1)
-    (in_bom yes) (on_board yes) (dnp no) (fields_autoplaced)
-    (property "Reference" "#PWR069" (at 363.22 49.53 0)
-      (effects (font (size 1.27 1.27)) hide)
-    )
-    (property "Value" "GND" (at 363.22 47.3131 0)
-      (effects (font (size 1.27 1.27)))
-    )
-    (property "Footprint" "" (at 363.22 43.18 0)
-      (effects (font (size 1.27 1.27)) hide)
-    )
-    (property "Datasheet" "" (at 363.22 43.18 0)
-      (effects (font (size 1.27 1.27)) hide)
-    )
-    (pin "1")
-    (instances
-      (project "T41-main-board-V012"
-        (path "/3c4b9d3b-a516-4fd7-b325-b74c836dee65"
-          (reference "#PWR069") (unit 1)
-        )
-      )
-    )
-  )
   (symbol (lib_id "Connector_Generic:Conn_01x02") (at 53.34 163.83 0) (mirror y) (unit 1)
     (in_bom yes) (on_board yes) (dnp no)
@@
     )
   )
-  (symbol (lib_id "Mechanical:MountingHole_Pad") (at 359.41 38.1 90) (unit 1)
-    (in_bom no) (on_board yes) (dnp no)
+  (symbol (lib_id "Mechanical:MountingHole") (at 359.41 38.1 90) (unit 1)
+    (in_bom yes) (on_board yes) (dnp no)
     (property "Reference" "H1" (at 354.33 38.1 90)
       (effects (font (size 1.27 1.27)))
@@
       (effects (font (size 1.27 1.27)) hide)
     )
-    (pin "1")
     (instances
       (project "T41-main-board-V012"
@@
     )
   )
-  (symbol (lib_id "Mechanical:MountingHole_Pad") (at 367.03 38.1 270) (unit 1)
-    (in_bom no) (on_board yes) (dnp no) (fields_autoplaced)
-    (property "Reference" "H3" (at 370.84 38.1 90)
+  (symbol (lib_id "Mechanical:MountingHole") (at 367.03 38.1 270) (unit 1)
+    (in_bom yes) (on_board yes) (dnp no) (fields_autoplaced)
+    (property "Reference" "H3" (at 369.57 38.1 90)
       (effects (font (size 1.27 1.27)) (justify left))
     )
@@
       (effects (font (size 1.27 1.27)) hide)
     )
-    (pin "1")
     (instances
       (project "T41-main-board-V012"

Commit message: Changed Q1 of main board to correct part FQP47P06
Parts:
- Q1: value IRF4905 -> FQP47P06; Mouser 942-IRF4905PBF -> (none)
Changed lines of the file:
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@@
   (title_block
     (title "T41 Main Board")
-    (date "2024-02-03")
+    (date "2024-02-17")
     (rev "V012.6")
     (comment 1 "         Transcribed to KiCAD by OG King-KI3P")
@@
       (effects (font (size 1.27 1.27)))
     )
-    (property "Value" "IRF4905" (at 184.15 45.72 90)
+    (property "Value" "FQP47P06" (at 184.15 45.72 90)
       (effects (font (size 1.27 1.27)))
     )
@@
       (effects (font (size 1.27 1.27) italic) (justify left) hide)
     )
-    (property "Datasheet" "http://www.infineon.com/dgdl/irf4905.pdf?fileId=5546d462533600a4015355e32165197c" (at 180.34 40.64 0)
+    (property "Datasheet" "https://www.onsemi.com/pdf/datasheet/fqp47p06-d.pdf" (at 180.34 40.64 0)
       (effects (font (size 1.27 1.27)) (justify left) hide)
     )
-    (property "Mouser" "942-IRF4905PBF" (at 180.34 40.64 0)
-      (effects (font (size 1.27 1.27)) hide)
-    )
+    (property "Mouser" "" (at 180.34 40.64 0)
+      (effects (font (size 1.27 1.27)) hide)
+    )

Commit message: Changed orientation of Q1 and D5 for reverse protection
Parts:
- removed H1, H2, H3, H4: ~, MountingHole:MountingHole_3mm_Pad, symbol Mechanical:MountingHole
- added H7, H8: EA-T220-38E, EAT22038E, symbol T41_Library:EA-T220-38E
- Q1: value FQP47P06 -> SUP90P06-09L
Connections:
- net +12V: now also D5.1 (K), Q1.3 (S); no longer Q1.2 (D)
- net at D1.2 (A), L2.1, R1.1: now also Q1.2 (D); no longer D5.1 (K), Q1.3 (S)
- no-connect marks 28 -> 32
Other:
- moved on the sheet: D5, Q1, R16

Commit message: Incorporate final QC changes from Bill: add altenative MOSFET switch footprint for voltage reversal protection
Parts:
- added Q4: SUP90P06-09L, Package_TO_SOT_THT:TO-220-3_Vertical, symbol Transistor_FET:IRF4905
- Q1: now not fitted
Connections:
- net +12V: now also Q4.2 (D)
- net at D5.2 (A), Q1.1 (G), Q2.2 (G)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: now also Q4.1 (G)
- net at D1.2 (A), L2.1, Q1.2 (D)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: now also Q4.3 (S)
Other:
- moved on the sheet: L2

Commit message: Added bypass capacitor to TCXO, removed clock divider circuit, replaced I/Q output DC blocking capacitors with 0R resistors
Other:
- note added: "If using 3V3, replace R4 and R5 with 0R?"
Changed lines of the file:
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@@
+		)
+	)
+	(text "If using 3V3, replace \nR4 and R5 with 0R?"
+		(exclude_from_sim no)
+		(at 200.66 172.974 0)
+		(effects
+			(font
+				(size 1.27 1.27)
+				(thickness 0.254)
+				(bold yes)
+				(color 255 0 0 1)
+			)
+			(justify left)
 		)
 	)
