File: T41_V012_Files_01-15-24/T41_V012_KiCad/T41-BPF-filter-board/T41-exciter-filter-board.kicad_pcb (KiCad board)
At the start: 2 copper layers, 100 x 100 mm, 197 parts, among them J1 TO PA, J2 FROM EXCITE, J3 12-13.8V, J4 Bands, J5 TO RECEIVE, J6 FROM LPF, U1 MASWSS0179, U10 MASWSS0179, U11 SN74LVC1G04DCK, U12 MASWSS0179, U13 MASWSS0179, U14 SN74LVC1G04DCK, U15 MASWSS0179, U16 MASWSS0179, U17 SN74LVC1G04DCK, U18 MASWSS0179, U19 MASWSS0179, U2 SN74LVC1G04DCK, U20 SN74LVC1G04DCK, U21 MASWSS0179, U22 LM1117T-3.3, U23 SN74LVC1G04DCK, U24 MASWSS0179, U25 MASWSS0179, U26 SN74LVC1G04DCK, U27 MASWSS0179, U28 MASWSS0179, U29 SN74LVC1G04DCK, U3 MASWSS0179, U30 MASWSS0179, U31 MASWSS0179, U35 MCP23017_SO, U36 MASWSS0179, U37 SN74LVC1G04DCK, U4 MASWSS0179, U5 SN74LVC1G04DCK, U6 MASWSS0179, U7 MASWSS0179, U8 SN74LVC1G04DCK, U9 MASWSS0179

Commit message: Added 1206 footprints alongside all the coil inductors in the BPF board to allow use of SMD inductors instead of toroids
Parts:
- added L10: L, Inductor_SMD:L_1206_3216Metric, F.Cu at (94.7, 110.8)
- added L11: L, Inductor_SMD:L_1206_3216Metric, F.Cu at (125.0, 110.8)
- added L12: L, Inductor_SMD:L_1206_3216Metric, F.Cu at (68.9, 118.9)
- added L13: L, Inductor_SMD:L_1206_3216Metric, F.Cu at (94.3, 118.9)
- added L14: L, Inductor_SMD:L_1206_3216Metric, F.Cu at (125.0, 118.9)
- added L15: L, Inductor_SMD:L_1206_3216Metric, F.Cu at (69.1, 127.0)
- added L16: L, Inductor_SMD:L_1206_3216Metric, F.Cu at (94.3, 127.0)
- added L17: L, Inductor_SMD:L_1206_3216Metric, F.Cu at (125.1, 127.0)
- added L18: L, Inductor_SMD:L_1206_3216Metric, F.Cu at (69.0, 135.2)
- added L19: L, Inductor_SMD:L_1206_3216Metric, F.Cu at (94.3, 135.3)
- added L20: L, Inductor_SMD:L_1206_3216Metric, F.Cu at (124.8, 135.2)
- added L21: L, Inductor_SMD:L_1206_3216Metric, F.Cu at (125.1, 53.1)
- added L22: L, Inductor_SMD:L_1206_3216Metric, F.Cu at (94.3, 53.1)
- added L23: L, Inductor_SMD:L_1206_3216Metric, F.Cu at (69.1, 53.2)
- added L24: L, Inductor_SMD:L_1206_3216Metric, F.Cu at (124.7, 69.4)
- added L25: L, Inductor_SMD:L_1206_3216Metric, F.Cu at (94.0, 69.4)
- added L26: L, Inductor_SMD:L_1206_3216Metric, F.Cu at (69.2, 69.4)
- added L27: L, Inductor_SMD:L_1206_3216Metric, F.Cu at (125.0, 85.6)
- added L28: L, Inductor_SMD:L_1206_3216Metric, F.Cu at (94.5, 85.6)
- added L29: L, Inductor_SMD:L_1206_3216Metric, F.Cu at (68.9, 85.6)
- added L3: L, Inductor_SMD:L_1206_3216Metric, F.Cu at (69.0, 61.3)
- added L30: L, Inductor_SMD:L_1206_3216Metric, F.Cu at (83.4, 61.3)
- added L31: L, Inductor_SMD:L_1206_3216Metric, F.Cu at (110.8, 61.3)
- added L32: L, Inductor_SMD:L_1206_3216Metric, F.Cu at (83.3, 77.5)
- added L33: L, Inductor_SMD:L_1206_3216Metric, F.Cu at (110.9, 77.6)
- added L34: L, Inductor_SMD:L_1206_3216Metric, F.Cu at (83.1, 110.8)
- added L35: L, Inductor_SMD:L_1206_3216Metric, F.Cu at (110.9, 110.7)
- added L36: L, Inductor_SMD:L_1206_3216Metric, F.Cu at (83.4, 118.9)
- added L37: L, Inductor_SMD:L_1206_3216Metric, F.Cu at (110.9, 118.9)
- added L38: L, Inductor_SMD:L_1206_3216Metric, F.Cu at (83.2, 127.0)
- added L39: L, Inductor_SMD:L_1206_3216Metric, F.Cu at (110.8, 127.0)
- added L4: L, Inductor_SMD:L_1206_3216Metric, F.Cu at (94.3, 61.3)
- added L40: L, Inductor_SMD:L_1206_3216Metric, F.Cu at (83.0, 135.1)
- added L41: L, Inductor_SMD:L_1206_3216Metric, F.Cu at (110.8, 135.1)
- added L42: L, Inductor_SMD:L_1206_3216Metric, F.Cu at (83.4, 53.1)
- added L43: L, Inductor_SMD:L_1206_3216Metric, F.Cu at (110.8, 53.1)
- added L44: L, Inductor_SMD:L_1206_3216Metric, F.Cu at (83.2, 69.4)
- added L45: L, Inductor_SMD:L_1206_3216Metric, F.Cu at (110.8, 69.4)
- added L46: L, Inductor_SMD:L_1206_3216Metric, F.Cu at (83.1, 85.6)
- added L47: L, Inductor_SMD:L_1206_3216Metric, F.Cu at (110.7, 85.6)
- added L5: L, Inductor_SMD:L_1206_3216Metric, F.Cu at (125.0, 61.3)
- added L6: L, Inductor_SMD:L_1206_3216Metric, F.Cu at (69.2, 77.5)
- added L7: L, Inductor_SMD:L_1206_3216Metric, F.Cu at (94.5, 77.6)
- added L8: L, Inductor_SMD:L_1206_3216Metric, F.Cu at (124.7, 77.6)
- added L9: L, Inductor_SMD:L_1206_3216Metric, F.Cu at (69.0, 110.7)
Routing:
- net /12/10m: track 114.4 -> 120.8 mm
- net /~{30m}: track 87.8 -> 92.6 mm, vias 2 -> 4
- net /RF54: track 22.4 -> 26.0 mm
- net /RF84: track 22.4 -> 26.0 mm
- net /RF24: track 22.4 -> 25.9 mm
- net /RF44: track 22.4 -> 25.9 mm
- net /RF74: track 22.4 -> 25.8 mm
- net /RF14: track 22.4 -> 25.7 mm
- net /RF86: track 24.3 -> 27.6 mm
- net /RF56: track 24.3 -> 27.6 mm
- net /RF34: track 22.4 -> 25.7 mm
- net /RF46: track 24.3 -> 27.5 mm
- net /RF66: track 24.3 -> 27.5 mm
- net /RF6: track 24.3 -> 27.5 mm
- net /RF64: track 22.4 -> 25.6 mm
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Other:
- board text added: "Design by AC8GY, KH9Z, layout by KI3P. 2024/02/03, V012.06"
- board text removed: "Design by AC8GY, KH9Z, layout by KI3P. 2024/01/26, V012.06"

Commit message: Corrected callsign for Bill on the BPF board silkscreen
Other:
- board text added: "Design by AC8GY, K9HZ, layout by KI3P. 2024/02/03, V012.06"
- board text removed: "Design by AC8GY, KH9Z, layout by KI3P. 2024/02/03, V012.06"
Changed lines of the file:
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@@
     (effects (font (size 1 1) (thickness 0.2) bold) (justify left bottom))
   )
-  (gr_text "Design by AC8GY, KH9Z, layout by KI3P. 2024/02/03, V012.06" (at 62.738 149.225) (layer "F.SilkS")
+  (gr_text "Design by AC8GY, K9HZ, layout by KI3P. 2024/02/03, V012.06" (at 62.738 149.225) (layer "F.SilkS")
     (effects (font (size 1.5 1.5) (thickness 0.3)) (justify left bottom))
   )

Commit message: Fixes to BPF board, adding missing decoupling capacitors
Parts:
- added C10: 0.1uF 50V, Capacitor_SMD:C_1206_3216Metric, F.Cu at (55.2, 77.3)
- added C11: 0.1uF 50V, Capacitor_SMD:C_1206_3216Metric, F.Cu at (55.1, 108.5)
- added C12: 0.1uF 50V, Capacitor_SMD:C_1206_3216Metric, F.Cu at (55.3, 117.6)
- added C13: 0.1uF 50V, Capacitor_SMD:C_1206_3216Metric, F.Cu at (55.1, 126.5)
- added C14: 0.1uF 50V, Capacitor_SMD:C_1206_3216Metric, F.Cu at (55.0, 134.7)
- added C15: 0.1uF 50V, Capacitor_SMD:C_1206_3216Metric, F.Cu at (142.9, 61.7)
- added C16: 0.1uF 50V, Capacitor_SMD:C_1206_3216Metric, F.Cu at (142.9, 77.9)
- added C17: 0.1uF 50V, Capacitor_SMD:C_1206_3216Metric, F.Cu at (142.7, 111.1)
- added C18: 0.1uF 50V, Capacitor_SMD:C_1206_3216Metric, F.Cu at (142.8, 119.2)
- added C19: 0.1uF 50V, Capacitor_SMD:C_1206_3216Metric, F.Cu at (142.8, 127.3)
- added C20: 0.1uF 50V, Capacitor_SMD:C_1206_3216Metric, F.Cu at (142.8, 135.2)
- added C21: 0.1uF 50V, Capacitor_SMD:C_1206_3216Metric, F.Cu at (54.9, 53.3)
- added C22: 0.1uF 50V, Capacitor_SMD:C_1206_3216Metric, F.Cu at (55.3, 69.1)
- added C23: 0.1uF 50V, Capacitor_SMD:C_1206_3216Metric, F.Cu at (55.5, 85.3)
- added C24: 0.1uF 50V, Capacitor_SMD:C_1206_3216Metric, F.Cu at (142.9, 53.5)
- added C25: 0.1uF 50V, Capacitor_SMD:C_1206_3216Metric, F.Cu at (142.9, 69.7)
- added C26: 0.1uF 50V, Capacitor_SMD:C_1206_3216Metric, F.Cu at (142.8, 85.9)
- added C27: 0.1uF 50V, Capacitor_SMD:C_1206_3216Metric, F.Cu at (72.7, 91.6)
- added C9: 0.1uF 50V, Capacitor_SMD:C_1206_3216Metric, F.Cu at (55.3, 61.0)
- C604: value 430 pF -> 380 pF
- L602, L604: value 680 nH -> 720 nH
- L603: value 22 nH -> 24 nH
- moved C700 1.95 mm to (72.7, 94.1), turned to 0 degrees
- moved C198 1.77 mm to (142.9, 72.7), turned to 0 degrees
- moved C108 1.75 mm to (142.9, 64.6), turned to 0 degrees
- moved C98 1.73 mm to (142.9, 56.4), turned to 0 degrees
- moved C208 1.70 mm to (142.9, 80.8), turned to 0 degrees
- moved C608 1.65 mm to (142.8, 138.4), turned to 0 degrees
- moved C408 1.60 mm to (142.8, 122.1), turned to 0 degrees
- moved C298 1.58 mm to (142.8, 88.8), turned to 0 degrees
- moved C508 1.58 mm to (142.8, 130.2), turned to 0 degrees
- moved C308 1.56 mm to (142.7, 114.0), turned to 0 degrees
Connections:
- U10 pad 1: GND -> /RRF28
- U10 pad 3: /RRF28 -> /RRF208
- U12 pad 1: GND -> /RRF30
- U12 pad 3: /RRF30 -> /RRF203
- U13 pad 1: GND -> /RRF38
- U13 pad 3: /RRF38 -> /RRF209
- U15 pad 1: GND -> /RRF40
- U15 pad 3: /RRF40 -> /RRF204
- U16 pad 1: GND -> /RRF48
- U16 pad 3: /RRF48 -> /RRF210
- U18 pad 1: GND -> /RRF50
- U18 pad 3: /RRF50 -> /RRF205
- U19 pad 1: GND -> /RRF58
- U19 pad 3: /RRF58 -> /RRF211
- U21 pad 1: unconnected-(U21-RF1-Pad1) -> /RRF250
- U24 pad 1: GND -> /RRF60
- U24 pad 3: /RRF60 -> /RRF212
- U25 pad 1: GND -> /RRF68
- U25 pad 3: /RRF68 -> /RRF215
- U27 pad 1: GND -> /RRF70
- U27 pad 3: /RRF70 -> /RRF213
- U28 pad 1: GND -> /RRF78
- U28 pad 3: /RRF78 -> /RRF216
- U3 pad 1: GND -> /RRF0
- U3 pad 3: /RRF0 -> /RRF200
- U30 pad 1: GND -> /RRF80
- U30 pad 3: /RRF80 -> /RRF214
- U31 pad 1: GND -> /RRF88
- U31 pad 3: /RRF88 -> /RRF217
- U4 pad 1: GND -> /RRF8
- U4 pad 3: /RRF8 -> /RRF206
- U6 pad 1: GND -> /RRF10
- U6 pad 3: /RRF10 -> /RRF201
- U7 pad 1: GND -> /RRF18
- U7 pad 3: /RRF18 -> /RRF207
- U9 pad 1: GND -> /RRF20
- U9 pad 3: /RRF20 -> /RRF202
Routing:
- net GND: track 27.2 -> 100.6 mm, vias 250 -> 242
- net /RFOUT: track 217.4 -> 191.1 mm
- net /RRF212: track 0.00 -> 2.94 mm
- net /RRF205: track 0.00 -> 2.94 mm
- net /RRF204: track 0.00 -> 2.81 mm
- net /RRF201: track 0.00 -> 2.78 mm
- net /RRF80: track 4.94 -> 7.64 mm
- net /RRF211: track 0.00 -> 2.68 mm
- net /RRF215: track 0.00 -> 2.67 mm
- net /RRF216: track 0.00 -> 2.66 mm
- net /RRF207: track 0.00 -> 2.66 mm
- net /RRF202: track 0.00 -> 2.65 mm
- net /RRF206: track 0.00 -> 2.64 mm
- net /RRF213: track 0.00 -> 2.63 mm
- net /RRF250: track 0.00 -> 2.63 mm
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Other:
- board text added: "12+10m"
- board text added: "17+15m"
- board text added: "A2 A1 A0 ADDR 0 0 0 0x20 0 0 1 0x21 0 1 0 0x22 0 1 1 0x23 1 0 0 0x24 1 0 1 0x25 1 1 0 0x26 1 1 1 0x27"
- board text added: "Design by AC8GY, K9HZ, layout by KI3P. 2024/03/09, V012.06"
- board text removed: "12+ 10m"
- board text removed: "17+ 15m"
- board text removed: "A2 A1 A0 ADDR 0 0 0 0 0 0 1 1 0 1 0 2 0 1 1 3 1 0 0 4 1 0 1 5 1 1 0 6 1 1 1 7"
- board text removed: "Design by AC8GY, K9HZ, layout by KI3P. 2024/02/03, V012.06"

Commit message: Additional fix to BPF board
Parts:
- moved C27 9.70 mm to (82.4, 91.6), turned to 0 degrees
- moved C701 1.85 mm to (82.4, 94.1), turned to 0 degrees
Connections:
- C27 pad 2: GND -> /RFOUT
Routing:
- net /RRF250: track 2.63 -> 4.89 mm
- net GND: track 100.6 -> 99.6 mm
