File: T41_V012_Files_01-15-24/T41_V012_KiCad/T41-BPF-filter-board/T41-exciter-filter-board.kicad_pcb (KiCad board)
At the start: 2 copper layers, 100 x 100 mm, 261 parts, among them J1 TO PA, J2 FROM EXCITE, J3 12-13.8V, J4 Bands, J5 TO RECEIVE, J6 FROM LPF, U1 MASWSS0179, U10 MASWSS0179, U11 SN74LVC1G04DCK, U12 MASWSS0179, U13 MASWSS0179, U14 SN74LVC1G04DCK, U15 MASWSS0179, U16 MASWSS0179, U17 SN74LVC1G04DCK, U18 MASWSS0179, U19 MASWSS0179, U2 SN74LVC1G04DCK, U20 SN74LVC1G04DCK, U21 MASWSS0179, U22 LM1117T-3.3, U23 SN74LVC1G04DCK, U24 MASWSS0179, U25 MASWSS0179, U26 SN74LVC1G04DCK, U27 MASWSS0179, U28 MASWSS0179, U29 SN74LVC1G04DCK, U3 MASWSS0179, U30 MASWSS0179, U31 MASWSS0179, U35 MCP23017_SO, U36 MASWSS0179, U37 SN74LVC1G04DCK, U4 MASWSS0179, U5 SN74LVC1G04DCK, U6 MASWSS0179, U7 MASWSS0179, U8 SN74LVC1G04DCK, U9 MASWSS0179

Commit message: Final fixes to BPF to change addressing of BYPASS path
Parts:
- added R7: 2k2, Resistor_SMD:R_1206_3216Metric, B.Cu at (72.8, 95.6)
- moved C700 10.0 mm to (82.4, 91.7), turned to 180 degrees
- moved C27 9.76 mm to (72.6, 91.8), turned to 180 degrees
Connections:
- C27 pad 2: /RFOUT -> /RFIN
- C700 pad 1: /RFIN -> /RFOUT
Routing:
- net /NF: track 45.4 -> 54.8 mm, vias 1 -> 2
- net /RRF100: track 2.45 -> 6.44 mm
- net /RRF250: track 4.89 -> 2.59 mm
- net GND: track 99.6 -> 98.2 mm
Other:
- board text added: "Design by AC8GY, K9HZ, layout by KI3P. 2024/04/20, V012.06"
- board text removed: "Design by AC8GY, K9HZ, layout by KI3P. 2024/03/09, V012.06"

Commit message: Added pulldown resistors to 12/10 and 17/15 diode combiners
Parts:
- added R8: 2k2, Resistor_SMD:R_1206_3216Metric, F.Cu at (107.2, 103.0)
- R7: moved to F.Cu
- moved R7 34.5 mm to (107.2, 97.5), turned to 90 degrees
- moved D1 0.23 mm to (111.0, 96.5)
- moved D2 0.19 mm to (111.0, 99.0)
- moved D3 0.15 mm to (111.0, 101.5)
- moved D4 0.11 mm to (111.0, 104.0)
Connections:
- R7 pad 1: /NF -> GND
- R7 pad 2: +3V3 -> /17/15m
Routing:
- net /NF: track 54.8 -> 45.4 mm, vias 2 -> 1
- net /17/15m: track 109.0 -> 111.5 mm
- net /12/10m: track 120.8 -> 123.2 mm
