File: T41_V012_Files_01-15-24/T41_V012_KiCad/T41-BPF-filter-board/T41-exciter-filter-board.kicad_sch (KiCad schematic)
At the start: 197 parts, among them J1 TO PA, J2 FROM EXCITE, J3 12-13.8V, J4 Bands, J5 TO RECEIVE, J6 FROM LPF, U1 MASWSS0179, U10 MASWSS0179, U11 SN74LVC1G04DCK, U12 MASWSS0179, U13 MASWSS0179, U14 SN74LVC1G04DCK, U15 MASWSS0179, U16 MASWSS0179, U17 SN74LVC1G04DCK, U18 MASWSS0179, U19 MASWSS0179, U2 SN74LVC1G04DCK, U20 SN74LVC1G04DCK, U21 MASWSS0179, U22 LM1117T-3.3, U23 SN74LVC1G04DCK, U24 MASWSS0179, U25 MASWSS0179, U26 SN74LVC1G04DCK, U27 MASWSS0179, U28 MASWSS0179, U29 SN74LVC1G04DCK, U3 MASWSS0179, U30 MASWSS0179, U31 MASWSS0179, U35 MCP23017_SO, U36 MASWSS0179, U37 SN74LVC1G04DCK, U4 MASWSS0179, U5 SN74LVC1G04DCK, U6 MASWSS0179, U7 MASWSS0179, U8 SN74LVC1G04DCK, U9 MASWSS0179

Commit message: Added 1206 footprints alongside all the coil inductors in the BPF board to allow use of SMD inductors instead of toroids
Parts:
- added L10, L11, L12, L13, L14, L15, L16, L17, L18, L19, L20, L21, L22, L23, L24, L25, L26, L27, L28, L29, L3, L30, L31, L32, L33, L34, L35, L36, L37, L38, L39, L4, L40, L41, L42, L43, L44, L45, L46, L47, L5, L6, L7, L8, L9: L, Inductor_SMD:L_1206_3216Metric, symbol Device:L
Connections:
- net GND: now also L10.2, L11.2, L12.2, L13.2, L14.2, L15.2, L16.2, L17.2, L18.2, L19.2, L20.2, L21.2, L22.2, L23.2, L24.2, L25.2, L26.2, L27.2, L28.2, L29.2, L3.2, L4.2, L5.2, L6.2, L7.2, L8.2, L9.2
- net RF12: now also L6.1
- net RF13: now also L32.2
- net RF14: now also L32.1, L7.1
- net RF15: now also L33.2
- net RF16: now also L33.1, L8.1
- net RF2: now also L3.1
- net RF22: now also L9.1
- net RF23: now also L34.2
- net RF24: now also L10.1, L34.1
- net RF25: now also L35.2
- net RF26: now also L11.1, L35.1
- net RF3: now also L30.2
- net RF32: now also L12.1
- net RF33: now also L36.2
- net RF34: now also L13.1, L36.1
- net RF35: now also L37.2
- net RF36: now also L14.1, L37.1
- net RF4: now also L30.1, L4.1
- net RF42: now also L15.1
- net RF43: now also L38.2
- net RF44: now also L16.1, L38.1
- net RF45: now also L39.2
- net RF46: now also L17.1, L39.1
- net RF5: now also L31.2
- net RF52: now also L18.1
- net RF53: now also L40.2
- net RF54: now also L19.1, L40.1
- net RF55: now also L41.2
- net RF56: now also L20.1, L41.1
- net RF6: now also L31.1, L5.1
- net RF62: now also L23.1
- net RF63: now also L42.2
- net RF64: now also L22.1, L42.1
- net RF65: now also L43.2
- net RF66: now also L21.1, L43.1
- net RF72: now also L26.1
- net RF73: now also L44.2
- net RF74: now also L25.1, L44.1
- net RF75: now also L45.2
- net RF76: now also L24.1, L45.1
- net RF82: now also L29.1
- net RF83: now also L46.2
- net RF84: now also L28.1, L46.1
- net RF85: now also L47.2
- net RF86: now also L27.1, L47.1
Other:
- moved on the sheet: C102, C104, C106, C192, C194, C196, C202, C204, C206, C292, C294, C296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

Commit message: Latest Updates
Latest Updates
Parts:
- C604: value 430 pF -> 380 pF
- L602, L604: value 680 nH -> 720 nH
- L603: value 22 nH -> 24 nH
Changed lines of the file:
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@@
   (title_block
     (title "T41 Exciter Filter Board")
-    (date "2024-02-03")
+    (date "2024-03-07")
     (rev "V 012.06")
     (comment 1 "       KiCad version by Oliver King KI3P")
@@
   (symbol (lib_id "Device:L") (at 133.35 199.39 0) (unit 1)
     (in_bom yes) (on_board yes) (dnp no) (fields_autoplaced)
-    (property "Reference" "L603" (at 134.6173 198.1779 0)
+    (property "Reference" "L603" (at 134.62 198.12 0)
       (effects (font (size 1.27 1.27)) (justify left))
     )
-    (property "Value" "22 nH" (at 134.6173 200.6021 0)
+    (property "Value" "24 nH" (at 134.62 200.66 0)
       (effects (font (size 1.27 1.27)) (justify left))
     )
@@
   (symbol (lib_id "Device:L") (at 148.59 190.5 90) (unit 1)
     (in_bom yes) (on_board yes) (dnp no) (fields_autoplaced)
-    (property "Reference" "L604" (at 148.59 185.8504 90)
+    (property "Reference" "L604" (at 148.59 185.42 90)
       (effects (font (size 1.27 1.27)))
     )
-    (property "Value" "680 nH" (at 148.59 188.2746 90)
+    (property "Value" "720 nH" (at 148.59 187.96 90)
       (effects (font (size 1.27 1.27)))
     )
@@
   (symbol (lib_id "Device:L") (at 123.19 190.5 90) (unit 1)
     (in_bom yes) (on_board yes) (dnp no) (fields_autoplaced)
-    (property "Reference" "L602" (at 123.19 185.8504 90)
+    (property "Reference" "L602" (at 123.19 185.42 90)
       (effects (font (size 1.27 1.27)))
     )
-    (property "Value" "680 nH" (at 123.19 188.2746 90)
+    (property "Value" "720 nH" (at 123.19 187.96 90)
       (effects (font (size 1.27 1.27)))
     )
@@
       (effects (font (size 1.27 1.27)) (justify right))
     )
-    (property "Value" "430 pF" (at 125.349 200.6021 0)
+    (property "Value" "380 pF" (at 125.349 200.6021 0)
       (effects (font (size 1.27 1.27)) (justify right))
     )

Commit message: Fixes to BPF board, adding missing decoupling capacitors
Parts:
- added C10, C11, C12, C13, C14, C15, C16, C17, C18, C19, C20, C21, C22, C23, C24, C25, C26, C27, C9: 0.1uF 50V, Capacitor_SMD:C_1206_3216Metric, symbol Device:C
Connections:
- net GND: now also C10.2, C11.2, C12.2, C13.2, C14.2, C15.1, C16.1, C17.1, C18.1, C19.1, C20.1, C21.1, C22.1, C23.1, C24.1, C25.1, C26.1, C27.2, C9.2; no longer U10.1 (RF1), U12.1 (RF1), U13.1 (RF1), U15.1 (RF1), U16.1 (RF1), U18.1 (RF1), U19.1 (RF1), U24.1 (RF1), U25.1 (RF1), U27.1 (RF1), U28.1 (RF1), U3.1 (RF1), U30.1 (RF1), U31.1 (RF1), U4.1 (RF1), U6.1 (RF1), U7.1 (RF1), U9.1 (RF1)
- net RRF0: now also U3.1 (RF1); no longer U3.3 (RF2)
- net RRF10: now also U6.1 (RF1); no longer U6.3 (RF2)
- net RRF18: now also U7.1 (RF1); no longer U7.3 (RF2)
- net RRF20: now also U9.1 (RF1); no longer U9.3 (RF2)
- net RRF28: now also U10.1 (RF1); no longer U10.3 (RF2)
- net RRF30: now also U12.1 (RF1); no longer U12.3 (RF2)
- net RRF38: now also U13.1 (RF1); no longer U13.3 (RF2)
- net RRF40: now also U15.1 (RF1); no longer U15.3 (RF2)
- net RRF48: now also U16.1 (RF1); no longer U16.3 (RF2)
- net RRF50: now also U18.1 (RF1); no longer U18.3 (RF2)
- net RRF58: now also U19.1 (RF1); no longer U19.3 (RF2)
- net RRF60: now also U24.1 (RF1); no longer U24.3 (RF2)
- net RRF68: now also U25.1 (RF1); no longer U25.3 (RF2)
- net RRF70: now also U27.1 (RF1); no longer U27.3 (RF2)
- net RRF78: now also U28.1 (RF1); no longer U28.3 (RF2)
- net RRF8: now also U4.1 (RF1); no longer U4.3 (RF2)
- net RRF80: now also U30.1 (RF1); no longer U30.3 (RF2)
- net RRF88: now also U31.1 (RF1); no longer U31.3 (RF2)
- net RRF250: now reaches U21.1 (RF1)
- net RRF250: now also C27.1
- new net RRF200: C9.1, U3.3 (RF2)
- new net RRF201: C10.1, U6.3 (RF2)
- new net RRF202: C11.1, U9.3 (RF2)
- new net RRF203: C12.1, U12.3 (RF2)
- new net RRF204: C13.1, U15.3 (RF2)
- new net RRF205: C14.1, U18.3 (RF2)
- new net RRF206: C15.2, U4.3 (RF2)
- new net RRF207: C16.2, U7.3 (RF2)
- new net RRF208: C17.2, U10.3 (RF2)
- new net RRF209: C18.2, U13.3 (RF2)
- new net RRF210: C19.2, U16.3 (RF2)
- new net RRF211: C20.2, U19.3 (RF2)
- new net RRF212: C21.2, U24.3 (RF2)
- new net RRF213: C22.2, U27.3 (RF2)
- new net RRF214: C23.2, U30.3 (RF2)
- new net RRF215: C24.2, U25.3 (RF2)
- new net RRF216: C25.2, U28.3 (RF2)
- new net RRF217: C26.2, U31.3 (RF2)
- no-connect marks 13 -> 12
Other:
- note added: "A2 A1 A0 ADDR 0 0 0 0x20 0 0 1 0x21 0 1 0 0x22 0 1 1 0x23 1 0 0 0x24 1 0 1 0x25 1 1 0 0x26 1 1 1 0x27"
- note removed: "A2 A1 A0 ADDR 0 0 0 0 0 0 1 1 0 1 0 2 0 1 1 3 1 0 0 4 1 0 1 5 1 1 0 6 1 1 1 7"
- moved on the sheet: C100, C108, C190, C198, C200, C208, C290, C298, C300, C308, C400, C408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

Commit message: Additional fix to BPF board
Connections:
- net GND: no longer C27.2
- net RFOUT: now also C27.2
Changed lines of the file:
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@@
 	)
 	(junction
+		(at 104.14 224.79)
+		(diameter 0)
+		(color 0 0 0 0)
+	)
+	(junction
 		(at 308.61 102.87)
 		(diameter 0)
@@
 	(wire
 		(pts
+			(xy 104.14 214.63) (xy 104.14 224.79)
+		)
+		(stroke
+			(width 0)
+			(type default)
+		)
+	)
+	(wire
+		(pts
 			(xy 168.91 30.48) (xy 173.99 30.48)
 		)
@@
 	(wire
 		(pts
-			(xy 60.96 213.36) (xy 58.42 213.36)
-		)
-		(stroke
-			(width 0)
-			(type default)
-		)
-	)
-	(wire
-		(pts
 			(xy 356.87 93.98) (xy 358.14 93.98)
 		)
@@
 	(wire
 		(pts
+			(xy 60.96 214.63) (xy 104.14 214.63)
+		)
+		(stroke
+			(width 0)
+			(type default)
+		)
+	)
+	(wire
+		(pts
 			(xy 133.35 66.04) (xy 133.35 60.96)
 		)
@@
 	(wire
 		(pts
-			(xy 60.96 214.63) (xy 60.96 213.36)
-		)
-		(stroke
-			(width 0)
-			(type default)
-		)
-	)
-	(wire
-		(pts
 			(xy 88.9 124.46) (xy 96.52 124.46)
 		)
@@
 					(unit 1)
 				)
-			)
-		)
-	)
-	(symbol
-		(lib_id "power:GND")
-		(at 58.42 213.36 0)
-		(unit 1)
-		(exclude_from_sim no)
-		(in_bom yes)
-		(on_board yes)
-		(dnp no)
-		(property "Reference" "#PWR041"
-			(at 58.42 219.71 0)
-			(effects
-				(font
-					(size 1.27 1.27)
-				)
-				(hide yes)
-			)
-		)
-		(property "Value" "GND"
-			(at 55.88 214.63 90)
-			(effects
-				(font
-					(size 1.27 1.27)
-				)
-			)
-		)
-		(property "Footprint" ""
-			(at 58.42 213.36 0)
-			(effects
-				(font
-					(size 1.27 1.27)
-				)
-				(hide yes)
-			)
-		)
-		(property "Datasheet" ""
-			(at 58.42 213.36 0)
-			(effects
-				(font
-					(size 1.27 1.27)
-				)
-				(hide yes)
-			)
-		)
-		(property "Description" ""
-			(at 58.42 213.36 0)
-			(effects
-				(font
-					(size 1.27 1.27)
-				)
-				(hide yes)
-			)
-		)
-		(pin "1"
-		)
-		(instances
-			(project "T41-exciter-filter-board"
-				(path "/56a77fe5-f7a5-414c-a0f7-d659071572ee"
-					(reference "#PWR041")
-					(unit 1)
-				)

Commit message: Final fixes to BPF to change addressing of BYPASS path
Parts:
- added R7: 2k2, Resistor_SMD:R_1206_3216Metric, symbol Device:R
Connections:
- net +3V3: now also R7.2
- net NF: now also R7.1
- net RFIN: now also C27.2; no longer C700.1
- net RFOUT: now also C700.1; no longer C27.2
Other:
- note added: "Pullup selects BYPASS when board is powered & I2C is not configured"
- moved on the sheet: C27, C700

Commit message: Added pulldown resistors to 12/10 and 17/15 diode combiners
Parts:
- added R8: 2k2, Resistor_SMD:R_1206_3216Metric, symbol Device:R
Connections:
- net +3V3: no longer R7.2
- net 12/10m: now also R8.2
- net 17/15m: now also R7.2
- net GND: now also R7.1, R8.1
- net NF: no longer R7.1
Other:
- note removed: "Pullup selects BYPASS when board is powered & I2C is not configured"
Changed lines of the file:
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@@
 	)
 	(junction
-		(at 16.51 227.33)
-		(diameter 0)
-		(color 0 0 0 0)
-	)
-	(junction
 		(at 109.22 74.93)
 		(diameter 0)
@@
 	)
 	(junction
-		(at 26.67 217.17)
-		(diameter 0)
-		(color 0 0 0 0)
-	)
-	(junction
 		(at 133.35 35.56)
 		(diameter 0)
@@
 	(wire
 		(pts
-			(xy 16.51 217.17) (xy 26.67 217.17)
-		)
-		(stroke
-			(width 0)
-			(type default)
-		)
-	)
-	(wire
-		(pts
 			(xy 307.34 43.18) (xy 308.61 43.18)
 		)
@@
 	(wire
 		(pts
-			(xy 16.51 224.79) (xy 16.51 227.33)
-		)
-		(stroke
-			(width 0)
-			(type default)
-		)
-	)
-	(wire
-		(pts
 			(xy 120.65 204.47) (xy 120.65 205.74)
 		)
@@
 		)
 	)
-	(text "Pullup selects BYPASS\nwhen board is powered\n& I2C is not configured"
-		(exclude_from_sim no)
-		(at 14.224 210.82 0)
-		(effects
-			(font
-				(size 1.27 1.27)
-			)
-			(justify left)
-		)
-	)
 	(text "RFCONTROL SIGNALS:\nRxTx: H=Tx, L=Rx"
 		(exclude_from_sim no)
@@
 	)
 	(symbol
-		(lib_id "Device:C")
-		(at 100.33 30.48 90)
+		(lib_id "Device:R")
+		(at 368.3 204.47 180)
 		(unit 1)
 		(exclude_from_sim no)
@@
 		(on_board yes)
 		(dnp no)
-		(fields_autoplaced yes)
-		(property "Reference" "C101"
-			(at 100.33 24.1767 90)
+		(property "Reference" "R8"
+			(at 370.586 203.454 0)
 			(effects
 				(font
 					(size 1.27 1.27)
 				)
+				(justify right)
 			)
 		)
-		(property "Value" "0.1uF 50V"
-			(at 100.33 26.6009 90)
+		(property "Value" "2k2"
+			(at 369.824 205.486 0)
 			(effects
 				(font
 					(size 1.27 1.27)
 				)
+				(justify right)
 			)
 		)
-		(property "Footprint" "Capacitor_SMD:C_1206_3216Metric"
-			(at 104.14 29.5148 0)
+		(property "Footprint" "Resistor_SMD:R_1206_3216Metric"
+			(at 370.078 204.47 90)
 			(effects
 				(font
@@
 		)
 		(property "Datasheet" "~"
-			(at 100.33 30.48 0)
+			(at 368.3 204.47 0)
 			(effects
 				(font
@@
 		)
 		(property "Description" ""
-			(at 100.33 30.48 0)
+			(at 368.3 204.47 0)
 			(effects
 				(font
@@
 			)
 		)
-		(property "Mouser Part Number" "C1206C104K5RACTU"
-			(at 100.33 30.48 0)
+		(property "Mouser Part Number" "652-CR1206FX-2201ELF"
+			(at 368.3 204.47 0)
 			(effects
 				(font
@@
 			(project "T41-exciter-filter-board"
 				(path "/56a77fe5-f7a5-414c-a0f7-d659071572ee"
-					(reference "C101")
+					(reference "R8")
 					(unit 1)
 				)
@@
 	)
 	(symbol
-		(lib_id "Device:R")
-		(at 16.51 220.98 180)
+		(lib_id "Device:C")
+		(at 100.33 30.48 90)
 		(unit 1)
 		(exclude_from_sim no)
@@
 		(on_board yes)
 		(dnp no)
-		(property "Reference" "R7"
-			(at 18.796 219.964 0)
+		(fields_autoplaced yes)
+		(property "Reference" "C101"
+			(at 100.33 24.1767 90)
 			(effects
 				(font
 					(size 1.27 1.27)
 				)
-				(justify right)
 			)
 		)
-		(property "Value" "2k2"
-			(at 18.034 221.996 0)
+		(property "Value" "0.1uF 50V"
+			(at 100.33 26.6009 90)
 			(effects
 				(font
 					(size 1.27 1.27)
 				)
-				(justify right)
 			)
 		)
-		(property "Footprint" "Resistor_SMD:R_1206_3216Metric"
-			(at 18.288 220.98 90)
+		(property "Footprint" "Capacitor_SMD:C_1206_3216Metric"
+			(at 104.14 29.5148 0)
 			(effects
 				(font
@@
 		)
 		(property "Datasheet" "~"
-			(at 16.51 220.98 0)
+			(at 100.33 30.48 0)
 			(effects
 				(font
@@
 		)
 		(property "Description" ""
-			(at 16.51 220.98 0)
+			(at 100.33 30.48 0)
 			(effects
 				(font
@@
 			)
 		)
-		(property "Mouser Part Number" "652-CR1206FX-2201ELF"
-			(at 16.51 220.98 0)
+		(property "Mouser Part Number" "C1206C104K5RACTU"
+			(at 100.33 30.48 0)
 			(effects
 				(font
@@
 			(project "T41-exciter-filter-board"
 				(path "/56a77fe5-f7a5-414c-a0f7-d659071572ee"
-					(reference "R7")
+					(reference "C101")
 					(unit 1)
 				)
@@
 	)
 	(symbol
+		(lib_id "power:GND")
+		(at 368.3 208.28 0)
+		(mirror y)
+		(unit 1)
+		(exclude_from_sim no)
+		(in_bom yes)
+		(on_board yes)
+		(dnp no)
+		(property "Reference" "#PWR061"
+			(at 368.3 214.63 0)
+			(effects
+				(font
+					(size 1.27 1.27)
+				)
+				(hide yes)
+			)
+		)
+		(property "Value" "GND"
+			(at 370.84 209.55 90)
+			(effects
+				(font
+					(size 1.27 1.27)
+				)
+			)
+		)
+		(property "Footprint" ""
+			(at 368.3 208.28 0)
+			(effects
+				(font
+					(size 1.27 1.27)
+				)
+				(hide yes)
+			)
+		)
+		(property "Datasheet" ""
+			(at 368.3 208.28 0)
+			(effects
+				(font
+					(size 1.27 1.27)
+				)
+				(hide yes)
+			)
+		)
+		(property "Description" ""
+			(at 368.3 208.28 0)
+			(effects
+				(font
+					(size 1.27 1.27)
+				)
+				(hide yes)
+			)
+		)
+		(pin "1"
+		)
+		(instances
+			(project "T41-exciter-filter-board"
+				(path "/56a77fe5-f7a5-414c-a0f7-d659071572ee"
+					(reference "#PWR061")
+					(unit 1)
+				)
+			)
+		)
+	)
+	(symbol
 		(lib_id "Device:C")
 		(at 139.7 190.5 270)
@@
 	)
 	(symbol
+		(lib_id "Device:R")
+		(at 368.3 186.69 180)
+		(unit 1)
+		(exclude_from_sim no)
+		(in_bom yes)
+		(on_board yes)
+		(dnp no)
+		(property "Reference" "R7"
+			(at 370.586 185.674 0)
+			(effects
+				(font
+					(size 1.27 1.27)
+				)
+				(justify right)
+			)
+		)
+		(property "Value" "2k2"
+			(at 369.824 187.706 0)
+			(effects
+				(font
+					(size 1.27 1.27)
+				)
+				(justify right)
+			)
+		)
+		(property "Footprint" "Resistor_SMD:R_1206_3216Metric"
+			(at 370.078 186.69 90)
+			(effects
+				(font
+					(size 1.27 1.27)
+				)
+				(hide yes)
+			)
+		)
+		(property "Datasheet" "~"
+			(at 368.3 186.69 0)
+			(effects
+				(font
+					(size 1.27 1.27)
+				)
+				(hide yes)
+			)
+		)
+		(property "Description" ""
+			(at 368.3 186.69 0)
+			(effects
+				(font
+					(size 1.27 1.27)
+				)
+				(hide yes)
+			)
+		)
+		(property "Mouser Part Number" "652-CR1206FX-2201ELF"
+			(at 368.3 186.69 0)
+			(effects
+				(font
+					(size 1.27 1.27)
+				)
+				(hide yes)
+			)
+		)
+		(pin "2"
+		)
+		(pin "1"
+		)
+		(instances
+			(project "T41-exciter-filter-board"
+				(path "/56a77fe5-f7a5-414c-a0f7-d659071572ee"
+					(reference "R7")
+					(unit 1)
+				)
+			)
+		)
+	)
+	(symbol
 		(lib_id "power:+3V3")
 		(at 26.67 22.86 0)
@@
 					(unit 1)
 				)
+			)
+		)
+	)
+	(symbol
+		(lib_id "power:GND")
+		(at 368.3 190.5 0)
+		(mirror y)
+		(unit 1)
+		(exclude_from_sim no)
+		(in_bom yes)
+		(on_board yes)
+		(dnp no)
+		(property "Reference" "#PWR041"
+			(at 368.3 196.85 0)
+			(effects
+				(font
+					(size 1.27 1.27)
+				)
+				(hide yes)
+			)
+		)
+		(property "Value" "GND"
+			(at 370.84 191.77 90)
+			(effects
+				(font
+					(size 1.27 1.27)
+				)
+			)
+		)
+		(property "Footprint" ""
+			(at 368.3 190.5 0)
+			(effects
+				(font
+					(size 1.27 1.27)
+				)
+				(hide yes)
+			)
+		)
+		(property "Datasheet" ""
+			(at 368.3 190.5 0)
+			(effects
+				(font
+					(size 1.27 1.27)
+				)
+				(hide yes)
+			)
+		)
+		(property "Description" ""
+			(at 368.3 190.5 0)
+			(effects
+				(font
+					(size 1.27 1.27)
+				)
+				(hide yes)
+			)
+		)
+		(pin "1"
+		)
+		(instances
+			(project "T41-exciter-filter-board"
+				(path "/56a77fe5-f7a5-414c-a0f7-d659071572ee"
+					(reference "#PWR041")
+					(unit 1)
+				)

Commit message: Added Glen VK3PE toroid winding details to BPF schematic
Other:
- note added: "1.5nF+100p"
- note added: "10T T37-2 6""
- note added: "13T T37-0 7""
- note added: "14t FT37-61 14""
- note added: "16T T37-0 9""
- note added: "17T T37-0 9""
- note added: "17T T37-10 11""
- note added: "18T T37-10 10""
- note added: "20T T37-10 11""
- note added: "20t T37-10 11""
- note added: "21T T37-0 11""
- note added: "22T T37-0 12""
- note added: "22T T37-1 12""
- note added: "22T T37-10 12""
- note added: "25T T37-1 13""
- note added: "26T T37-0 14""
- note added: "26T T37-1 14""
- note added: "26T T37-6 14""
- note added: "27T T37-6 14""
- note added: "34T T37-0 18""
- note added: "38T T37-10 20""
- note added: "7T T37-0 4""
- note added: "9T T37-0 5""
- note added: "ALL TOROIDS WOUND WITH #28 WIRE 0.32mm"
- note added: "JULY 30th 2024 VK3PE ADDED SOME NOTES"
- note added: "June 1st 2024 vk3pe: corrected wire length for L91 and L95"

Commit message: Updated instructions in BPF schematic for second receiver
Other:
- note added: "Added for backwards compatibility with V010/V011 LPF boards and V012 second receiver operation. Only populate if using V012 2nd receiver or with V010/V011 LPF boards."
- note added: "June 1 2024: VK3PE Corrected wire length for L91 and L95 July 30 2024: VK3PE Added some notes August 25 2024: KI3P Clarified instructions in red box"
- note added: "Solder JP10 and JP11 closed if using V012 LPF boards and single receiver"
- note removed: "Added for backwards compatibility with V010/V011 LPF boards. Do not populate if using V012 LPF boards."
- note removed: "JULY 30th 2024 VK3PE ADDED SOME NOTES"
- note removed: "June 1st 2024 vk3pe: corrected wire length for L91 and L95"
- note removed: "Solder JP10 and JP11 closed if using V012 LPF boards"
Changed lines of the file:
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@@
 	(title_block
 		(title "T41 Exciter Filter Board")
-		(date "2024-04-20")
+		(date "2024-08-25")
 		(rev "V 012.06")
 		(comment 1 "       KiCad version by Oliver King KI3P")
@@
 		)
 	)
-	(text "June 1st 2024 vk3pe: corrected wire length for L91  and L95"
+	(text "June 1 2024: VK3PE Corrected wire length for L91 and L95\nJuly 30 2024: VK3PE Added some notes\nAugust 25 2024: KI3P Clarified instructions in red box"
 		(exclude_from_sim no)
-		(at 270.51 245.364 0)
+		(at 196.342 241.3 0)
 		(effects
 			(font
@@
 				(color 255 42 21 1)
 			)
+			(justify left)
 		)
 	)
-	(text "Added for backwards compatibility\nwith V010/V011 LPF boards. Do not \npopulate if using V012 LPF boards."
+	(text "Added for backwards compatibility \nwith V010/V011 LPF boards and V012 \nsecond receiver operation. Only \npopulate if using V012 2nd receiver \nor with V010/V011 LPF boards."
 		(exclude_from_sim no)
-		(at 78.74 254 0)
+		(at 77.978 258.318 0)
 		(effects
 			(font
@@
 		)
 	)
-	(text "JULY 30th 2024 VK3PE ADDED SOME NOTES"
-		(exclude_from_sim no)
-		(at 250.444 250.698 0)
-		(effects
-			(font
-				(size 3 3)
-				(color 25 28 255 1)
-			)
-		)
-	)
 	(text "ADDRESS SELECT"
 		(exclude_from_sim no)
@@
 		)
 	)
-	(text "Solder JP10 and JP11 closed\nif using V012 LPF boards"
+	(text "Solder JP10 and JP11 closed\nif using V012 LPF boards and\nsingle receiver"
 		(exclude_from_sim no)
 		(at 130.81 237.49 0)
