File: K9HZ_LPF_Module/K9HZ_LPF_V1.00_Schematics/K9HZ_100W_11band_LPF-TR-carrier/K9HZ_100W_11band_LPF-TR-carrier.kicad_sch (KiCad schematic)
At the start: 12 parts, among them J22.1 ANTENNA, J22.2 TRANSMIT, J23.1 RECEIVE, J23.2 TR CTL, K1 HF41F/12-ZS, K2 HF41F/12-ZS, Q1 BS170

Commit message: Updated LPF carrier board schematic with 6.8k resistor value
Parts:
- R2: value 10k -> 6.8k; Mouser Part Number 652-CR1206JW-103ELF -> 652-CR1206JW-682ELF
