File: K9HZ_100W_PA/K9HZ_100W_KiCad/K9HZ_100W_KiCad.kicad_pcb (KiCad board)
At the start: 2 copper layers, 125 x 83.7 mm, 74 parts, among them J1 BANDS, J2 RF_IN, J4 12V, 20A, J5 RF_OUT, J7 Temp monitor, Q1 BSS84, Q2 BS170, Q3 BD677, Q4 RD100HHF1C, Q5 RD100HHF1C, T1 BN43-2402, T2 BN43-3312, U2 AP7381-33Y-13, U3 MCP3021A0T-E/OT, U4 ZXCT1010, U5 L4931CDT50

Commit message: Fixed footprint of T2 in 100W PA
Parts:
- moved C11 30.6 mm to (193.2, 128.7), turned to 0 degrees
- moved C14 28.5 mm to (193.2, 138.8), turned to 0 degrees
- moved C12 28.4 mm to (193.2, 132.1), turned to 0 degrees
- moved C13 27.6 mm to (193.2, 135.4), turned to 0 degrees
Routing:
- net GND: vias 497 -> 485
Other:
- board text added: "K9HZ 100W 1-54 MHz 12V PA V1.05 - 08/03/2024 Copyright 2023 WJ Schmidt - K9HZ"
- board text removed: "K9HZ 100W 1-54 MHz 12V PA V1.04 - 7/31/2024 Copyright 2023 WJ Schmidt - K9HZ"

Commit message: Added silkscreen art for 100W amp bias pot control per Glenn VK3PE suggestion
Parts:
- moved RV1 5.08 mm to (112.3, 97.0), turned to -90 degrees
- moved RV2 5.08 mm to (112.3, 133.1), turned to 90 degrees
Connections:
- RV1 pad 1: Net-(Q1-D) -> Net-(Q3-B)
- RV1 pad 3: Net-(Q3-B) -> Net-(Q1-D)
- RV2 pad 1: Net-(Q1-D) -> Net-(Q3-B)
- RV2 pad 3: Net-(Q3-B) -> Net-(Q1-D)
Other:
- board text added: "Increase bias"
