File: K9HZ_100W_PA/K9HZ_100W_KiCad/K9HZ_100W_KiCad.kicad_sch (KiCad schematic)
At the start: 87 parts, among them J1 BANDS, J2 RF_IN, J3 Over-Temp Alarm, J4 12V, 20A, J5 RF_OUT, J7 Temp monitor, Q1 BSS84, Q2 BS170, Q3 BD677, Q4 RD100HHF1C, Q5 RD100HHF1C, T1 BN43-2402, T2 BN43-3312, U1 ADT75, U2 AP7381-33Y-13, U3 MCP3021A0T-E/OT, U4 ZXCT1010, U5 L4931CDT50

Commit message: Added silkscreen art for 100W amp bias pot control per Glenn VK3PE suggestion
Connections:
- net at RV1.1, RV2.1: now also Q3.1 (B); no longer Q1.3 (D)
- net at RV1.3, RV2.3: now also Q1.3 (D); no longer Q3.1 (B)
Other:
- moved on the sheet: RV2
Changed lines of the file:
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@@
 	(symbol
 		(lib_id "Device:R_Potentiometer")
-		(at 134.62 172.72 0)
-		(mirror y)
+		(at 134.62 172.72 180)
 		(unit 1)
 		(exclude_from_sim no)
@@
 		(dnp no)
 		(property "Reference" "RV2"
-			(at 136.398 171.5078 0)
+			(at 136.398 173.9322 0)
 			(effects
 				(font
@@
 		)
 		(property "Value" "500R"
-			(at 136.398 173.9321 0)
+			(at 136.398 171.5079 0)
 			(effects
 				(font
@@
 		(lib_id "Device:R_Potentiometer")
 		(at 104.14 172.72 0)
+		(mirror x)
 		(unit 1)
 		(exclude_from_sim no)
@@
 		(on_board yes)
 		(dnp no)
-		(fields_autoplaced yes)
 		(property "Reference" "RV1"
-			(at 102.362 171.5078 0)
+			(at 102.362 173.9322 0)
 			(effects
 				(font
@@
 		)
 		(property "Value" "500R"
-			(at 102.362 173.9321 0)
+			(at 102.362 171.5079 0)
 			(effects
 				(font
