File: T41_V012_Mini_Files/T41_V012_Mini_Projects/T41 mini-LPF+PA-board-V012/T41-mini-LPF+PA-board-V012.kicad_sch (KiCad schematic)
At the start: 169 parts, among them J17 RF interconnect, J22 RF interconnect, J26 LPF CTRL LOW, J27 LPF CTRL HI, K10 HF41F/12-ZS, K11 HF41F/12-ZS, K12 HF41F/12-ZS, K13 HF41F/12-ZS, K14 HF41F/12-ZS, K15 HF41F/12-ZS, K16 HF41F/12-ZS, K17 HF41F/12-ZS, K18 HF41F/12-ZS, K19 HF41F/12-ZS, K20 HF41F/12-ZS, K21 HF41F/12-ZS, K22 HF41F/12-ZS, K23 HF41F/12-ZS, K24 HF41F/12-ZS, K25 HF41F/12-ZS, K26 HF41F/12-ZS, K27 HF41F/12-ZS, K28 HF41F/12-ZS, K29 HF41F/12-ZS, K32 HF41F/12-ZS, K33 HF41F/12-ZS, K8 HF41F/12-ZS, K9 HF41F/12-ZS

Commit message: Updates
Updates
Parts:
- removed C100, C39, C67: 60pF 100V, Capacitor_SMD:C_1206_3216Metric, symbol Device:C
- removed C101, C26: 390pF 100V, Capacitor_SMD:C_1206_3216Metric, symbol Device:C
- removed C102, C104, C28, C33, C36, C42, C61, C83, C95, C97: 150pF 100V, Capacitor_SMD:C_1206_3216Metric, symbol Device:C
- removed C103, C25, C43, C44, C48, C54, C55, C59, C73, C77, C79, C87, C88: 330pF 100V, Capacitor_SMD:C_1206_3216Metric, symbol Device:C
- removed C105, C24, C35, C41, C53, C72, C85, C90: 82pF 100V, Capacitor_SMD:C_1206_3216Metric, symbol Device:C
- removed C116, C118, C119, C120, C121, C122, C123, C124, C125, C126, C127, C157, C158: 0.1uF 50V, Capacitor_SMD:C_1206_3216Metric, symbol Device:C
- removed C29, C91: 1500pF 100V, Capacitor_SMD:C_1206_3216Metric, symbol Device:C
- removed C30, C40, C47, C78, C89, C92: 470pF 100V, Capacitor_SMD:C_1206_3216Metric, symbol Device:C
- removed C31, C93: 560pF 100V, Capacitor_SMD:C_1206_3216Metric, symbol Device:C
- removed C32, C38, C52, C56, C58, C74, C76, C94, C99: 100pF 100V, Capacitor_SMD:C_1206_3216Metric, symbol Device:C
- removed C34, C49, C80, C96: 220pF 100V, Capacitor_SMD:C_1206_3216Metric, symbol Device:C
- removed C37, C98: 120pF 100V, Capacitor_SMD:C_1206_3216Metric, symbol Device:C
- removed C45, C84: 2200pF 100V, Capacitor_SMD:C_1206_3216Metric, symbol Device:C
- removed C46, C86: 1200pF 100V, Capacitor_SMD:C_1206_3216Metric, symbol Device:C
- removed C50, C81: 180pF 100V, Capacitor_SMD:C_1206_3216Metric, symbol Device:C
- removed C51, C82: 91pF 100V, Capacitor_SMD:C_1206_3216Metric, symbol Device:C
- removed C57, C75: 56pF 100V, Capacitor_SMD:C_1206_3216Metric, symbol Device:C
- removed C60, C62, C64: 47pF 100V, Capacitor_SMD:C_1206_3216Metric, symbol Device:C
- removed C63, C69: 27pF 100V, Capacitor_SMD:C_1206_3216Metric, symbol Device:C
- removed C65: 33pF 100V, Capacitor_SMD:C_1206_3216Metric, symbol Device:C
- removed C66, C68: 68pF 100V, Capacitor_SMD:C_1206_3216Metric, symbol Device:C
- removed C70: 14pF 100V, Capacitor_SMD:C_1206_3216Metric, symbol Device:C
- removed C71: 39pF 100V, Capacitor_SMD:C_1206_3216Metric, symbol Device:C
- removed J26: LPF CTRL LOW, Connector_IDC:IDC-Header_2x05_P2.54mm_Vertical, symbol T41_Library:IDC_2x5
- removed J27: LPF CTRL HI, Connector_IDC:IDC-Header_2x05_P2.54mm_Vertical, symbol T41_Library:IDC_2x5
- removed K10, K11, K15, K18, K24, K25, K26, K27, K28, K29, K32, K33, K8, K9: HF41F/12-ZS, T41_Library:Relay_SPDT_HF41F12-ZS, symbol Relay:Relay_SPDT
- removed L10, L32: 0.447uH, T41_Library:T68-6-toroid-vertical, symbol Device:L_Ferrite
- removed L11, L33: 0.337uH, T41_Library:T68-6-toroid-vertical, symbol Device:L_Ferrite
- removed L12, L34: 0.335uH, T41_Library:T68-6-toroid-vertical, symbol Device:L_Ferrite
- removed L13, L35: 0.188uH, T41_Library:T68-6-toroid-vertical, symbol Device:L_Ferrite
- removed L14: 4.73uH, T41_Library:T68-6-toroid-vertical, symbol Device:L_Ferrite
- removed L15: 2.43uH, T41_Library:T68-6-toroid-vertical, symbol Device:L_Ferrite
- removed L16: 1.60uH, T41_Library:T68-6-toroid-vertical, symbol Device:L_Ferrite
- removed L17: 1.22uH, T41_Library:T68-6-toroid-vertical, symbol Device:L_Ferrite
- removed L18: 0.843uH, T41_Library:T68-6-toroid-vertical, symbol Device:L_Ferrite
- removed L19: 0.608uH, T41_Library:T68-6-toroid-vertical, symbol Device:L_Ferrite
- removed L20: 0.471uH, T41_Library:T68-6-toroid-vertical, symbol Device:L_Ferrite
- removed L21: 0.406uH, T41_Library:T68-6-toroid-vertical, symbol Device:L_Ferrite
- removed L22: 0.342uH, T41_Library:T68-6-toroid-vertical, symbol Device:L_Ferrite
- removed L23: 0.305uH, T41_Library:T68-6-toroid-vertical, symbol Device:L_Ferrite
- removed L24: 0.170uH, T41_Library:T68-6-toroid-vertical, symbol Device:L_Ferrite
- removed L25, L3: 5.21uH, T41_Library:T68-6-toroid-vertical, symbol Device:L_Ferrite
- removed L26, L4: 2.68uH, T41_Library:T68-6-toroid-vertical, symbol Device:L_Ferrite
- removed L27, L5: 1.76uH, T41_Library:T68-6-toroid-vertical, symbol Device:L_Ferrite
- removed L28, L6: 1.34uH, T41_Library:T68-6-toroid-vertical, symbol Device:L_Ferrite
- removed L29, L7: 0.928uH, T41_Library:T68-6-toroid-vertical, symbol Device:L_Ferrite
- removed L30, L8: 0.670uH, T41_Library:T68-6-toroid-vertical, symbol Device:L_Ferrite
- removed L31, L9: 0.519uH, T41_Library:T68-6-toroid-vertical, symbol Device:L_Ferrite
- added C1, C10, C11, C12, C13, C14, C2, C20, C3, C4, C5, C6, C600, C601, C607, C608, C7, C700, C701, C8, C9: 0.1uF 50V, Capacitor_SMD:C_1206_3216Metric, symbol Device:C
- added C602, C606: 240 pF, Capacitor_SMD:C_1206_3216Metric, symbol Device:C
- added C603, C605: 13 pF, Capacitor_SMD:C_1206_3216Metric, symbol Device:C
- added C604: 380 pF, Capacitor_SMD:C_1206_3216Metric, symbol Device:C
- added D1, D2, D3, D4, D5, D6, D7: 1N4148, Diode_THT:D_DO-35_SOD27_P7.62mm_Horizontal, symbol Diode:1N4148
- added J1: TO PA, Connector_Coaxial:SMA_Amphenol_901-144_Vertical, symbol Connector:Conn_Coaxial
- added J2: FROM EXCITE, Connector_Coaxial:SMA_Amphenol_901-144_Vertical, symbol Connector:Conn_Coaxial
- added J23.1: RECEIVE, Connector_PinSocket_2.54mm:PinSocket_1x05_P2.54mm_Vertical, symbol Connector:Conn_01x05_Socket
- added J3: 12-13.8V, TerminalBlock:TerminalBlock_bornier-2_P5.08mm, symbol Connector:Screw_Terminal_01x02
- added J4: Antenna, Connector_Coaxial:SMA_Amphenol_901-144_Vertical, symbol Connector:Conn_Coaxial
- added J5: TO RECEIVE, Connector_Coaxial:SMA_Amphenol_901-144_Vertical, symbol Connector:Conn_Coaxial
- added J6: FROM LPF, Connector_Coaxial:SMA_Amphenol_901-144_Vertical, symbol Connector:Conn_Coaxial
- added J7, J8: PA+BPF+LPF, Connector_PinHeader_2.54mm:PinHeader_2x05_P2.54mm_Vertical, symbol Connector_Generic:Conn_02x04_Odd_Even
- added JP10, JP11: SolderJumper_2_Open, Jumper:SolderJumper-2_P1.3mm_Open_TrianglePad1.0x1.5mm, symbol Jumper:SolderJumper_2_Open
- added K1, K2: HF41F/12-ZS, T41_Library:Relay_SPDT_HF41F12-ZS, symbol Relay:Relay_SPDT
- added L1: 10uH 20%, Inductor_SMD:L_Bourns-SRN6028, symbol Device:L
- added L18, L19, L20, L40, L41: L, Inductor_SMD:L_1206_3216Metric, symbol Device:L
- added L601, L605: 39 nH, T41_Library:FT37-toroid-vertical, symbol Device:L
- added L602, L604: 720 nH, T41_Library:FT37-toroid-vertical, symbol Device:L
- added L603: 24 nH, T41_Library:FT37-toroid-vertical, symbol Device:L
- added Q1, Q2, Q3, Q4, Q5, Q6, Q7, Q8: BS170, Package_TO_SOT_THT:TO-92_Inline, symbol Transistor_FET:BS170
- added R1: 50R, Resistor_SMD:R_1206_3216Metric, symbol Device:R
- added R2, R3, R4, R5, R6, R7, R8, R9: 6.8k, Resistor_SMD:R_1206_3216Metric, symbol Device:R
- added U1, U18, U19, U21, U36: MASWSS0179, T41_Library:MASWSS0179-SOT-26, symbol RF_Switch:MASWSS0179
- added U17, U20, U37: SN74LVC1G04DCK, T41_Library:SOT-SC70, symbol 74xGxx:74LVC1G04
- C27: value 150pF 100V -> 0.1uF 50V; Mouser Part Number 80-C1206C151J1G -> C1206C104K5RACTU
Connections:
- net +12V: no longer C107.1, C108.1, K14.A1, K16.A1
- net B160M: no longer K21.A1
- net B30M: no longer K23.A1
- net B40M: no longer K22.A1
- net B60M: no longer K20.A1
- net B80M: no longer K19.A1
- net GND: now also C1.2, C10.2, C11.2, C12.2, C13.2, C14.2, C2.2, C20.1, C3.2, C4.2, C602.1, C604.1, C606.1, C9.2, J1.2 (Ext), J2.2 (Ext), J3.2 (Pin_2), J4.2 (Ext), J5.2 (Ext), J6.2 (Ext), J7.8 (Pin_8), J8.8 (Pin_8), K1.14, L18.2, L19.2, L20.2, L601.2, L603.2, L605.2, Q1.3 (S), Q2.3 (S), Q3.3 (S), Q4.3 (S), Q5.3 (S), Q6.3 (S), Q7.3 (S), Q8.3 (S), R1.2, R2.2, R3.2, R4.2, R5.2, R6.2, R7.2, R8.2, R9.2, U17.3 (GND), U18.2 (GND), U19.2 (GND), U20.3 (GND), U21.2 (GND), U36.2 (GND), U37.3 (GND); no longer C27.1
- net RF1: now also K2.11; no longer J17.1 (In)
- net RF10: no longer names the net of K19.11
- net RF11: no longer names the net of K13.11
- net RF14: no longer names the net of K20.11
- net RF15: no longer names the net of K12.11
- net RF18: no longer names the net of K22.11
- net RF19: no longer names the net of C27.2
- net RF19: now also C600.1, JP10.2 (B), U1.5 (RFC); no longer K17.11
- net RF2: no longer names the net of K16.11
- net RF22: no longer names the net of K23.11
- net RF5: no longer names the net of K21.11
- net RF7: no longer names the net of K14.11
- new net: C608.2, C700.1, C701.2, JP11.2 (B), U36.5 (RFC)
- new net: C108.1, K14.A1
- new net: J23.1.1 (Pin_1), J23.1.2 (Pin_2), J23.1.3 (Pin_3), J23.1.4 (Pin_4), J23.1.5 (Pin_5), K1.11
- new net: D1.2 (A), K1.A1, K2.A1, Q2.1 (D)
- new net: K2.12, R1.1
- new net: J3.1 (Pin_1), L1.1
- new net +3V3: U17.5 (VCC), U20.5 (VCC), U37.5 (VCC)
- new net +5V: C1.1, C107.1, D1.1 (K), D2.1 (K), D3.1 (K), D4.1 (K), D5.1 (K), D6.1 (K), D7.1 (K), J7.6 (Pin_6), J8.6 (Pin_6), K1.A2, K16.A1, K2.A2
- new net 6m: U17.2, U18.6 (V1), U19.6 (V1)
- new net ANT: J4.1 (In), K1.12, K2.14
- new net BAND0: C3.1, J8.1 (Pin_1), Q3.2 (G), R3.1
- new net BAND1: C4.1, J8.2 (Pin_2), Q1.2 (G), R4.1
- new net BAND2: C9.1, J8.3 (Pin_3), Q4.2 (G), R5.1
- new net BAND3: C10.1, J8.4 (Pin_4), Q5.2 (G), R6.1
- new net BAND4: C11.1, J8.5 (Pin_5), Q6.2 (G), R7.1
- new net BBAND0: K21.A1
- new net BBAND1: K19.A1
- new net BBAND2: K20.A1
- new net BBAND3: K22.A1
- new net BBAND4: K23.A1
- new net NF: U20.2, U21.6 (V1)
- new net RF52: C601.2, C602.2, C603.2, L18.1, L601.1
- new net RF53: C603.1, L40.2, L602.1
- new net RF54: C604.2, C605.2, L19.1, L40.1, L602.2, L603.1
- new net RF55: C605.1, L41.2, L604.1
- new net RF56: C606.2, C607.1, L20.1, L41.1, L604.2, L605.1
- new net RF90: C5.1, J2.1 (In), JP10.1 (A)
- new net RF91: C8.2, J1.1 (In), JP11.1 (A)
- new net RF92: C6.1, J5.1 (In)
- new net RF93: C7.2, J6.1 (In)
- new net RRF100: C700.2, U21.3 (RF2)
- new net RRF101: C701.1, U21.5 (RFC)
- new net RRF205: C14.1, U18.3 (RF2)
- new net RRF211: C20.2, U19.3 (RF2)
- new net RRF250: C27.1, U21.1 (RF1)
- new net RRF50: C600.2, U18.1 (RF1)
- new net RRF51: C601.1, U18.5 (RFC)
- new net RRF57: C607.2, U19.5 (RFC)
- new net RRF58: C608.1, U19.1 (RF1)
- new net RRF90: C5.2, U1.1 (RF1)
- new net RRF91: C6.2, U1.3 (RF2)
- new net RRF92: C8.1, U36.1 (RF1)
- new net RRF93: C7.1, U36.3 (RF2)
- new net RXTX: C13.1, J8.7 (Pin_7), Q7.2 (G), R9.1, U1.6 (V1), U36.6 (V1), U37.2
- new net TX: C12.1, C2.1, D7.2 (A), Q2.2 (G), Q7.1 (D), Q8.2 (G), R2.1, R8.1
- new net _BAND0: D2.2 (A), Q3.1 (D)
- new net _BAND1: D3.2 (A), Q1.1 (D)
- new net _BAND2: D4.2 (A), Q4.1 (D)
- new net _BAND3: D5.2 (A), Q5.1 (D)
- new net _BAND4: D6.2 (A), Q6.1 (D)
- new net ~{6m}: U17.4, U18.4 (V2), U19.4 (V2)
- new net ~{NF}: U20.4, U21.4 (V2)
- new net ~{RXTX}: U1.4 (V2), U36.4 (V2), U37.4
Other:
- note added: "+5V"
- note added: "17T T37-10 11""
- note added: "6m"
- note added: "7T T37-0 4""
- note added: "9T T37-0 5""
- note added: "Added for backwards compatibility with V010/V011 LPF boards and V012 second receiver operation. Only populate if using V012 2nd receiver or with V010/V011 LPF boards."
- note added: "BAND1"
- note added: "BAND2"
- note added: "BAND3"
- note added: "BAND4"
- note added: "BAND_0"
- note added: "BAND_1"
- note added: "Band_2"
- note added: "Band_3"
- note added: "Band_4"
- note added: "Bypass"
- note added: "GND"
- note added: "RXTX"
- note added: "Solder JP10 and JP11 closed if using V012 LPF boards and single receiver"
- note removed: "10M [1001]"
- note removed: "12M [1000]"
- note removed: "15M [0111]"
- note removed: "160M [0001]"
- note removed: "17M [0110]"
- note removed: "20M [0101]"
- note removed: "30M [0100]"
- note removed: "40M [0011]"
- note removed: "60M [0000]"
- note removed: "6M [1010]"
- note removed: "80M [0010]"
- note removed: "All toroids wound on T68-6 cores"
- note removed: "LPFs"
- note removed: "NO FILT [1111]"
- title: K9HZ 100W 11 Band LPF: Filter board -> T41 Mini LPF+BPF+PA
- moved on the sheet: C107, C108, C110, C112, C114, H5, H6, J17, K12, K13, K14, K16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
