File: T41_V012_Mini_Files/T41_V012_Mini_Projects/T41-mini-Main+RF-board-V012/T41-Main+RF-board-V012.kicad_pcb (KiCad board)
At the start: 4 copper layers, 100 x 100 mm, 221 parts, among them J1 IQ_Out, J2 RF_IN, J3 RFControl, J4 12-13.8V, J5 IQ_In, J6 RF_OUT, Q1 BS170, U1 74CBTLV3253DR, U10 SN74LVC1G04DCK, U106 AD8599, U107 OPA2209, U11 Si5351A-B-GT, U12 PE4312, U13 MAR-3SM+, U14 LM7805CT, U15 LM1117T-3.3, U16 LM358B, U17 LM317L, U2 PSA-8A+, U21 MCP23017_SO, U3 PE4312, U4 74CBTLV3253DR, U5 SN74LVC1G04DCK, U6 MC33078, U7 MASWSS0179, U8 MC33078, U9 MASWSS0179, Y1 ECS-TX053-S3, Y2 25MHz

Commit message: Updates
Updates
Parts:
- removed G1, G2, G3, G4, G5, G6, TP14, TP15, TP16, TP17, TP18: TestPoint, Connector_PinHeader_2.54mm:PinHeader_1x01_P2.54mm_Vertical
- removed JP13, JP3: AttenuatorBypass, Connector_PinHeader_2.54mm:PinHeader_1x02_P2.54mm_Vertical
- removed JP15, JP16, JP17: SolderJumper_2_Open, Jumper:SolderJumper-2_P1.3mm_Open_TrianglePad1.0x1.5mm
- removed JP4: CAL isolation, Connector_PinHeader_2.54mm:PinHeader_1x02_P2.54mm_Vertical
- removed JP5: CLK0, Connector_PinHeader_2.54mm:PinHeader_1x02_P2.54mm_Vertical
- removed JP6: CLK1, Connector_PinHeader_2.54mm:PinHeader_1x02_P2.54mm_Vertical
- removed L107: FB, Resistor_SMD:R_1206_3216Metric
- removed R37, R65: 0, Resistor_SMD:R_1206_3216Metric
- removed TR2: ADT2-1T, RF_Mini-Circuits:Mini-Circuits_CD542_H2.84mm
- removed U106: AD8599, Package_SO:SOIC-8_3.9x4.9mm_P1.27mm
- removed U107: OPA2209, Package_SO:SOIC-8_3.9x4.9mm_P1.27mm
- removed U7: MASWSS0179, T41_Library:MASWSS0179-SOT-26
- removed Y2: 25MHz, Crystal:Crystal_SMD_HC49-SD_HandSoldering
- added C100: 0.1uF 50V, Capacitor_SMD:C_1206_3216Metric, F.Cu at (57.0, 96.3)
- added C14: 2.2uF 16V, Capacitor_SMD:C_1206_3216Metric, F.Cu at (23.1, 89.6)
- added C3: 0.1uF 50V, Capacitor_SMD:C_1206_3216Metric, F.Cu at (23.1, 59.4)
- added C74: 0.1uF 50V, Capacitor_SMD:C_1206_3216Metric, F.Cu at (51.4, 56.1)
- added C75: 0.1uF 50V, Capacitor_SMD:C_1206_3216Metric, F.Cu at (51.4, 59.4)
- added C76: 10uF 50V, Capacitor_SMD:C_1206_3216Metric, F.Cu at (51.4, 62.8)
- added C77: 1uF 50V, Capacitor_SMD:C_1206_3216Metric, F.Cu at (51.4, 66.1)
- added C78: 1uF 50V, Capacitor_SMD:C_1206_3216Metric, F.Cu at (51.4, 69.5)
- added C79: 1uF 50V, Capacitor_SMD:C_1206_3216Metric, F.Cu at (51.4, 72.8)
- added C81: 10nF 50V, Capacitor_SMD:C_1206_3216Metric, F.Cu at (51.4, 79.5)
- added C82: 10nF 50V, Capacitor_SMD:C_1206_3216Metric, F.Cu at (51.4, 82.9)
- added C83: 10nF 50V, Capacitor_SMD:C_1206_3216Metric, F.Cu at (51.4, 86.2)
- added C84: 10nF 50V, Capacitor_SMD:C_1206_3216Metric, F.Cu at (51.4, 89.6)
- added C86: 0.1uF 50V, Capacitor_SMD:C_1206_3216Metric, F.Cu at (51.4, 96.3)
- added C87: 0.1uF 50V, Capacitor_SMD:C_1206_3216Metric, F.Cu at (51.4, 99.6)
- added C88: 0.1uF 50V, Capacitor_SMD:C_1206_3216Metric, F.Cu at (57.0, 56.1)
- added C89: 0.1uF 50V, Capacitor_SMD:C_1206_3216Metric, F.Cu at (57.0, 59.4)
- added C90: 0.1uF 50V, Capacitor_SMD:C_1206_3216Metric, F.Cu at (57.0, 62.8)
- added C91: 0.1uF 50V, Capacitor_SMD:C_1206_3216Metric, F.Cu at (57.0, 66.1)
- added C92: 0.1uF 50V, Capacitor_SMD:C_1206_3216Metric, F.Cu at (57.0, 69.5)
- added C93: 10uF 50V, Capacitor_SMD:C_1206_3216Metric, F.Cu at (57.0, 72.8)
- added C94: 10uF 50V, Capacitor_SMD:C_1206_3216Metric, F.Cu at (57.0, 76.2)
- added C95: 180pF 50V, Capacitor_SMD:C_1206_3216Metric, F.Cu at (57.0, 79.5)
- added C96: 105pF 50V, Capacitor_SMD:C_1206_3216Metric, F.Cu at (57.0, 82.9)
- added C97: 180pF 50V, Capacitor_SMD:C_1206_3216Metric, F.Cu at (57.0, 86.2)
- added C98: 105pF 50V, Capacitor_SMD:C_1206_3216Metric, F.Cu at (57.0, 89.6)
- added C99: 0.1uF 50V, Capacitor_SMD:C_1206_3216Metric, F.Cu at (57.0, 92.9)
- added D1: LED, LED_THT:LED_D3.0mm, F.Cu at (55.1, 104.0)
- added D2: LED, LED_THT:LED_D3.0mm, F.Cu at (55.1, 109.5)
- added Encoder1: RotaryEncoder_Switch, Rotary_Encoder:RotaryEncoder_Bourns_Vertical_PEC12R-3x17F-Sxxxx, F.Cu at (61.4, 102.8)
- added Encoder2: RotaryEncoder_Switch, Rotary_Encoder:RotaryEncoder_Bourns_Vertical_PEC12R-3x17F-Sxxxx, F.Cu at (61.4, 118.5)
- added Encoder3: RotaryEncoder_Switch, Rotary_Encoder:RotaryEncoder_Bourns_Vertical_PEC12R-3x17F-Sxxxx, F.Cu at (61.4, 134.3)
- added Encoder4: RotaryEncoder_Switch, Rotary_Encoder:RotaryEncoder_Bourns_Vertical_PEC12R-3x17F-Sxxxx, F.Cu at (61.4, 150.0)
- added H2: EA-T220-38E, T41_KiCad_Library:EAT22038E, F.Cu at (136.6, 99.2)
- added H3: ~, MountingHole:MountingHole_4.3mm_M4_DIN965_Pad, F.Cu at (118.3, 58.9)
- added J10: TX RF Out, Connector_PinHeader_2.54mm:PinHeader_1x02_P2.54mm_Vertical, F.Cu at (120.1, 128.3)
- added J11: PA POWER +12V, Connector_PinHeader_2.54mm:PinHeader_2x06_P2.54mm_Vertical, F.Cu at (118.4, 136.6)
- added J7: Mic_In, T41_KiCad_Library:Jack_3.5mm_STX-3081_Horizontal, F.Cu at (189.2, 88.7)
- added J8: Header, Connector_PinHeader_2.54mm:PinHeader_1x02_P2.54mm_Vertical, F.Cu at (110.9, 128.3)
- added J9: RX RF in, Connector_PinHeader_2.54mm:PinHeader_1x02_P2.54mm_Vertical, F.Cu at (115.5, 128.3)
- added SW1: SW_Omron_B3FS, Button_Switch_SMD:SW_SPST_B3S-1000, F.Cu at (25.8, 105.5)
- added SW10: SW_Omron_B3FS, Button_Switch_SMD:SW_SPST_B3S-1000, F.Cu at (36.9, 130.9)
- added SW11: SW_Omron_B3FS, Button_Switch_SMD:SW_SPST_B3S-1000, F.Cu at (36.9, 139.3)
- added SW12: SW_Omron_B3FS, Button_Switch_SMD:SW_SPST_B3S-1000, F.Cu at (36.9, 147.8)
- added SW13: SW_Omron_B3FS, Button_Switch_SMD:SW_SPST_B3S-1000, F.Cu at (47.9, 105.5)
- added SW14: SW_Omron_B3FS, Button_Switch_SMD:SW_SPST_B3S-1000, F.Cu at (47.9, 114.0)
- added SW15: SW_Omron_B3FS, Button_Switch_SMD:SW_SPST_B3S-1000, F.Cu at (47.9, 122.4)
- added SW16: SW_Omron_B3FS, Button_Switch_SMD:SW_SPST_B3S-1000, F.Cu at (47.9, 130.9)
- added SW17: SW_Omron_B3FS, Button_Switch_SMD:SW_SPST_B3S-1000, F.Cu at (47.9, 139.3)
- added SW18: SW_Omron_B3FS, Button_Switch_SMD:SW_SPST_B3S-1000, F.Cu at (47.9, 147.8)
- added SW2: SW_Omron_B3FS, Button_Switch_SMD:SW_SPST_B3S-1000, F.Cu at (25.8, 114.0)
- added SW3: SW_Omron_B3FS, Button_Switch_SMD:SW_SPST_B3S-1000, F.Cu at (25.8, 122.4)
- added SW4: SW_Omron_B3FS, Button_Switch_SMD:SW_SPST_B3S-1000, F.Cu at (25.8, 130.9)
- added SW5: SW_Omron_B3FS, Button_Switch_SMD:SW_SPST_B3S-1000, F.Cu at (25.8, 139.3)
- added SW6: SW_Omron_B3FS, Button_Switch_SMD:SW_SPST_B3S-1000, F.Cu at (25.8, 147.8)
- added SW7: SW_Omron_B3FS, Button_Switch_SMD:SW_SPST_B3S-1000, F.Cu at (36.9, 105.5)
- added SW8: SW_Omron_B3FS, Button_Switch_SMD:SW_SPST_B3S-1000, F.Cu at (36.9, 114.0)
- added SW9: SW_Omron_B3FS, Button_Switch_SMD:SW_SPST_B3S-1000, F.Cu at (36.9, 122.4)
- added U18: LM358B, Package_SO:SOIC-8_3.9x4.9mm_P1.27mm, F.Cu at (109.6, 77.5)
- added U19: SN74LVC1G04DCK, T41_KiCad_Library:SOT-SC70, F.Cu at (185.4, 93.2)
- added U20: LM317L, Package_SO:SOIC-8_3.9x4.9mm_P1.27mm, F.Cu at (109.6, 84.1)
- C1, C11, C51, C60, C71: value 10uF 50V -> 0.1uF 50V
- C10, C17: value 10nF 50V -> 0.1uF 50V
- C12: value 10uF 50V -> 10uF 16V
- C15: value 1uF 50V -> 10uF 16V
- C16: value 0.1uF 50V -> 2.2uF 16V
- C19: value 180pF 50V -> 0.1uF 50V
- C2: value 1uF 50V -> 470uF 25V; footprint Capacitor_SMD:C_1206_3216Metric -> Capacitor_THT:CP_Radial_D10.0mm_P5.00mm
- C20, C22, C27, C29: value 0.1uF 50V -> 10uF 16V
- C21: value 105pF 50V -> 10uF 16V
- C23: value 0.1uF 50V -> 2.2nF
- C24: value 1uF 50V -> 2.2nF
- C28, C4: value 10nF 50V -> 10uF 16V
- C31, C43, C47, C52: value 0.1uF 50V -> 0.01uF 50V
- C32, C35, C36, C48: value 10uF 50V -> 0.01uF 50V
- C33: value 2.2nF 50V -> 0.01uF 50V
- C34: value 0.2uF 50V -> 0.01uF 50V
- C37, C54: value 10nF 50V -> 0.01uF 50V
- C38: value 0.2uF 50V -> 10uF 50V
- C41, C42: value 10uF 50V -> 10nF 50V
- C44: value 0.2uF 50V -> 0.1uF 50V
- C45, C53, C56, C58, C59, C62: value 0.1uF 50V -> 10uF 50V
- C46: value 2.2nF 50V -> 10uF 50V
- C49: value 0.1uF 50V -> 2.2nF 50V
- C5: value 105pF 50V -> 470uF 25V; footprint Capacitor_SMD:C_1206_3216Metric -> Capacitor_THT:CP_Radial_D10.0mm_P5.00mm
- C50: value 0.2uF 50V -> 2.2nF 50V
- C6: value 0.1uF 50V -> 470uF 25V; footprint Capacitor_SMD:C_1206_3216Metric -> Capacitor_THT:CP_Radial_D10.0mm_P5.00mm
- C64, C65, C66: value 0.1uF 50V -> 0.2uF 50V
- C67: value 10uF 50V -> 0.2uF 50V
- C69: value 470uF 25V -> 0.1uF 50V; footprint Capacitor_THT:CP_Radial_D10.0mm_P5.00mm -> Capacitor_SMD:C_1206_3216Metric
- C8: value 180pF 50V -> 10uF 16V
- C80: value 0.1uF 50V -> 1uF 50V
- C9: value 1uF 50V -> 0.1uF 50V
- H1: value ~ -> EA-T220-38E; footprint MountingHole:MountingHole_3.2mm_M3_Pad -> T41_KiCad_Library:EAT22038E
- H4: value EA-T220-38E -> ~; footprint T41_Library:EAT22038E -> MountingHole:MountingHole_4.3mm_M4_DIN965_Pad
- J1: value IQ_Out -> 12-13.8V; footprint T41_Library:Jack_3.5mm_STX-3081_Horizontal -> TerminalBlock:TerminalBlock_bornier-2_P5.08mm
- J2: value RF_IN -> Display; footprint Connector_Coaxial:SMA_Amphenol_901-144_Vertical -> Connector_PinHeader_2.54mm:PinHeader_2x04_P2.54mm_Vertical
- J3: value RFControl -> PA+BPF+LPF; footprint Connector_IDC:IDC-Header_2x05_P2.54mm_Vertical -> Connector_PinHeader_2.54mm:PinHeader_2x04_P2.54mm_Vertical
- J4: value 12-13.8V -> USBHost; footprint TerminalBlock:TerminalBlock_bornier-2_P5.08mm -> Connector_IDC:IDC-Header_2x03_P2.54mm_Vertical
- J5: value IQ_In -> Keys/PTT; footprint T41_Library:Jack_3.5mm_STX-3081_Horizontal -> Connector_IDC:IDC-Header_2x03_P2.54mm_Vertical
- J6: value RF_OUT -> Rec_Out; footprint Connector_Coaxial:SMA_Amphenol_901-144_Vertical -> T41_KiCad_Library:Jack_3.5mm_STX-3081_Horizontal
- L1, L2, L3: value FB -> 10uH 20%; footprint Resistor_SMD:R_1206_3216Metric -> Inductor_SMD:L_Bourns-SRN6028
- L10, L4: value 1.5uH -> FB
- L11: value 10uH 20% -> 1.5uH; footprint Inductor_SMD:L_Bourns-SRN6028 -> Resistor_SMD:R_1206_3216Metric
- L12, L13: value 10uH 20% -> FB; footprint Inductor_SMD:L_Bourns-SRN6028 -> Resistor_SMD:R_1206_3216Metric
- L6: value FB -> 1.5uH
- R1: value 2k -> 2K2
- R10, R11: value 5k1 -> 10k
- R12: value 10k -> 2k2 1%
- R13: value 2k -> 2k2 1%
- R14: value 36R5 -> 10k 1%
- R15, R19: value 500R -> 10k 1%
- R16, R54: value 100R -> 2k2
- R17: value 5k1 -> 2k2
- R18: value 5k1 -> 10k 1%
- R2, R3: value 5k1 -> 470R
- R20, R21: value 10k -> 10k 1%
- R22: value 100R -> 49R9 1%
- R23, R24: value 10k -> 49R9 1%
- R25: value 10k 1% -> 49R9 1%
- R26: value 2k2 -> 36R5
- R27: value 49R9 1% -> 2.2K
- R29: value 10k 1% -> 500R
- R30: value 10k -> 500R
- R31: value 2k2 1% -> 100k
- R32: value 10k 1% -> 10k
- R33: value 49R9 1% -> 10k
- R34, R49, R50: value 2k2 -> 10k
- R35: value 0 -> 2k2
- R36: value 10k 1% -> 2k2
- R38: value 49R9 1% -> 51k
- R39: value 10k -> 100R
- R40, R42: value 0 -> 100R
- R41: value 10k 1% -> 100R
- R43: value 49R9 1% -> 1k2
- R44: value 10k -> 2k
- R45: value 2k2 1% -> 2k
- R46: value 10k 1% -> 1k8
- R48: value 100k -> 10k
- R5, R6: value 5k1 -> 100R
- R51: value 2k2 -> 330R
- R52: value 2k2 -> 100R
- R53: value 10k -> 2k2
- R55: value 10k -> 5k1
- R56: value 1k8 -> 5k1
- R57: value 330R -> 5k1
- R58: value 51k -> 5k1
- R59: value 1k2 -> 5k1
- R60, R61, R62: value 2k2 -> 5k1
- R63: value 2k2 -> 0
- R7: value 10k -> 2.2K
- R8: value 100R -> 330
- R9: value 10k -> 330
- TR1: value ADT1-1 -> ADT2-1T
- U1: value 74CBTLV3253DR -> LM7805CT; footprint Package_SO:SOIC-16_3.9x9.9mm_P1.27mm -> Package_TO_SOT_THT:TO-220-3_Vertical
- U10: value SN74LVC1G04DCK -> PSA-8A+; footprint T41_Library:SOT-SC70 -> Package_TO_SOT_SMD:SOT-363_SC-70-6
- U11: value Si5351A-B-GT -> 74CBTLV3253DR; footprint Package_SO:MSOP-10_3x3mm_P0.5mm -> Package_SO:SOIC-16_3.9x9.9mm_P1.27mm
- U12: value PE4312 -> MCP23017_SO; footprint T41_Library:PE4312-QFN-20 -> Package_SO:SOIC-28W_7.5x17.9mm_P1.27mm
- U13: value MAR-3SM+ -> 74CBTLV3253DR; footprint T41_Library:Mini-Circuits_WW107 -> Package_SO:SOIC-16_3.9x9.9mm_P1.27mm
- U14: value LM7805CT -> MAR-3SM+; footprint Package_TO_SOT_THT:TO-220-3_Vertical -> T41_KiCad_Library:Mini-Circuits_WW107
- U15: value LM1117T-3.3 -> Si5351A-B-GT; footprint Package_TO_SOT_THT:TO-220-3_Vertical -> Package_SO:MSOP-10_3x3mm_P0.5mm
- U16: value LM358B -> AD8599
- U17: value LM317L -> MASWSS0179; footprint Package_SO:SOIC-8_3.9x4.9mm_P1.27mm -> T41_KiCad_Library:MASWSS0179-SOT-26
- U2: value PSA-8A+ -> LM1117T-3.3; footprint Package_TO_SOT_SMD:SOT-363_SC-70-6 -> Package_TO_SOT_THT:TO-220-3_Vertical
- U21: value MCP23017_SO -> OPA2209; footprint Package_SO:SOIC-28W_7.5x17.9mm_P1.27mm -> Package_SO:SOIC-8_3.9x4.9mm_P1.27mm
- U3: value PE4312 -> Teensy4.1; footprint T41_Library:PE4312-QFN-20 -> T41_KiCad_Library:Teensy41
- U4: value 74CBTLV3253DR -> PCM5102; footprint Package_SO:SOIC-16_3.9x9.9mm_P1.27mm -> Package_SO:TSSOP-20_4.4x6.5mm_P0.65mm
- U5: value SN74LVC1G04DCK -> PCM1808PW; footprint T41_Library:SOT-SC70 -> Package_SO:TSSOP-14_4.4x5mm_P0.65mm
- U6: value MC33078 -> MCP23017_SO; footprint Package_SO:SOIC-8_3.9x4.9mm_P1.27mm -> Package_SO:SOIC-28W_7.5x17.9mm_P1.27mm
- U9: value MASWSS0179 -> MC33078; footprint T41_Library:MASWSS0179-SOT-26 -> Package_SO:SOIC-8_3.9x4.9mm_P1.27mm
- Y1: value ECS-TX053-S3 -> 25MHz; footprint T41_Library:Oscillator_ECS_TXO53_S3 -> Crystal:Crystal_SMD_HC49-SD_HandSoldering
- moved C53 118.4 mm to (40.1, 79.5)
- moved C11 118.1 mm to (23.1, 79.5), turned to 0 degrees
- moved C18 117.2 mm to (28.8, 56.1), turned to 0 degrees
- moved J3 116.3 mm to (170.6, 93.5)
- moved C1 114.0 mm to (23.1, 56.1), turned to 0 degrees
- moved C63 111.9 mm to (45.7, 66.1), turned to 0 degrees
- moved C26 109.6 mm to (28.8, 82.9), turned to 0 degrees
- moved TP3 106.2 mm to (79.8, 145.8)
- moved C47 105.7 mm to (40.1, 59.4), turned to 0 degrees
- moved C66 104.3 mm to (45.7, 76.2), turned to 0 degrees
- moved C58 104.2 mm to (40.1, 96.3)
- moved C8 103.9 mm to (23.1, 69.5), turned to 0 degrees
- moved C70 102.2 mm to (45.7, 89.6), turned to 0 degrees
- moved C68 102.2 mm to (45.7, 82.9), turned to 0 degrees
- moved C7 100.2 mm to (23.1, 66.1), turned to 0 degrees
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Connections:
- C1 pad 1: GND -> +5V
- C1 pad 2: Net-(C1-Pad2) -> GND
- C10 pad 1: GND -> Net-(U2-VO)
- C10 pad 2: Net-(C10-Pad2) -> GND
- C11 pad 1: GND -> +3V3
- C11 pad 2: Net-(C11-Pad2) -> GND
- C12 pad 1: GND -> +3V3
- C12 pad 2: +5V -> GND
- C13 pad 1: GND -> +3V3
- C13 pad 2: +5V -> GND
- C15 pad 1: Net-(C15-Pad1) -> +3V3
- C15 pad 2: Net-(U1-1B2) -> GND
- C16 pad 1: Net-(J2-In) -> Net-(U4-CAPP)
- C16 pad 2: Net-(C16-Pad2) -> Net-(U4-CAPM)
- C17 pad 1: GND -> +5V
- C17 pad 2: Net-(C15-Pad1) -> GND
- C18 pad 1: +5V -> +3V3
- C19 pad 1: GND -> Net-(U4-LDOO)
- C19 pad 2: Net-(U107B-+) -> GND
- C2 pad 1: Net-(C2-Pad1) -> +12V
- C2 pad 2: Net-(U1-1B1) -> GND
- C20 pad 1: GND -> +5V
- C20 pad 2: Net-(C20-Pad2) -> GND
- C21 pad 1: Net-(C21-Pad1) -> +3V3
- C21 pad 2: Net-(C21-Pad2) -> GND
- C22 pad 1: Net-(C22-Pad1) -> Net-(U4-LDOO)
- C22 pad 2: Net-(JP3-A) -> GND
- C23 pad 1: GND -> Net-(C23-Pad1)
- C23 pad 2: Net-(U106C-V+) -> GND
- C24 pad 1: Net-(C24-Pad1) -> GND
- C24 pad 2: Net-(U1-1B3) -> Net-(C24-Pad2)
- C25 pad 1: Net-(U106C-V+) -> +5V
- C26 pad 1: Net-(U107C-V+) -> Net-(U5-VREF)
- C27 pad 1: Net-(U2-OUT) -> Net-(C23-Pad1)
- C27 pad 2: Net-(U1-1A) -> Net-(C27-Pad2)
- C28 pad 1: GND -> Net-(C24-Pad2)
- C28 pad 2: Net-(C24-Pad1) -> Net-(C28-Pad2)
- C29 pad 1: Net-(U3-RF2) -> Net-(U5-VREF)
- C29 pad 2: Net-(JP3-B) -> GND
- C30 pad 2: Net-(U4-VCC) -> +3V3
- C31 pad 1: /ExciterEnable -> Net-(U6-GPB3)
- C32 pad 1: Net-(C32-Pad1) -> Net-(U6-GPB1)
- C32 pad 2: Net-(C32-Pad2) -> GND
- C33 pad 1: Net-(C32-Pad1) -> GND
- C33 pad 2: Net-(U6A--) -> Net-(U6-GPA5)
- C34 pad 1: Net-(U4-1B4) -> Net-(U6-GPB0)
- C35 pad 1: Net-(C35-Pad1) -> GND
- C35 pad 2: Net-(C35-Pad2) -> Net-(U6-GPB4)
- C36 pad 1: Net-(C36-Pad1) -> Net-(U6-GPA2)
- C36 pad 2: Net-(C36-Pad2) -> GND
- C37 pad 1: Net-(C37-Pad1) -> GND
- C37 pad 2: GND -> Net-(U6-GPB5)
- C38 pad 1: Net-(U4-1B1) -> Net-(C38-Pad1)
- C38 pad 2: GND -> /TX Q
- C39 pad 1: Net-(U6A-+) -> Net-(C39-Pad1)
- C39 pad 2: GND -> /TX I
- C4 pad 2: Net-(C2-Pad1) -> +5V
- C40 pad 1: GND -> +5V
- C40 pad 2: Net-(C40-Pad2) -> GND
- C41 pad 1: Net-(C40-Pad2) -> Net-(C41-Pad1)
- C42 pad 2: Net-(C42-Pad2) -> GND
- C43 pad 1: Net-(C43-Pad1) -> GND
- C43 pad 2: Net-(U7-RF1) -> Net-(U6-GPB6)
- C44 pad 1: Net-(U4-1B3) -> Net-(U8C-V+)
- C45 pad 1: Net-(JP13-A) -> Net-(U8A-+)
- C45 pad 2: Net-(U12-RF1) -> GND
- C46 pad 1: Net-(C42-Pad1) -> Net-(U8A-+)
- C46 pad 2: Net-(U8A--) -> GND
- C47 pad 1: Net-(U13-OUT) -> Net-(U6-GPB2)
- C47 pad 2: Net-(U7-RF2) -> GND
- C48 pad 1: Net-(C48-Pad1) -> GND
- C48 pad 2: Net-(C48-Pad2) -> Net-(U6-GPB7)
- C49 pad 1: Net-(U11-XA) -> Net-(C49-Pad1)
- C49 pad 2: Net-(Y1-OUT) -> Net-(U9A--)
- C5 pad 1: Net-(C5-Pad1) -> Net-(U1-VO)
- C5 pad 2: Net-(C5-Pad2) -> GND
- C50 pad 1: Net-(U4-1B2) -> Net-(C50-Pad1)
- C50 pad 2: GND -> Net-(U8A--)
- C51 pad 1: Net-(C51-Pad1) -> GND
- C51 pad 2: Net-(C51-Pad2) -> Net-(U8A-+)
- C52 pad 1: Net-(U11-VDD) -> Net-(U6-GPA3)
- C53 pad 1: Net-(U9-RF1) -> Net-(U8A-+)
- C53 pad 2: Net-(J6-In) -> GND
- C54 pad 1: Net-(C54-Pad1) -> Net-(U6-GPA4)
- C55 pad 1: GND -> Net-(J9-Pin_2)
- C55 pad 2: /ExciterEnable -> Net-(U10-IN)
- C56 pad 1: GND -> Net-(C49-Pad1)
- C56 pad 2: Net-(Q1-G) -> Net-(C56-Pad2)
- C57 pad 1: Net-(U6A-+) -> Net-(C57-Pad1)
- C57 pad 2: GND -> Net-(C57-Pad2)
- C58 pad 1: Net-(U9-RF2) -> Net-(C50-Pad1)
- C58 pad 2: /RFIN -> Net-(C58-Pad2)
- C59 pad 1: GND -> Net-(C59-Pad1)
- C59 pad 2: Net-(U6A-+) -> Net-(C59-Pad2)
- C6 pad 1: GND -> Net-(U2-VO)
- C6 pad 2: Net-(U1-VCC) -> GND
- C60 pad 1: Net-(U6A-+) -> Net-(U9C-V+)
- C61 pad 1: +5V -> GND
- C61 pad 2: GND -> +5V
- C62 pad 1: Net-(U13-IN) -> GND
- C62 pad 2: Net-(U11-CLK2) -> +5V
- C63 pad 1: Net-(JP13-B) -> GND
- C63 pad 2: Net-(U9-RFC) -> +3V3
- C64 pad 1: Net-(U6C-V+) -> Net-(U11-1B4)
- C65 pad 1: Net-(U8C-V+) -> Net-(U11-1B1)
- C66 pad 1: GND -> Net-(U11-1B3)
- C66 pad 2: +3V3 -> GND
- C67 pad 1: Net-(U14-VO) -> Net-(U11-1B2)
- C68 pad 1: Net-(U14-VO) -> Net-(U10-OUT)
- C68 pad 2: GND -> Net-(U13-1A)
- C69 pad 1: +12V -> GND
- C69 pad 2: GND -> Net-(Q1-G)
- C7 pad 1: GND -> +3V3
- C7 pad 2: Net-(U106C-V+) -> GND
- C70 pad 1: +12V -> GND
- C70 pad 2: GND -> Net-(C70-Pad2)
- C71 pad 1: Net-(U15-VO) -> GND
- C71 pad 2: GND -> Net-(U11-VCC)
- C72 pad 1: Net-(U15-VO) -> GND
- C72 pad 2: GND -> /ExciterEnable
- C73 pad 1: GND -> /ExciterEnable
- C73 pad 2: Net-(U16A-+) -> GND
- C8 pad 1: GND -> +3V3
- C8 pad 2: Net-(U107A-+) -> GND
- C80 pad 1: GND -> Net-(C80-Pad1)
- C80 pad 2: +3V3 -> Net-(U13-1B3)
- C85 pad 1: GND -> Net-(U14-IN)
- C85 pad 2: Net-(Y1-VDD) -> Net-(U15-CLK2)
- C9 pad 1: Net-(C10-Pad2) -> Net-(U1-VO)
- C9 pad 2: Net-(U1-1B4) -> GND
- H1 pad 1: GND -> unconnected-(H1-Pad1)
- H4 pad 1: unconnected-(H4-Pad1) -> GND
- J2 pad 1: Net-(J2-In) -> GND
- J3 pad 1: /SCL -> /BAND0
- J3 pad 2: GND -> /BAND1
- J3 pad 3: /SDA -> /BAND2
- J3 pad 4: GND -> /BAND3
- J3 pad 5: GND -> /BAND4
- J3 pad 6: /X Mode -> +5V
- J3 pad 7: /CW on/off -> /RXTX
- J3 pad 8: unconnected-(J3-Pin_8-Pad8) -> GND
- J4 pad 1: Net-(J4-Pin_1) -> unconnected-(J4-Pin_1-Pad1)
- J4 pad 2: GND -> unconnected-(J4-Pin_2-Pad2)
- L1 pad 1: Net-(JP1-A) -> +12P
- L1 pad 2: Net-(U1-VCC) -> +12V
- L10 pad 1: Net-(L10-Pad1) -> +3V3
- L10 pad 2: Net-(U13-OUT) -> Net-(U15-VDD)
- L11 pad 1: Net-(U15-VO) -> Net-(L11-Pad1)
- L11 pad 2: +3V3 -> Net-(U14-OUT)
- L12 pad 1: Net-(U14-VO) -> Net-(U16C-V+)
- L13 pad 1: Net-(J4-Pin_1) -> Net-(U21C-V+)
- L13 pad 2: +12V -> +5V
- L2 pad 1: Net-(U107C-V+) -> Net-(U2-VO)
- L2 pad 2: +5V -> +3V3
- L3 pad 1: Net-(U106C-V+) -> Net-(U1-VO)
- L4 pad 1: Net-(L4-Pad1) -> Net-(U8C-V+)
- L4 pad 2: Net-(U2-OUT) -> +5V
- L5 pad 1: +3V3 -> Net-(U9C-V+)
- L5 pad 2: Net-(U4-VCC) -> +5V
- L6 pad 1: +3V3 -> Net-(L6-Pad1)
- L6 pad 2: Net-(L6-Pad2) -> Net-(U10-OUT)
- L7 pad 1: Net-(Y1-VDD) -> +3V3
- L7 pad 2: +3V3 -> Net-(U11-VCC)
- L8 pad 1: Net-(U6C-V+) -> +3V3
- L8 pad 2: +5V -> Net-(L8-Pad2)
- L9 pad 1: Net-(U8C-V+) -> Net-(JP1-A)
- L9 pad 2: +5V -> Net-(U13-VCC)
- R1 pad 1: Net-(U106A--) -> Net-(U4-XSMT)
- R1 pad 2: Net-(R1-Pad2) -> +3V3
- R10 pad 1: Net-(C11-Pad2) -> Net-(C38-Pad1)
- R10 pad 2: Net-(U107B--) -> Net-(C41-Pad1)
- R11 pad 1: Net-(U107B--) -> Net-(C39-Pad1)
- R11 pad 2: Net-(C21-Pad1) -> Net-(C42-Pad1)
- R12 pad 1: Net-(U1-1~{OE}) -> Net-(C41-Pad1)
- R12 pad 2: GND -> Net-(U9A--)
- R13 pad 1: Net-(U106B--) -> Net-(C42-Pad1)
- R13 pad 2: Net-(R13-Pad2) -> Net-(U8A--)
- R14 pad 1: +5V -> Net-(C41-Pad1)
- R14 pad 2: Net-(L4-Pad1) -> Net-(C49-Pad1)
- R15 pad 1: Net-(JP1-A) -> Net-(C42-Pad1)
- R15 pad 2: Net-(C20-Pad2) -> Net-(C50-Pad1)
- R16 pad 1: Net-(C15-Pad1) -> Net-(U8A-+)
- R16 pad 2: Net-(U106B--) -> Net-(U8C-V+)
- R17 pad 1: Net-(R13-Pad2) -> GND
- R17 pad 2: Net-(C21-Pad2) -> Net-(U8A-+)
- R18 pad 1: Net-(C21-Pad2) -> Net-(C49-Pad1)
- R18 pad 2: Net-(U107B-+) -> Net-(U9B--)
- R19 pad 1: Net-(C20-Pad2) -> Net-(C50-Pad1)
- R19 pad 2: GND -> Net-(U8B--)
- R2 pad 1: Net-(U107A--) -> Net-(C23-Pad1)
- R2 pad 2: Net-(C5-Pad1) -> Net-(U4-OUTL)
- R20 pad 1: Net-(C20-Pad2) -> Net-(U9B--)
- R20 pad 2: Net-(U1-1A) -> Net-(C57-Pad1)
- R21 pad 1: Net-(U106C-V+) -> Net-(U8B--)
- R21 pad 2: Net-(U106B-+) -> Net-(C59-Pad1)
- R22 pad 1: Net-(C24-Pad1) -> Net-(C56-Pad2)
- R22 pad 2: Net-(U106B-+) -> Net-(U11-1B4)
- R23 pad 1: Net-(U106B-+) -> Net-(C57-Pad2)
- R23 pad 2: GND -> Net-(U11-1B1)
- R24 pad 1: GND -> Net-(C58-Pad2)
- R24 pad 2: Net-(U3-Data) -> Net-(U11-1B3)
- R25 pad 1: Net-(C37-Pad1) -> Net-(C59-Pad2)
- R25 pad 2: Net-(C32-Pad1) -> Net-(U11-1B2)
- R26 pad 1: Net-(C40-Pad2) -> +5V
- R26 pad 2: Net-(L6-Pad2) -> Net-(L6-Pad1)
- R27 pad 1: Net-(C32-Pad2) -> +3V3
- R27 pad 2: Net-(U4-1B4) -> Net-(U12-~{RESET})
- R28 pad 1: Net-(U3-C16) -> Net-(Q1-G)
- R28 pad 2: /RC16 -> /RXTX
- R29 pad 1: Net-(U6B--) -> Net-(JP1-A)
- R29 pad 2: Net-(C36-Pad1) -> Net-(C70-Pad2)
- R3 pad 1: Net-(C1-Pad2) -> Net-(C24-Pad2)
- R3 pad 2: Net-(U107A--) -> Net-(U4-OUTR)
- R30 pad 1: Net-(C35-Pad1) -> Net-(C70-Pad2)
- R30 pad 2: Net-(C37-Pad1) -> GND
- R31 pad 1: Net-(C37-Pad1) -> Net-(Q1-G)
- R31 pad 2: Net-(U6A--) -> GND
- R32 pad 1: Net-(C32-Pad1) -> Net-(C70-Pad2)
- R32 pad 2: Net-(U6B--) -> Net-(U13-1A)
- R33 pad 1: Net-(C36-Pad2) -> /ExciterEnable
- R33 pad 2: Net-(U4-1B1) -> +3V3
- R34 pad 1: GND -> Net-(U13-1~{OE})
- R34 pad 2: Net-(C40-Pad2) -> GND
- R35 pad 1: Net-(U4-S1) -> Net-(C75-Pad2)
- R35 pad 2: Net-(JP5-A) -> Net-(L8-Pad2)
- R36 pad 1: Net-(C54-Pad1) -> GND
- R36 pad 2: Net-(C42-Pad1) -> Net-(C75-Pad2)
- R38 pad 1: Net-(C42-Pad2) -> Net-(U18A-+)
- R38 pad 2: Net-(U4-1B3) -> /CW
- R39 pad 1: /ExciterEnable -> Net-(C79-Pad1)
- R39 pad 2: +3V3 -> Net-(U16B--)
- R4 pad 1: Net-(C2-Pad1) -> /CLK
- R4 pad 2: Net-(U106A--) -> Net-(U5-SCKI)
- R40 pad 1: Net-(U1-S1) -> Net-(C80-Pad1)
- R40 pad 2: Net-(JP5-A) -> Net-(U16B-+)
- R41 pad 1: Net-(U8B--) -> Net-(C77-Pad1)
- R41 pad 2: Net-(C51-Pad1) -> Net-(U16A--)
- R42 pad 1: Net-(U1-S0) -> Net-(C78-Pad1)
- R42 pad 2: Net-(JP6-A) -> Net-(U16A-+)
- R43 pad 1: Net-(C51-Pad2) -> Net-(U18A--)
- R43 pad 2: Net-(U4-1B2) -> GND
- R44 pad 1: Net-(C48-Pad1) -> Net-(U16A--)
- R44 pad 2: Net-(C54-Pad1) -> Net-(R44-Pad2)
- R45 pad 1: Net-(C54-Pad1) -> Net-(U16B--)
- R45 pad 2: Net-(U8A--) -> Net-(R45-Pad2)
- R46 pad 1: Net-(C42-Pad1) -> Net-(U20-ADJ)
- R46 pad 2: Net-(U8B--) -> Net-(U18A--)
- R47 pad 1: Net-(Q1-G) -> Net-(U16C-V+)
- R47 pad 2: /RXTX -> Net-(U16A-+)
- R48 pad 1: Net-(Q1-G) -> Net-(U16A-+)
- R49 pad 1: /SCL -> Net-(U16C-V+)
- R49 pad 2: +3V3 -> Net-(U16B-+)
- R5 pad 1: Net-(R1-Pad2) -> /LRCK
- R5 pad 2: Net-(C5-Pad2) -> Net-(U5-LRCK)
- R50 pad 1: Net-(U6A-+) -> Net-(U16B-+)
- R50 pad 2: Net-(U8C-V+) -> GND
- R51 pad 1: /SDA -> Net-(R51-Pad1)
- R51 pad 2: +3V3 -> Net-(U20-ADJ)
- R52 pad 1: GND -> Net-(L11-Pad1)
- R52 pad 2: Net-(U6A-+) -> Net-(R51-Pad1)
- R53 pad 1: GND -> /SDA
- R53 pad 2: Net-(U12-Data) -> +3V3
- R54 pad 1: Net-(L10-Pad1) -> /SCL
- R54 pad 2: Net-(R54-Pad2) -> +3V3
- R55 pad 1: Net-(U12-C16) -> Net-(R44-Pad2)
- R55 pad 2: /TC16 -> Net-(C96-Pad2)
- R56 pad 1: Net-(U17-ADJ) -> Net-(R45-Pad2)
- R56 pad 2: Net-(U16A--) -> Net-(C98-Pad2)
- R57 pad 1: Net-(R54-Pad2) -> Net-(C93-Pad2)
- R57 pad 2: Net-(U17-ADJ) -> Net-(U21A--)
- R58 pad 1: Net-(U16A-+) -> Net-(C96-Pad2)
- R58 pad 2: /CW on/off -> Net-(U21A-+)
- R59 pad 1: Net-(U16A--) -> Net-(C94-Pad2)
- R59 pad 2: GND -> Net-(U21B--)
- R6 pad 1: Net-(C5-Pad2) -> /BCK
- R6 pad 2: Net-(U107A-+) -> Net-(U5-BCK)
- R60 pad 1: Net-(JP15-B) -> Net-(C98-Pad2)
- R60 pad 2: +3V3 -> Net-(U21B-+)
- R61 pad 1: Net-(JP16-B) -> Net-(U21A--)
- R61 pad 2: +3V3 -> Net-(C96-Pad1)
- R62 pad 1: Net-(U21-~{RESET}) -> Net-(U21B--)
- R62 pad 2: +3V3 -> Net-(C98-Pad1)
- R63 pad 1: Net-(JP17-B) -> Net-(C96-Pad1)
- R63 pad 2: +3V3 -> /RX Q
- R64 pad 1: Net-(C5-Pad1) -> Net-(C98-Pad1)
- R64 pad 2: /Q_out -> /RX I
- R7 pad 1: Net-(U106C-V+) -> +3V3
- R7 pad 2: Net-(U106A-+) -> Net-(U6-~{RESET})
- R8 pad 1: Net-(C10-Pad2) -> GND
- R8 pad 2: Net-(U106A-+) -> Net-(D1-K)
- R9 pad 1: Net-(U106A-+) -> GND
- R9 pad 2: GND -> Net-(D2-K)
- TP1 pad 1: Net-(C2-Pad1) -> +5V
- TP10 pad 1: Net-(U4-1B1) -> Net-(C79-Pad1)
- TP11 pad 1: Net-(U4-1B3) -> Net-(C77-Pad1)
- TP12 pad 1: Net-(U4-2A) -> /RX Q
- TP13 pad 1: Net-(U4-1B2) -> /RX I
- TP2 pad 1: /Q_out -> +3V3
- TP3 pad 1: /I_out -> Net-(U11-1B4)
- TP4 pad 1: Net-(C22-Pad1) -> Net-(U11-1B1)
- TP5 pad 1: Net-(C15-Pad1) -> Net-(U11-1B3)
- TP6 pad 1: Net-(U1-1A) -> Net-(U11-1B2)
- TP7 pad 1: Net-(U4-1B4) -> Net-(U13-1A)
- TP8 pad 1: Net-(U4-1A) -> Net-(U11-1A)
- TP9 pad 1: Net-(C35-Pad2) -> Net-(U11-2A)
- TR1 pad 2: (no net) -> unconnected-(TR1-Pad2)
- TR1 pad 3: Net-(C16-Pad2) -> Net-(C86-Pad1)
- TR1 pad 4: Net-(C22-Pad1) -> Net-(U11-2A)
- TR1 pad 5: (no net) -> Net-(C75-Pad2)
- TR1 pad 6: GND -> Net-(U11-1A)
- U1 pad 1: Net-(U1-1~{OE}) -> +12V
- U1 pad 2: Net-(U1-S1) -> GND
- U1 pad 3: Net-(U1-1B4) -> Net-(U1-VO)
- U10 pad 1: (no net) -> GND
- U10 pad 2: /Cal -> GND
- U10 pad 3: GND -> Net-(U10-IN)
- U10 pad 4: Net-(U9-V1) -> GND
- U10 pad 5: +3V3 -> GND
- U11 pad 1: Net-(U11-VDD) -> /ExciterEnable
- U11 pad 10: Net-(JP5-B) -> Net-(U11-1B4)
- U11 pad 2: Net-(U11-XA) -> Net-(U11-S1)
- U11 pad 3: Net-(U11-XB) -> Net-(U11-1B4)
- U11 pad 4: /SCL -> Net-(U11-1B3)
- U11 pad 5: /SDA -> Net-(U11-1B2)
- U11 pad 6: Net-(U11-CLK2) -> Net-(U11-1B1)
- U11 pad 7: Net-(U11-VDD) -> Net-(U11-1A)
- U11 pad 9: Net-(JP6-B) -> Net-(U11-2A)
- U12 pad 1: Net-(U12-C16) -> Net-(U12-GPB0)
- U12 pad 11: GND -> unconnected-(U12-NC-Pad11)
- U12 pad 12: GND -> /SCL1
- U12 pad 13: GND -> /SDA1
- U12 pad 14: Net-(JP13-B) -> unconnected-(U12-NC-Pad14)
- U12 pad 15: /TC8 -> GND
- U12 pad 16: /TC4 -> GND
- U12 pad 17: /TC2 -> GND
- U12 pad 18: GND -> Net-(U12-~{RESET})
- U12 pad 19: /TC1 -> unconnected-(U12-INTB-Pad19)
- U12 pad 2: Net-(U12-RF1) -> Net-(U12-GPB1)
- U12 pad 20: /TC0.5 -> /INT1
- U12 pad 21: GND -> Net-(U12-GPA0)
- U12 pad 3: Net-(U12-Data) -> Net-(U12-GPB2)
- U12 pad 4: unconnected-(U12-Clock-Pad4) -> Net-(U12-GPB3)
- U12 pad 5: +3V3 -> Net-(U12-GPB4)
- U12 pad 6: +3V3 -> Net-(U12-GPB5)
- U12 pad 7: GND -> Net-(U12-GPB6)
- U12 pad 8: GND -> Net-(U12-GPB7)
- U13 pad 1: Net-(U13-IN) -> Net-(U13-1~{OE})
- U13 pad 2: GND -> Net-(U11-S1)
- U13 pad 3: Net-(U13-OUT) -> Net-(U13-1B4)
- U13 pad 4: GND -> Net-(U13-1B3)
- U14 pad 1: +12V -> Net-(U14-IN)
- U14 pad 3: Net-(U14-VO) -> Net-(U14-OUT)
- U15 pad 1: GND -> Net-(U15-VDD)
- U15 pad 2: Net-(U15-VO) -> Net-(U15-XA)
- U15 pad 3: +12V -> Net-(U15-XB)
- U16 pad 1: Net-(U17-ADJ) -> Net-(R44-Pad2)
- U16 pad 5: (no net) -> Net-(U16B-+)
- U16 pad 6: (no net) -> Net-(U16B--)
- U16 pad 7: (no net) -> Net-(R45-Pad2)
- U16 pad 8: +12V -> Net-(U16C-V+)
- U17 pad 1: +12V -> Net-(U17-RF1)
- U17 pad 2: Net-(R54-Pad2) -> GND
- U17 pad 3: Net-(R54-Pad2) -> Net-(U17-RF2)
- U17 pad 4: Net-(U17-ADJ) -> Net-(U17-V2)
- U17 pad 5: unconnected-(U17-NC-Pad5) -> Net-(J10-Pin_1)
- U17 pad 6: Net-(R54-Pad2) -> /TX Mode
- U2 pad 2: GND -> Net-(U2-VO)
- U2 pad 3: Net-(JP3-B) -> +12V
- U21 pad 1: /TC0.5 -> Net-(C96-Pad1)
- U21 pad 2: /TC1 -> Net-(U21A--)
- U21 pad 3: /TC2 -> Net-(U21A-+)
- U21 pad 4: /TC4 -> GND
- U21 pad 5: /TC8 -> Net-(U21B-+)
- U21 pad 6: /TC16 -> Net-(U21B--)
- U21 pad 7: unconnected-(U21-GPB6-Pad7) -> Net-(C98-Pad1)
- U21 pad 8: unconnected-(U21-GPB7-Pad8) -> Net-(U21C-V+)
- U3 pad 1: Net-(U3-C16) -> GND
- U3 pad 10: GND -> /Rx
- U3 pad 11: GND -> unconnected-(U3-9_OUT1C-Pad11)
- U3 pad 12: GND -> /C/S
- U3 pad 13: GND -> /MOSI
- U3 pad 14: Net-(U3-RF2) -> /MISO
- U3 pad 15: /RC8 -> unconnected-(U3-3V3-Pad15)
- U3 pad 16: /RC4 -> unconnected-(U3-24_A10_TX6_SCL2-Pad16)
- U3 pad 17: /RC2 -> unconnected-(U3-25_A11_RX6_SDA2-Pad17)
- U3 pad 18: GND -> unconnected-(U3-26_A12_MOSI1-Pad18)
- U3 pad 19: /RC1 -> /BAND0
- U3 pad 2: Net-(JP3-A) -> unconnected-(U3-0_RX1_CRX2_CS1-Pad2)
- U3 pad 20: /RC0.5 -> /BAND1
- U3 pad 21: GND -> /BAND2
- U3 pad 3: Net-(U3-Data) -> unconnected-(U3-1_TX1_CTX2_MISO1-Pad3)
- U3 pad 5: +3V3 -> unconnected-(U3-3_LRCLK2-Pad5)
- U3 pad 6: +3V3 -> unconnected-(U3-4_BCLK2-Pad6)
- U3 pad 7: GND -> unconnected-(U3-5_IN2-Pad7)
- U3 pad 8: GND -> /ADC_IN
- U3 pad 9: +3V3 -> /Tx
- U4 pad 1: /ExciterEnable -> +3V3
- U4 pad 10: Net-(U4-1B4) -> GND
- U4 pad 11: Net-(U4-1B3) -> GND
- U4 pad 12: Net-(U4-1B2) -> GND
- U4 pad 13: Net-(U4-1B1) -> /BCK
- U4 pad 14: Net-(U4-S0) -> /DAUDIO_OUT
- U4 pad 15: /ExciterEnable -> /LRCK
- U4 pad 16: Net-(U4-VCC) -> GND
- U4 pad 2: Net-(U4-S1) -> Net-(U4-CAPP)
- U4 pad 3: Net-(U4-1B4) -> GND
- U4 pad 4: Net-(U4-1B3) -> Net-(U4-CAPM)
- U4 pad 5: Net-(U4-1B2) -> Net-(U4-VNEG)
- U4 pad 6: Net-(U4-1B1) -> Net-(U4-OUTL)
- U4 pad 7: Net-(U4-1A) -> Net-(U4-OUTR)
- U4 pad 8: GND -> +3V3
- U4 pad 9: Net-(U4-2A) -> GND
- U5 pad 1: (no net) -> Net-(U5-VREF)
- U5 pad 2: /X Mode -> GND
- U5 pad 3: GND -> +5V
- U5 pad 4: Net-(U7-V2) -> +3V3
- U5 pad 5: +3V3 -> GND
- U6 pad 1: Net-(C32-Pad1) -> Net-(U6-GPB0)
- U6 pad 2: Net-(U6A--) -> Net-(U6-GPB1)
- U6 pad 3: Net-(U6A-+) -> Net-(U6-GPB2)
- U6 pad 4: GND -> Net-(U6-GPB3)
- U6 pad 5: Net-(U6A-+) -> Net-(U6-GPB4)
- U6 pad 6: Net-(U6B--) -> Net-(U6-GPB5)
- U6 pad 7: Net-(C36-Pad1) -> Net-(U6-GPB6)
- U6 pad 8: Net-(U6C-V+) -> Net-(U6-GPB7)
- U8 pad 1: Net-(C42-Pad1) -> Net-(C50-Pad1)
- U8 pad 3: Net-(U6A-+) -> Net-(U8A-+)
- U8 pad 5: Net-(U6A-+) -> Net-(U8A-+)
- U8 pad 7: Net-(C51-Pad1) -> Net-(C59-Pad1)
- U9 pad 1: Net-(U9-RF1) -> Net-(C49-Pad1)
- U9 pad 2: GND -> Net-(U9A--)
- U9 pad 3: Net-(U9-RF2) -> Net-(U8A-+)
- U9 pad 4: /Cal -> GND
- U9 pad 5: Net-(U9-RFC) -> Net-(U8A-+)
- U9 pad 6: Net-(U9-V1) -> Net-(U9B--)
- Y1 pad 1: GND -> Net-(U15-XA)
- Y1 pad 2: (no net) -> Net-(U15-XB)
Routing:
- net +3V3: track 343.8 -> 0.00 mm, vias 12 -> 0
- net +5V: track 232.4 -> 0.00 mm, vias 6 -> 0
- net /TC16: track 146.5 -> 0.00 mm, vias 2 -> 0
- net /TC8: track 132.7 -> 0.00 mm, vias 2 -> 0
- net /RFIN: track 131.7 -> 0.00 mm, vias 1 -> 0
- net /TC4: track 131.6 -> 0.00 mm, vias 2 -> 0
- net /Cal: track 130.2 -> 0.00 mm, vias 1 -> 0
- net /TC2: track 129.4 -> 0.00 mm, vias 2 -> 0
- net /TC1: track 125.9 -> 0.00 mm, vias 2 -> 0
- net /TC0.5: track 123.5 -> 0.00 mm, vias 2 -> 0
- net /X Mode: track 118.5 -> 0.00 mm, vias 3 -> 0
- net +12V: track 98.9 -> 0.00 mm, vias 3 -> 0
- net /SCL: track 85.7 -> 0.00 mm, vias 2 -> 0
- net /CW on/off: track 80.6 -> 0.00 mm, vias 1 -> 0
- net /SDA: track 78.1 -> 0.00 mm, vias 2 -> 0
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- removed copper zone on B.Cu, net GND
- removed copper zone on F.Cu, net GND
- removed copper zone on In1.Cu, net GND
- removed copper zone on In2.Cu, net GND
Other:
- board outline removed
- copper layers 4 -> 2
- board text removed: "+12V"
- board text removed: "3V3"
- board text removed: "5V"
- board text removed: "A0"
- board text removed: "A1"
- board text removed: "A2"
- board text removed: "ADDRESS SELECT"
- board text removed: "Anti-alias filters"
- board text removed: "Auto cal switch"
- board text removed: "CAL Isolation"
- board text removed: "CLK0 jumper"
- board text removed: "CLK1 jumper"
- board text removed: "CW envelope shaping"
- board text removed: "Clock generation"
- board text removed: "GND"
- board text removed: "Gain control bypass"
- board text removed: "Input RF amp"
- board text removed: "Mode select"
- board text removed: "Phasing op amps"
- board text removed: "Power"
- board text removed: "Quadrature sampling"
- board text removed: "Quadrature sampling detector"
- board text removed: "RF CONTROL"
- board text removed: "RF OUT"
- board text removed: "RX RF gain control"
- board text removed: "Receive IQ OUT"
- board text removed: "Receive RF IN"
- board text removed: "T41 RF Board: V12.07 Designed by AC8GY/K9HZ Layout by KI3P 4 layer, 2025/01/16"
- board text removed: "TCXO upgrade"
- board text removed: "TX gain control"
- board text removed: "Transmit IQ IN"
- board text removed: "exciter"
