File: T41_V012_Mini_Files/T41_V012_Mini_Projects/T41-mini-Main+RF-board-V012/T41-Main+RF-board-V012.kicad_sch (KiCad schematic)
At the start: 206 parts, among them J1 TX RF Out, J13 Header, J14 Rec_Out, J16 Mic_In, J2 RX RF in, J24 USBHost, J3 Display, J4 12-13.8V, J5 PA+LPF, J9 Keys/PTT, Q1 BS170, U1 74CBTLV3253DR, U10 PCM5102, U106 AD8599, U107 OPA2209, U11 Si5351A-B-GT, U12 Teensy4.1, U13 MAR-3SM+, U16 LM358B, U17 LM317L, U18 Teensy_Audio_Adaptor, U2 LM7805CT, U3 LM1117T-3.3, U4 74CBTLV3253DR, U5 SN74LVC1G04DCK, U6 MC33078, U7 MASWSS0179, U8 MC33078, U9 PCM1808PW, Y2 25MHz

Commit message: T41 Mini Update
T41 Mini Update
Parts:
- added C30, C55, C61, C63: 0.1uF 50V, Capacitor_SMD:C_1206_3216Metric, symbol Device:C
- added C31, C32, C33, C34, C35, C36, C37, C43, C47, C48, C52, C54: 0.01uF 50V, Capacitor_SMD:C_1206_3216Metric, symbol Device:C
- added C62: 10uF 50V, Capacitor_SMD:C_1206_3216Metric, symbol Device:C
- added D1, D2: LED, symbol Device:LED
- added Encoder1, Encoder2, Encoder3, Encoder4: RotaryEncoder_Switch, symbol Device:RotaryEncoder_Switch
- added L6: 1.5uH, Resistor_SMD:R_1206_3216Metric, symbol Device:L
- added R26: 36R5, Resistor_SMD:R_1206_3216Metric, symbol Device:R
- added R27, R7: 2.2K, Resistor_SMD:R_1206_3216Metric, symbol Device:R
- added R8, R9: 330, Resistor_SMD:R_1206_3216Metric, symbol Device:R
- added SW1, SW10, SW11, SW12, SW13, SW14, SW15, SW16, SW17, SW18, SW2, SW3, SW4, SW5, SW6, SW7, SW8, SW9: SW_Omron_B3FS, symbol Switch:SW_Omron_B3FS
- added U10: PSA-8A+, Package_TO_SOT_SMD:SOT-363_SC-70-6, symbol T41_Library:PSA-8A+
- added U12, U6: MCP23017_SO, Package_SO:SOIC-28W_7.5x17.9mm_P1.27mm, symbol Interface_Expansion:MCP23017_SO
- renumbered C79 to C1, C22 to C10, C18 to C100, C66 to C11, C67 to C12, C68 to C13, C69 to C14, C70 to C15, C29 to C16, C27 to C17, C29 to C18, C71 to C19, C3 to C2, C45 to C20, C49 to C21, C72 to C22, C74 to C23, C75 to C24, C78 to C25, C63 to C26, C76 to C27, C77 to C28, C27 to C29, C35 to C38, C48 to C39, C80 to C4, C61 to C40, C37 to C41, C54 to C42, C65 to C44, C39 to C45, C57 to C46, C33 to C49, C12 to C5, C46 to C50, C59 to C51, C60 to C53, C32 to C56, C36 to C57, C42 to C58, C51 to C59, C13 to C6, C64 to C60, C34 to C64, C38 to C65, C44 to C66, C50 to C67, C16 to C68, C56 to C69, C53 to C7, C20 to C70, C30 to C71, C55 to C72, C31 to C73, C6 to C74, C40 to C75, C41 to C76, C2 to C77, C9 to C78, C15 to C79, C58 to C8, C24 to C80, C4 to C81, C10 to C82, C17 to C83, C28 to C84, C62 to C85, C43 to C86, C47 to C87, C73 to C88, C52 to C89, C14 to C9, C7 to C90, C25 to C91, C23 to C92, C1 to C93, C11 to C94, C8 to C95, C5 to C96, C19 to C97, C21 to C98, C26 to C99, H7 to H1, H8 to H2, H1 to H3, H2 to H5, H3 to H6, J4 to J1, J1 to J10, J3 to J2, J5 to J3, J24 to J4, J9 to J5, J14 to J6, J16 to J7, J13 to J8, J2 to J9, L13 to L1, L107 to L10, L10 to L11, L3 to L12, L2 to L13, L4 to L2, L7 to L3, L9 to L4, L8 to L5, L5 to L7, L6 to L8, L1 to L9, R14 to R1, R30 to R10, R44 to R11, R31 to R12, R45 to R13, R25 to R14, R36 to R15, R50 to R16, R52 to R17, R32 to R18, R46 to R19, R37 to R2, R29 to R20, R41 to R21, R27 to R22, R33 to R23, R38 to R24, R43 to R25, R47 to R28, R15 to R29, R40 to R3, R19 to R30, R48 to R31, R20 to R32, R39 to R33, R12 to R34, R26 to R35, R34 to R36, R73 to R37, R58 to R38, R16 to R39, R24 to R4, R22 to R40, R4 to R41, R8 to R42, R59 to R43, R1 to R44, R13 to R45, R56 to R46, R7 to R47, R9 to R48, R21 to R49, R28 to R5, R23 to R50, R57 to R51, R54 to R52, R51 to R53, R49 to R54, R5 to R55, R17 to R56, R3 to R57, R6 to R58, R10 to R59, R35 to R6, R18 to R60, R2 to R61, R11 to R62, R64 to R63, R65 to R64, TP4 to TP1, TP5 to TP10, TP1 to TP11, TP2 to TP12, TP3 to TP13, TP9 to TP2, TP7 to TP3, TP10 to TP4, TP11 to TP5, TP13 to TP6, TP6 to TP7, TP12 to TP9, TR2 to TR1, U2 to U1, U4 to U11, U1 to U13, U13 to U14, U11 to U15, U106 to U16, U7 to U17, U16 to U18, U5 to U19, U3 to U2, U17 to U20, U107 to U21, U12 to U3, U10 to U4, U9 to U5, U18 to U7, U6 to U9, Y2 to Y1
Connections:
- net +3V3: now also C30.2, C63.2, R27.1, R7.1, U12.9 (VDD), U6.17 (A2), U6.9 (VDD)
- net +5V: now also C61.2, C62.2, R26.1
- net GND: now also C30.1, C31.2, C32.2, C33.1, C34.2, C35.1, C36.2, C37.1, C43.1, C47.2, C48.1, C52.2, C54.2, C61.1, C62.1, C63.1, Encoder1.C, Encoder1.S2, Encoder2.C, Encoder2.S2, Encoder3.C, Encoder3.S2, Encoder4.C, Encoder4.S2, R8.1, R9.1, SW1.2, SW10.2, SW11.2, SW12.2, SW13.2, SW14.2, SW15.2, SW16.2, SW17.2, SW18.2, SW2.2, SW3.2, SW4.2, SW5.2, SW6.2, SW7.2, SW8.2, SW9.2, U10.1 (GND), U10.2 (GND), U10.4 (GND), U10.5 (GND), U12.10 (VSS), U12.15 (A0), U12.16 (A1), U12.17 (A2), U6.10 (VSS), U6.15 (A0), U6.16 (A1)
- net INT1: now also U12.20 (INTA)
- net INT2: now also U6.20 (INTA)
- net SCL1: now also U12.12 (SCK), U6.12 (SCK)
- net SCLK: now also J2.8 (Pin_8)
- net SDA1: now also U12.13 (SDA), U6.13 (SDA)
- net at C68.1: now also L6.2, U10.6 (OUT); no longer J9.2 (Pin_2)
- net BAND0 (80m) renamed BAND3
- net BAND3: now also J3.4 (Pin_4); no longer J3.5 (Pin_5)
- net BAND1 (40m) renamed BAND4
- net BAND4: now also J3.5 (Pin_5); no longer J3.4 (Pin_4)
- net BAND2 (20m) renamed BAND1
- net BAND1: now also J3.2 (Pin_2); no longer J3.3 (Pin_3)
- net BAND3 (15m) renamed BAND2
- net BAND2: now also J3.3 (Pin_3); no longer J3.2 (Pin_2)
- net BAND4 (10m) renamed BAND0
- new net: SW16.1, U12.8 (GPB7)
- new net: SW8.1, U12.28 (GPA7)
- new net: C32.1, Encoder1.B, U6.2 (GPB1)
- new net: L6.1, R26.2
- new net: SW14.1, U12.6 (GPB5)
- new net: C34.1, Encoder1.A, U6.1 (GPB0)
- new net: C36.1, Encoder1.S1, U6.23 (GPA2)
- new net: C37.2, Encoder3.B, U6.6 (GPB5)
- new net: C31.1, Encoder2.B, U6.4 (GPB3)
- new net: C48.2, Encoder4.B, U6.8 (GPB7)
- new net: SW1.1, U12.21 (GPA0)
- new net: R7.2, U6.18 (~{RESET})
- new net: C55.1, J9.2 (Pin_2)
- new net: SW9.1, U12.1 (GPB0)
- new net: SW17.1, U6.21 (GPA0)
- new net: SW18.1, U6.22 (GPA1)
- new net: C52.1, Encoder2.S1, U6.24 (GPA3)
- new net: C54.1, Encoder4.S1, U6.25 (GPA4)
- new net: C33.2, Encoder3.S1, U6.26 (GPA5)
- new net: D2.2 (A), U6.27 (GPA6)
- new net: D1.2 (A), U6.28 (GPA7)
- new net: C47.1, Encoder2.A, U6.3 (GPB2)
- new net: C35.2, Encoder3.A, U6.5 (GPB4)
- new net: C43.2, Encoder4.A, U6.7 (GPB6)
- new net: D1.1 (K), R8.2
- new net: C55.2, U10.3 (IN)
- new net: D2.1 (K), R9.2
- new net: SW3.1, U12.23 (GPA2)
- new net: R27.2, U12.18 (~{RESET})
- new net: SW10.1, U12.2 (GPB1)
- new net: SW2.1, U12.22 (GPA1)
- new net: SW4.1, U12.24 (GPA3)
- new net: SW5.1, U12.25 (GPA4)
- new net: SW6.1, U12.26 (GPA5)
- new net: SW7.1, U12.27 (GPA6)
- new net: SW11.1, U12.3 (GPB2)
- new net: SW12.1, U12.4 (GPB3)
- new net: SW13.1, U12.5 (GPB4)
- new net: SW15.1, U12.7 (GPB6)
Other:
- note added: "BAND0"
- note added: "BAND1"
- note added: "BAND2"
- note added: "BAND3"
- note added: "BAND4"
- note removed: "10M"
- note removed: "15M"
- note removed: "20M"
- note removed: "40M"
- note removed: "80M"
- note removed: "Front Panel"
- moved on the sheet: C1, C10, C100, C11, C12, C13, C14, C15, C16, C17, C18, C19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

Commit message: Updates
Updates
Parts:
- added J11: PA POWER +12V, Connector_PinHeader_2.54mm:PinHeader_2x06_P2.54mm_Vertical, symbol Connector_Generic:Conn_02x06_Odd_Even
- D1, D2: footprint (none) -> LED_THT:LED_D3.0mm
- Encoder1, Encoder2, Encoder3, Encoder4: footprint (none) -> Rotary_Encoder:RotaryEncoder_Bourns_Vertical_PEC12R-3x17F-Sxxxx
- H1, H2: footprint EAT22038E -> T41_KiCad_Library:EAT22038E
- J10, J9: footprint (none) -> Connector_PinHeader_2.54mm:PinHeader_1x02_P2.54mm_Vertical
- J2: footprint (none) -> Connector_PinHeader_2.54mm:PinHeader_2x04_P2.54mm_Vertical
- J3: value PA+LPF -> PA+BPF+LPF; footprint (none) -> Connector_PinHeader_2.54mm:PinHeader_2x04_P2.54mm_Vertical
- J6, J7: footprint T41_Library:Jack_3.5mm_STX-3081_Horizontal -> T41_KiCad_Library:Jack_3.5mm_STX-3081_Horizontal
- SW1, SW10, SW11, SW12, SW13, SW14, SW15, SW16, SW17, SW18, SW2, SW3, SW4, SW5, SW6, SW7, SW8, SW9: footprint (none) -> Button_Switch_SMD:SW_SPST_B3S-1000
- U14: footprint T41_Library:Mini-Circuits_WW107 -> T41_KiCad_Library:Mini-Circuits_WW107
- U17: footprint T41_Library:MASWSS0179-SOT-26 -> T41_KiCad_Library:MASWSS0179-SOT-26
- U19: footprint T41_Library:SOT-SC70 -> T41_KiCad_Library:SOT-SC70
- U3: footprint T41_Library:Teensy41 -> T41_KiCad_Library:Teensy41
Connections:
- net Xmit Mode is gone; now on net TX Mode: U3.26 (34_RX8)
- net +12V: no longer J3.6 (Pin_6)
- net +5V: now also J3.6 (Pin_6)
- net ADC_IN: now also U3.8 (6_OUT1D)
- net GND: now also Encoder1.SH, Encoder2.SH, Encoder3.SH, Encoder4.SH, J11.10 (Pin_10), J11.11 (Pin_11), J11.12 (Pin_12), J11.7 (Pin_7), J11.8 (Pin_8), J11.9 (Pin_9)
- net SCL: no longer R53.1, U15.5 (SDA), U3.40 (18_A4_SDA), U7.18 (SDA)
- net TX Q: now reaches C38.2, U7.1 (Q)
- net TX I: now reaches C39.2, U7.2 (I)
- net RX I: now reaches R64.2, TP13.1, U5.14 (VIN_R)
- net RX Q: now reaches R63.2, TP12.1, U5.13 (VIN_L)
- net +12P: now reaches J1.1 (Pin_1), L1.1
- net +12P: now also J11.1 (Pin_1), J11.2 (Pin_2), J11.3 (Pin_3), J11.4 (Pin_4), J11.5 (Pin_5), J11.6 (Pin_6)
- net A21: no longer names the net of U3.32 (40_A16)
- net A22: no longer names the net of U3.33 (41_A17)
- net CW on/off renamed CW
- net X Mode renamed TX Mode
- new net SDA: R53.1, U15.5 (SDA), U3.40 (18_A4_SDA), U7.18 (SDA)
- no-connect marks 18 -> 38
Other:
- note removed: "+12V"
- note removed: "BAND0"
- note removed: "BAND1"
- note removed: "BAND2"
- note removed: "BAND3"
- note removed: "BAND4"
- note removed: "GND"
- note removed: "RF RECEIVE CHAIN ->"
- note removed: "RF TRANSMIT CHAIN ->"
- note removed: "RX I Input"
- note removed: "RX Q Input"
- note removed: "RXTX"
- note removed: "TX I Input"
- note removed: "TX Q Input"
- moved on the sheet: C1, C10, C11, C12, C13, C14, C15, C16, C17, C18, C19, C2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
