File: T41_V012_Files/T41_V012_PCBs/T41_V012_PCBs_KiCad/T41-RF-board-V012/T41-RF-board-V012.kicad_pcb (KiCad board)
At the start: 4 copper layers, 100 x 100 mm, 221 parts, among them J1 IQ_Out, J2 RF_IN, J3 RFControl, J4 12-13.8V, J5 IQ_In, J6 RF_OUT, Q1 BS170, U1 74CBTLV3253DR, U10 SN74LVC1G04DCK, U106 AD8599, U107 OPA2209, U11 Si5351A-B-GT, U12 PE4312, U13 MAR-3SM+, U14 LM7805CT, U15 LM1117T-3.3, U16 LM358B, U17 LM317L, U2 PSA-8A+, U21 MCP23017_SO, U3 PE4312, U4 74CBTLV3253DR, U5 SN74LVC1G04DCK, U6 MC33078, U7 MASWSS0179, U8 MC33078, U9 MASWSS0179, Y1 ECS-TX053-S3, Y2 25MHz

Commit message: Work in progress -- still need to add the clock daughter board
Parts:
- removed C49, C52, C66, C85: 0.1uF 50V, Capacitor_SMD:C_1206_3216Metric
- removed JP13, JP3: AttenuatorBypass, Connector_PinHeader_2.54mm:PinHeader_1x02_P2.54mm_Vertical
- removed JP5: CLK0, Connector_PinHeader_2.54mm:PinHeader_1x02_P2.54mm_Vertical
- removed JP6: CLK1, Connector_PinHeader_2.54mm:PinHeader_1x02_P2.54mm_Vertical
- removed L107, L7: FB, Resistor_SMD:R_1206_3216Metric
- removed R24, R28, R53, R55: 10k, Resistor_SMD:R_1206_3216Metric
- removed TP15, TP16: TestPoint, Connector_PinHeader_2.54mm:PinHeader_1x01_P2.54mm_Vertical
- removed U12: PE4312, T41_Library:PE4312-QFN-20
- removed Y1: ECS-TX053-S3, T41_Library:Oscillator_ECS_TXO53_S3
- removed Y2: 25MHz, Crystal:Crystal_SMD_HC49-SD_HandSoldering
- U11: value Si5351A-B-GT -> T41_Attenuator_Daughter; footprint Package_SO:MSOP-10_3x3mm_P0.5mm -> T41_Library:T41_Attenuator_Daughter
- U3: value PE4312 -> T41_Attenuator_Daughter; footprint T41_Library:PE4312-QFN-20 -> T41_Library:T41_Attenuator_Daughter
- moved U3 100.3 mm to (123.7, 145.9), turned to 90 degrees
- moved U11 59.7 mm to (69.7, 51.7)
- moved G4 19.3 mm to (86.1, 106.9)
- moved C45 6.97 mm to (123.7, 136.9), turned to 90 degrees
- moved C22 4.14 mm to (61.7, 57.3), turned to 90 degrees
- moved C27 0.41 mm to (71.9, 66.8)
Connections:
- C22 pad 2: Net-(JP3-A) -> Net-(U11-RF1)
- C29 pad 1: Net-(U3-RF2) -> Net-(U11-RF2)
- C45 pad 2: Net-(U12-RF1) -> Net-(U3-RF2)
- C62 pad 2: Net-(U11-CLK2) -> Net-(J8-Pin_1)
- C63 pad 1: Net-(JP13-B) -> Net-(U3-RF1)
- R35 pad 2: Net-(JP5-A) -> Net-(J8-Pin_3)
- R37 pad 2: Net-(JP6-A) -> Net-(J8-Pin_4)
- R40 pad 1: Net-(U1-S1) -> Net-(J7-Pin_2)
- R40 pad 2: Net-(JP5-A) -> Net-(U1-S1)
- R42 pad 1: Net-(U1-S0) -> Net-(J7-Pin_1)
- R42 pad 2: Net-(JP6-A) -> Net-(U1-S0)
- U11 pad 1: Net-(U11-VDD) -> /RC0.5
- U11 pad 10: Net-(JP5-B) -> /RC4
- U11 pad 2: Net-(U11-XA) -> Net-(U11-RF1)
- U11 pad 3: Net-(U11-XB) -> GND
- U11 pad 4: /SCL -> +3V3
- U11 pad 5: /SDA -> GND
- U11 pad 6: Net-(U11-CLK2) -> /RC16
- U11 pad 7: Net-(U11-VDD) -> GND
- U11 pad 8: GND -> Net-(U11-RF2)
- U11 pad 9: Net-(JP6-B) -> /RC8
- U3 pad 1: Net-(U3-C16) -> /TC0.5
- U3 pad 10: GND -> /TC4
- U3 pad 11: GND -> /TC2
- U3 pad 12: GND -> /TC1
- U3 pad 2: Net-(JP3-A) -> Net-(U3-RF1)
- U3 pad 3: Net-(U3-Data) -> GND
- U3 pad 4: unconnected-(U3-Clock-Pad4) -> +3V3
- U3 pad 5: +3V3 -> GND
- U3 pad 6: +3V3 -> /TC16
- U3 pad 8: GND -> Net-(U3-RF2)
- U3 pad 9: +3V3 -> /TC8
Routing:
- net GND: track 50.5 -> 10.9 mm, vias 225 -> 184
- net /SCL: track 85.7 -> 49.9 mm, vias 2 -> 1
- net /SDA: track 78.1 -> 44.7 mm, vias 2 -> 1
- net Net-(U11-CLK2): track 30.8 -> 0.00 mm
- net Net-(JP5-A): track 30.0 -> 0.00 mm
- net Net-(JP6-A): track 29.8 -> 0.00 mm
- net Net-(J8-Pin_1): track 0.00 -> 27.6 mm
- net +3V3: track 343.8 -> 322.2 mm
- net /TC1: track 125.9 -> 105.1 mm, vias 2 -> 1
- net Net-(JP5-B): track 19.6 -> 0.00 mm
- net Net-(JP13-B): track 19.2 -> 0.00 mm
- net Net-(JP3-A): track 19.1 -> 0.00 mm
- net Net-(JP6-B): track 17.3 -> 0.00 mm
- net Net-(U11-VDD): track 16.6 -> 0.00 mm, vias 2 -> 0
- net /TC2: track 129.4 -> 113.3 mm, vias 2 -> 1
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Other:
- board text added: "RX gain control"
- board text removed: "CLK0 jumper"
- board text removed: "CLK1 jumper"
- board text removed: "Gain control bypass"
- board text removed: "RX RF gain control"
- board text removed: "TCXO upgrade"

Commit message: Initial commit of new RF board with clock and attenuators broken out to daughter boards
Parts:
- added U12: T41_DualClock_Daughter, T41_Library:T41_DualClock_Daughter, F.Cu at (87.1, 92.2)
- moved G4 31.0 mm to (114.3, 94.0)
- moved R37 8.89 mm to (98.3, 106.7), turned to 180 degrees
- moved R35 7.33 mm to (88.6, 106.7), turned to 180 degrees
- moved R40 0.57 mm to (90.2, 78.2), turned to 90 degrees
- moved R42 0.57 mm to (87.1, 78.2), turned to 90 degrees
Routing:
- net /SCL: track 49.9 -> 75.4 mm
- net /SDA: track 44.7 -> 69.6 mm
- net +3V3: track 322.2 -> 332.0 mm
- net Net-(U12-CLK5): track 0.11 -> 8.96 mm
- net Net-(U4-S0): track 35.4 -> 27.0 mm
- net Net-(U4-S1): track 30.2 -> 24.7 mm
- net Net-(U12-CLK4): track 0.00 -> 4.34 mm
- net Net-(U12-CLK6): track 27.6 -> 31.5 mm
- net Net-(U12-CLK1): track 0.00 -> 2.56 mm
- net Net-(U12-CLK0): track 0.00 -> 2.35 mm
- net GND: vias 184 -> 189
Other:
- board text added: "T41 RF Board: V12.1 Desig: AC8GY/K9HZ/KI3P 4 layer, 2025/12/27"
- board text removed: "T41 RF Board: V12.07 Designed by AC8GY/K9HZ Layout by KI3P 4 layer, 2025/01/16"

Commit message: Version of RF board with clock and attenuator daughterboards sent to Bill for comment
Other:
- board text added: "RX0"
- board text added: "RX90"
- board text added: "TX0"
- board text added: "TX90"
Changed lines of the file:
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@@
 			)
 		)
+		(fp_text user "GND"
+			(at 14.732 -9.144 0)
+			(unlocked yes)
+			(layer "F.SilkS")
+			(effects
+				(font
+					(size 1 1)
+					(thickness 0.2)
+					(bold yes)
+				)
+				(justify left bottom)
+			)
+		)
 		(fp_text user "SCL"
 			(at 14.732 -2.032 0)
@@
 		)
 		(embedded_fonts no)
-		(model "/home/oliver/Sync/Ham/T41/T41/T41_KiCad_Library/3D_models/HFD4_relay.step"
-			(offset
-				(xyz -1.2 -5.9 0)
-			)
-			(scale
-				(xyz 1 1 1)
-			)
-			(rotate
-				(xyz 0 0 0)
-			)
-		)
 	)
 	(footprint "Capacitor_SMD:C_1206_3216Metric"
@@
 		)
 		(embedded_fonts no)
-		(model "/home/oliver/Sync/Ham/T41/T41/T41_KiCad_Library/3D_models/HFD4_relay.step"
-			(offset
-				(xyz -1.2 -5.9 0)
-			)
-			(scale
-				(xyz 1 1 1)
-			)
-			(rotate
-				(xyz 0 0 0)
-			)
-		)
 	)
 	(footprint "Capacitor_SMD:C_1206_3216Metric"
@@
 		)
 		(embedded_fonts no)
-		(model "/home/oliver/Sync/Ham/T41/T41/T41_KiCad_Library/3D_models/HFD4_relay.step"
-			(offset
-				(xyz -1.2 -5.9 0)
-			)
-			(scale
-				(xyz 1 1 1)
-			)
-			(rotate
-				(xyz 0 0 0)
-			)
-		)
 	)
 	(footprint "Capacitor_SMD:C_1206_3216Metric"
@@
 		)
 	)
+	(gr_text "TX0"
+		(at 100.584 107.188 0)
+		(layer "F.SilkS")
+		(effects
+			(font
+				(size 1 1)
+				(thickness 0.15)
+			)
+			(justify left bottom)
+		)
+	)
 	(gr_text "T41 RF Board: V12.1\nDesig: AC8GY/K9HZ/KI3P\n4 layer, 2025/12/27"
 		(at 61.214 79.248 270)
@@
 		)
 	)
+	(gr_text "RX90"
+		(at 91.186 80.772 0)
+		(layer "F.SilkS")
+		(effects
+			(font
+				(size 1 1)
+				(thickness 0.15)
+			)
+			(justify left bottom)
+		)
+	)
 	(gr_text "CW envelope\nshaping"
 		(at 114.046 119.888 0)
@@
 		)
 	)
+	(gr_text "TX90"
+		(at 82.55 107.442 0)
+		(layer "F.SilkS")
+		(effects
+			(font
+				(size 1 1)
+				(thickness 0.15)
+			)
+			(justify left bottom)
+		)
+	)
 	(gr_text "ADDRESS\nSELECT"
 		(at 68.741 79.3 0)
 		(layer "F.SilkS")
 		(effects
+			(font
+				(size 1 1)
+				(thickness 0.15)
+			)
+			(justify left bottom)
+		)
+	)
+	(gr_text "RX0"
+		(at 82.55 76.708 0)
+		(layer "F.SilkS")
+		(effects

Commit message: H1 removed and some via transitions removed for reduced EMI
Parts:
- removed H4: EA-T220-38E, T41_Library:EAT22038E
- moved J1 9.05 mm to (147.8, 58.3), turned to 90 degrees
- moved TP8 0.74 mm to (98.2, 130.2)
- turned C36 to -90 degrees
Routing:
- net +5V: track 232.4 -> 254.9 mm
- net Net-(U107B--): track 12.7 -> 25.5 mm, vias 2 -> 0
- net Net-(U6A-+): track 44.8 -> 54.7 mm, vias 2 -> 0
- net Net-(U1-1B4): track 17.5 -> 25.4 mm, vias 2 -> 0
- net /I_out: track 18.3 -> 25.3 mm
- net /RXTX: track 51.7 -> 57.9 mm, vias 2 -> 0
- net Net-(U107A--): track 13.4 -> 7.37 mm, vias 2 -> 0
- net /Q_out: track 22.0 -> 16.1 mm
- net Net-(U4-1B2): track 32.7 -> 37.8 mm, vias 1 -> 0
- net Net-(U4-1B1): track 25.8 -> 30.5 mm
- net Net-(C5-Pad1): track 25.0 -> 29.1 mm
- net Net-(C36-Pad2): track 7.84 -> 4.89 mm
- net Net-(C51-Pad1): track 14.3 -> 17.0 mm
- net Net-(U4-1B3): track 33.8 -> 35.9 mm, vias 1 -> 0
- net /X Mode: track 118.5 -> 120.3 mm, vias 3 -> 1
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
Commit message: New layouts for RF board, clock board, and attenuator board are done
Parts:
- removed C48, C51: 10uF 50V, Capacitor_SMD:C_1206_3216Metric
- added C14: 10uF 50V, Capacitor_SMD:C_1206_3216Metric, F.Cu at (121.9, 65.2)
- added C3: 10uF 50V, Capacitor_SMD:C_1206_3216Metric, F.Cu at (83.9, 73.2)
- added L7: FB, Resistor_SMD:R_1206_3216Metric, F.Cu at (68.7, 73.2)
- added R24: 0, Resistor_SMD:R_1206_3216Metric, F.Cu at (114.3, 141.7)
- added R28: 0, Resistor_SMD:R_1206_3216Metric, F.Cu at (114.3, 135.8)
- added R53: 0, Resistor_SMD:R_1206_3216Metric, F.Cu at (114.3, 126.7)
- added R55: 0, Resistor_SMD:R_1206_3216Metric, F.Cu at (113.8, 121.2)
- added R66: 0, Resistor_SMD:R_1206_3216Metric, F.Cu at (138.2, 138.3)
- added R67: 0, Resistor_SMD:R_1206_3216Metric, F.Cu at (137.7, 121.0)
- R15, R19: value 500R -> 10k
- R52: value 2k2 -> 1k1
- moved J5 95.3 mm to (147.4, 129.7), turned to 90 degrees
- moved J6 90.2 mm to (54.6, 129.2), turned to 0 degrees
- moved C53 89.9 mm to (55.4, 118.7), turned to -90 degrees
- moved TP14 89.2 mm to (143.7, 121.0), turned to 180 degrees
- moved TP9 88.0 mm to (142.4, 138.3), turned to 180 degrees
- moved C58 87.4 mm to (52.1, 114.2), turned to 90 degrees
- moved U9 84.5 mm to (56.4, 113.9), turned to 90 degrees
- moved G5 80.7 mm to (137.7, 142.9), turned to 90 degrees
- moved R56 76.4 mm to (63.0, 136.7), turned to 90 degrees
- moved U10 76.0 mm to (61.6, 114.0), turned to 0 degrees
- moved C63 74.3 mm to (61.0, 117.1), turned to 180 degrees
- moved U17 73.3 mm to (62.5, 130.4), turned to -90 degrees
- moved C60 71.6 mm to (131.0, 111.4), turned to 0 degrees
- moved C32 70.7 mm to (138.7, 73.2), turned to -90 degrees
- moved C73 70.2 mm to (66.8, 139.8), turned to 0 degrees
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Connections:
- C12 pad 2: +5V -> Net-(C12-Pad2)
- C13 pad 2: +5V -> Net-(C12-Pad2)
- C32 pad 1: Net-(C32-Pad1) -> GND
- C32 pad 2: Net-(C32-Pad2) -> Net-(U107C-V+)
- C33 pad 1: Net-(C32-Pad1) -> Net-(C33-Pad1)
- C35 pad 1: Net-(C35-Pad1) -> GND
- C35 pad 2: Net-(C35-Pad2) -> Net-(U6C-V+)
- C36 pad 1: Net-(C36-Pad1) -> GND
- C36 pad 2: Net-(C36-Pad2) -> Net-(U8C-V+)
- C42 pad 1: Net-(C42-Pad1) -> GND
- C42 pad 2: Net-(C42-Pad2) -> Net-(U4-VCC)
- C46 pad 1: Net-(C42-Pad1) -> Net-(C46-Pad1)
- J5 pad R: Net-(C35-Pad2) -> Net-(J5-PadR)
- R14 pad 1: +5V -> Net-(C12-Pad2)
- R25 pad 2: Net-(C32-Pad1) -> Net-(C33-Pad1)
- R27 pad 1: Net-(C32-Pad2) -> Net-(R24-Pad1)
- R29 pad 2: Net-(C36-Pad1) -> Net-(R28-Pad2)
- R30 pad 1: Net-(C35-Pad1) -> Net-(R30-Pad1)
- R32 pad 1: Net-(C32-Pad1) -> Net-(C33-Pad1)
- R33 pad 1: Net-(C36-Pad2) -> Net-(R28-Pad1)
- R36 pad 2: Net-(C42-Pad1) -> Net-(C46-Pad1)
- R38 pad 1: Net-(C42-Pad2) -> Net-(R38-Pad1)
- R46 pad 1: Net-(C42-Pad1) -> Net-(C46-Pad1)
- TP9 pad 1: Net-(C35-Pad2) -> Net-(J5-PadR)
- U6 pad 1: Net-(C32-Pad1) -> Net-(C33-Pad1)
- U6 pad 7: Net-(C36-Pad1) -> Net-(R28-Pad2)
- U8 pad 1: Net-(C42-Pad1) -> Net-(C46-Pad1)
Routing:
- net /Cal: track 131.5 -> 11.5 mm, vias 1 -> 0
- net GND: track 10.9 -> 120.0 mm, vias 217 -> 372
- net /TC8: track 125.8 -> 18.8 mm, vias 1 -> 0
- net /TC4: track 119.2 -> 14.6 mm, vias 1 -> 0
- net /TC2: track 113.6 -> 10.4 mm, vias 1 -> 0
- net /TC16: track 134.6 -> 32.7 mm, vias 1 -> 0
- net /TC1: track 105.1 -> 6.65 mm, vias 1 -> 0
- net /RFIN: track 131.7 -> 35.5 mm
- net /TC0.5: track 117.4 -> 27.0 mm, vias 1 -> 0
- net +5V: track 254.9 -> 174.5 mm, vias 6 -> 7
- net /X Mode: track 120.3 -> 59.7 mm, vias 1 -> 0
- net +12V: track 98.9 -> 156.6 mm, vias 3 -> 2
- net +3V3: track 332.0 -> 279.3 mm, vias 12 -> 8
- net Net-(C42-Pad1): track 26.2 -> 0.00 mm
- net /CW on/off: track 80.6 -> 55.2 mm
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Other:
- board text added: "Quadrature detector"
- board text added: "Quadrature exciter"
- board text added: "RX IQ OUT"
- board text added: "RX RF IN"
- board text added: "T41 RF Board: V12.1 Desig: AC8GY/K9HZ/KI3P 4 layer, 2025/12/31"
- board text added: "TX IQ IN"
- board text added: "TX RF OUT"
- board text removed: "Quadrature sampling"
- board text removed: "Quadrature sampling detector"
- board text removed: "RF OUT"
- board text removed: "Receive IQ OUT"
- board text removed: "Receive RF IN"
- board text removed: "T41 RF Board: V12.1 Desig: AC8GY/K9HZ/KI3P 4 layer, 2025/12/27"
- board text removed: "Transmit IQ IN"
- board text removed: "exciter"
