File: T41_V012_Files/T41_V012_PCBs/T41_V012_PCBs_KiCad/T41-RF-board-V012/T41-RF-board-V012.kicad_pcb (KiCad board)
At the start: 4 copper layers, 100 x 100 mm, 209 parts, among them J1 IQ_Out, J2 RF_IN, J3 RFControl, J4 12-13.8V, J5 IQ_In, J6 RF_OUT, Q1 BS170, U1 74CBTLV3253DR, U10 SN74LVC1G04DCK, U106 AD8599, U107 OPA2209, U11 T41_Attenuator_Daughter, U12 T41_DualClock_Daughter, U13 MAR-3SM+, U14 LM7805CT, U15 LM1117T-3.3, U16 LM358B, U17 LM317L, U2 PSA-8A+, U21 MCP23017_SO, U3 T41_Attenuator_Daughter, U4 74CBTLV3253DR, U5 SN74LVC1G04DCK, U6 MC33078, U7 MASWSS0179, U8 MC33078, U9 MASWSS0179

Commit message: Changed transmit chain direction on schematic to match RF board
Connections:
- net Net-(U12-CLK0) renamed /RX0
- net Net-(U12-CLK1) renamed /RX90
- net Net-(U12-CLK6) renamed /CW
- net Net-(U4-S0) renamed /TX0
- net Net-(U4-S1) renamed /TX90
Other:
- board text added: "T41 RF Board: V12.8 Desig: AC8GY/K9HZ/KI3P 4 layer, 2025/12/31"
- board text removed: "T41 RF Board: V12.1 Desig: AC8GY/K9HZ/KI3P 4 layer, 2025/12/31"

Commit message: RF board updated to reverse the direction of the transmit chain, making routing easier and less prone to noise.
Parts:
- R56: value 1k8 -> 1k6
- R59: value 1k2 -> 1k1
- moved R28 0.64 mm to (113.7, 135.8)
- moved L8 0.64 mm to (117.3, 126.7)
- moved R24 0.63 mm to (113.7, 141.7)
- moved R53 0.63 mm to (113.7, 126.7)
- moved R55 0.13 mm to (113.7, 121.2)
- moved L9 0.06 mm to (113.1, 111.9)
Connections:
- R35 pad 1: /TX90 -> Net-(U4-S1)
- R35 pad 2: Net-(U12-CLK4) -> /TX0
- R37 pad 1: /TX0 -> Net-(U4-S0)
- R37 pad 2: Net-(U12-CLK5) -> /TX90
- R40 pad 1: /RX90 -> /RX0
- R42 pad 1: /RX0 -> /RX90
- U12 pad 1: Net-(U12-CLK4) -> /TX0
- U12 pad 11: /RX90 -> /RX0
- U12 pad 12: /RX0 -> /RX90
- U12 pad 2: Net-(U12-CLK5) -> /TX90
- U4 pad 14: /TX0 -> Net-(U4-S0)
- U4 pad 2: /TX90 -> Net-(U4-S1)
Routing:
- net GND: track 120.0 -> 244.3 mm, vias 372 -> 424
- net Net-(U4-S1): track 0.00 -> 38.1 mm
- net /TX90: track 39.8 -> 2.83 mm
- net /TX0: track 34.5 -> 2.83 mm
- net Net-(U4-S0): track 0.00 -> 30.4 mm
- net Net-(U12-CLK4): track 2.83 -> 0.00 mm
- net Net-(U12-CLK5): track 2.83 -> 0.00 mm
- net Net-(U16A-+): track 7.44 -> 8.67 mm
- net /SCL: track 87.4 -> 88.0 mm
