File: T41_V012_Files/T41_V012_PCBs/T41_V012_PCBs_KiCad/T41-RF-board-V012/T41-RF-board-V012.kicad_sch (KiCad schematic)
At the start: 222 parts, among them J1 IQ_Out, J2 RF_IN, J3 RFControl, J4 12-13.8V, J5 IQ_In, J6 RF_OUT, Q1 BS170, U1 74CBTLV3253DR, U10 SN74LVC1G04DCK, U106 AD8599, U107 OPA2209, U11 Si5351A-B-GT, U12 PE4312, U13 MAR-3SM+, U14 LM7805CT, U15 LM1117T-3.3, U16 LM358B, U17 LM317L, U2 PSA-8A+, U21 MCP23017_SO, U3 PE4312, U4 74CBTLV3253DR, U5 SN74LVC1G04DCK, U6 MC33078, U7 MASWSS0179, U8 MC33078, U9 MASWSS0179, Y1 ECS-TX053-S3, Y2 25MHz

Commit message: Work in progress -- still need to add the clock daughter board
Parts:
- removed C49, C52, C66, C85: 0.1uF 50V, Capacitor_SMD:C_1206_3216Metric, symbol Device:C
- removed JP13, JP3: AttenuatorBypass, Connector_PinHeader_2.54mm:PinHeader_1x02_P2.54mm_Vertical, symbol Jumper:Jumper_2_Open
- removed JP5: CLK0, Connector_PinHeader_2.54mm:PinHeader_1x02_P2.54mm_Vertical, symbol Jumper:Jumper_2_Open
- removed JP6: CLK1, Connector_PinHeader_2.54mm:PinHeader_1x02_P2.54mm_Vertical, symbol Jumper:Jumper_2_Open
- removed L107, L7: FB, Resistor_SMD:R_1206_3216Metric, symbol Device:L
- removed R24, R28, R53, R55: 10k, Resistor_SMD:R_1206_3216Metric, symbol Device:R
- removed TP15, TP16: TestPoint, Connector_PinHeader_2.54mm:PinHeader_1x01_P2.54mm_Vertical, symbol Connector:TestPoint
- removed U11: Si5351A-B-GT, Package_SO:MSOP-10_3x3mm_P0.5mm, symbol Oscillator:Si5351A-B-GT
- removed U12, U3: PE4312, T41_Library:PE4312-QFN-20, symbol T41_Library:PE4312
- removed Y1: ECS-TX053-S3, T41_Library:Oscillator_ECS_TXO53_S3, symbol T41_Library:ECS-TX053-S3
- removed Y2: 25MHz, Crystal:Crystal_SMD_HC49-SD_HandSoldering, symbol Device:Crystal
- added J7: RX VFO, symbol Connector:Conn_01x04_Socket
- added J8: TX VFO, symbol Connector:Conn_01x04_Socket
- added J9: Power & I2C, symbol Connector:Conn_01x04_Socket
- added U11, U3: T41_Attenuator_Daughter, T41_Library:T41_Attenuator_Daughter, symbol T41_Library:T41_Attenuator_Daughter
Connections:
- net +3V3: now also J9.2 (Pin_2), U11.4 (3V3), U3.4 (3V3)
- net GND: now also J7.3 (Pin_3), J8.2 (Pin_2), J9.1 (Pin_1), U11.3 (GND), U11.5 (GND), U11.7 (GND), U3.3 (GND), U3.5 (GND), U3.7 (GND)
- net RC0.5: now also U11.1 (0.5dB)
- net RC1: now also U11.12 (1dB)
- net RC16: now also U11.6 (16dB)
- net RC2: now also U11.11 (2dB)
- net RC4: now also U11.10 (4dB)
- net RC8: now also U11.9 (8dB)
- net SCL: now also J9.4 (Pin_4)
- net SDA: now also J9.3 (Pin_3)
- net TC0.5: now also U3.1 (0.5dB)
- net TC1: now also U3.12 (1dB)
- net TC16: now also U3.6 (16dB)
- net TC2: now also U3.11 (2dB)
- net TC4: now also U3.10 (4dB)
- net TC8: now also U3.9 (8dB)
- net at C63.1: now also U3.2 (RF1)
- net at C45.2: now also U3.8 (RF2)
- net at R37.2: now also J8.4 (Pin_4); no longer R42.2
- net at R35.2: now also J8.3 (Pin_3); no longer R40.2
- net at C62.2: now also J8.1 (Pin_1)
- net at R42.1: now also J7.1 (Pin_1); no longer U1.14 (S0)
- net at C22.2: now also U11.2 (RF1)
- net at R40.1: now also J7.2 (Pin_2); no longer U1.2 (S1)
- net at C29.1: now also U11.8 (RF2)
- new net: R42.2, U1.14 (S0)
- new net: R40.2, U1.2 (S1)
- no-connect marks 15 -> 13
Other:
- note removed: "Clock selector MF circuitry"
- moved on the sheet: R35, R37, R40, R42

Commit message: Initial commit of new RF board with clock and attenuators broken out to daughter boards
Parts:
- removed J7: RX VFO, symbol Connector:Conn_01x04_Socket
- removed J8: TX VFO, symbol Connector:Conn_01x04_Socket
- removed J9: Power & I2C, symbol Connector:Conn_01x04_Socket
- added U12: T41_DualClock_Daughter, T41_Library:T41_DualClock_Daughter, symbol T41_Library:T41_DualClock_Daughter
Connections:
- net +3V3: now also U12.7 (3V3)
- net GND: now also U12.10 (GND), U12.3 (GND), U12.8 (GND)
- net SCL: now also U12.5 (SCL)
- net SDA: now also U12.6 (SDA)
- net at C62.2: now also U12.4 (CLK6)
- net at R35.2: now also U12.1 (CLK4)
- net at R37.2: now also U12.2 (CLK5)
- net at R42.1: now also U12.12 (CLK0)
- net at R40.1: now also U12.11 (CLK1)
- no-connect marks 13 -> 14
Other:
- moved on the sheet: R40, R42

Commit message: Updated titles for schematics and printed to PDF
Changed lines of the file:
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@@
 	(title_block
 		(title "T41 RF Board")
-		(date "2024-12-13")
-		(rev "V012.7")
-		(comment 1 "        Transcribed to KiCAD by OG King-KI3P")
+		(date "2025-12-27")
+		(rev "V012.8")
+		(comment 1 "        Additional work by Oliver KI3P")
 		(comment 2 "By Al Peter-AC8GY, Revised by WJ Schmidt-K9HZ")
-		(comment 3 "Change log: Removed clock divider")
+		(comment 3 "Change log: Added daughterboards")
 	)
 	(text "RF output"
@@
 	(wire
 		(pts
-			(xy 205.74 152.4) (xy 207.01 152.4)
+			(xy 205.74 153.67) (xy 209.55 153.67)
 		)
 		(stroke
@@
 	(wire
 		(pts
-			(xy 205.74 153.67) (xy 205.74 152.4)
-		)
-		(stroke
-			(width 0)
-			(type default)
-		)
-	)
-	(wire
-		(pts
 			(xy 172.72 275.59) (xy 177.8 275.59)
 		)
@@
 	(wire
 		(pts
-			(xy 207.01 156.21) (xy 207.01 154.94)
-		)
-		(stroke
-			(width 0)
-			(type default)
-		)
-	)
-	(wire
-		(pts
 			(xy 245.11 198.12) (xy 245.11 200.66)
 		)
@@
 	(wire
 		(pts
-			(xy 205.74 156.21) (xy 207.01 156.21)
+			(xy 205.74 156.21) (xy 209.55 156.21)
 		)
 		(stroke
@@
 	)
 	(label "SDA"
-		(at 207.01 152.4 0)
+		(at 209.55 153.67 0)
 		(effects
 			(font
@@
 	)
 	(label "SCL"
-		(at 207.01 154.94 0)
+		(at 209.55 156.21 0)
 		(effects
 			(font

Commit message: H1 removed and some via transitions removed for reduced EMI
Parts:
- removed H4: EA-T220-38E, EAT22038E, symbol T41_Library:EA-T220-38E
Connections:
- no-connect marks 14 -> 12
Other:
- moved on the sheet: G4
Changed lines of the file:
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@@
 	)
 	(junction
-		(at 148.59 50.8)
-		(diameter 0)
-		(color 0 0 0 0)
-	)
-	(junction
 		(at 142.24 55.88)
 		(diameter 0)
@@
 	)
 	(junction
+		(at 139.7 55.88)
+		(diameter 0)
+		(color 0 0 0 0)
+	)
+	(junction
 		(at 78.74 243.84)
 		(diameter 0)
@@
 	)
 	(no_connect
-		(at 135.89 43.18)
-	)
-	(no_connect
 		(at 93.98 144.78)
 	)
@@
 	)
 	(no_connect
-		(at 135.89 40.64)
-	)
-	(no_connect
 		(at 156.21 156.21)
 	)
@@
 	(wire
 		(pts
-			(xy 148.59 50.8) (xy 148.59 55.88)
-		)
-		(stroke
-			(width 0)
-			(type default)
-		)
-	)
-	(wire
-		(pts
 			(xy 53.34 129.54) (xy 58.42 129.54)
 		)
@@
 	(wire
 		(pts
+			(xy 139.7 55.88) (xy 142.24 55.88)
+		)
+		(stroke
+			(width 0)
+			(type default)
+		)
+	)
+	(wire
+		(pts
 			(xy 148.59 233.68) (xy 158.75 233.68)
 		)
@@
 	(wire
 		(pts
+			(xy 139.7 38.1) (xy 137.16 38.1)
+		)
+		(stroke
+			(width 0)
+			(type default)
+		)
+	)
+	(wire
+		(pts
 			(xy 106.68 195.58) (xy 106.68 205.74)
 		)
@@
 	(wire
 		(pts
+			(xy 148.59 55.88) (xy 148.59 50.8)
+		)
+		(stroke
+			(width 0)
+			(type default)
+		)
+	)
+	(wire
+		(pts
 			(xy 335.28 212.09) (xy 334.01 212.09)
 		)
@@
 	(wire
 		(pts
-			(xy 148.59 50.8) (xy 153.67 50.8)
-		)
-		(stroke
-			(width 0)
-			(type default)
-		)
-	)
-	(wire
-		(pts
 			(xy 129.54 102.87) (xy 129.54 96.52)
 		)
@@
 	(wire
 		(pts
+			(xy 139.7 38.1) (xy 139.7 55.88)
+		)
+		(stroke
+			(width 0)
+			(type default)
+		)
+	)
+	(wire
+		(pts
 			(xy 134.62 91.44) (xy 140.97 91.44)
 		)
@@
 	(wire
 		(pts
-			(xy 139.7 55.88) (xy 142.24 55.88)
-		)
-		(stroke
-			(width 0)
-			(type default)
-		)
-	)
-	(wire
-		(pts
 			(xy 52.07 165.1) (xy 54.61 165.1)
 		)
@@
 	)
 	(symbol
-		(lib_id "T41_Library:EA-T220-38E")
-		(at 135.89 40.64 0)
-		(unit 1)
-		(exclude_from_sim no)
-		(in_bom yes)
-		(on_board yes)
-		(dnp no)
-		(property "Reference" "H4"
-			(at 144.78 34.29 0)
-			(effects
-				(font
-					(size 1.27 1.27)
-				)
-				(justify left)
-			)
-		)
-		(property "Value" "EA-T220-38E"
-			(at 139.7 36.83 0)
-			(effects
-				(font
-					(size 1.27 1.27)
-				)
-				(justify left)
-			)
-		)
-		(property "Footprint" "EAT22038E"
-			(at 152.4 135.56 0)
-			(effects
-				(font
-					(size 1.27 1.27)
-				)
-				(justify left top)
-				(hide yes)
-			)
-		)
-		(property "Datasheet" "https://www.ohmite.com/assets/docs/sink_e.pdf?r=false"
-			(at 152.4 235.56 0)
-			(effects
-				(font
-					(size 1.27 1.27)
-				)
-				(justify left top)
-				(hide yes)
-			)
-		)
-		(property "Description" ""
-			(at 135.89 40.64 0)
-			(effects
-				(font
-					(size 1.27 1.27)
-				)
-				(hide yes)
-			)
-		)
-		(property "Height" "38.35"
-			(at 152.4 435.56 0)
-			(effects
-				(font
-					(size 1.27 1.27)
-				)
-				(justify left top)
-				(hide yes)
-			)
-		)
-		(property "Mouser Part Number" "588-EA-T220-38E"
-			(at 152.4 535.56 0)
-			(effects
-				(font
-					(size 1.27 1.27)
-				)
-				(justify left top)
-				(hide yes)
-			)
-		)
-		(property "Mouser Price/Stock" "https://www.mouser.co.uk/ProductDetail/Ohmite/EA-T220-38E?qs=6weo7U0lPxCX9kcQhGcuZQ%3D%3D"
-			(at 152.4 635.56 0)
-			(effects
-				(font
-					(size 1.27 1.27)
-				)
-				(justify left top)
-				(hide yes)
-			)
-		)
-		(property "Manufacturer_Name" "Ohmite"
-			(at 152.4 735.56 0)
-			(effects
-				(font
-					(size 1.27 1.27)
-				)
-				(justify left top)
-				(hide yes)
-			)
-		)
-		(property "Manufacturer_Part_Number" "EA-T220-38E"
-			(at 152.4 835.56 0)
-			(effects
-				(font
-					(size 1.27 1.27)
-				)
-				(justify left top)
-				(hide yes)
-			)
-		)
-		(pin "1"
-		)
-		(pin "2"
-		)
-		(instances
-			(project "T41-RF-board-V012"
-				(path "/3c4b9d3b-a516-4fd7-b325-b74c836dee65"
-					(reference "H4")
-					(unit 1)
-				)
-			)
-		)
-	)
-	(symbol
 		(lib_id "Amplifier_Operational:MC33078")
 		(at 99.06 205.74 0)
@@
 	(symbol
 		(lib_id "Connector:TestPoint")
-		(at 153.67 50.8 0)
+		(at 137.16 38.1 0)
 		(unit 1)
 		(exclude_from_sim no)
@@
 		(dnp no)
 		(property "Reference" "G4"
-			(at 154.94 46.99 0)
+			(at 138.43 34.29 0)
 			(effects
 				(font
@@
 		)
 		(property "Value" "TestPoint"
-			(at 153.67 49.53 0)
+			(at 137.16 36.83 0)
 			(effects
 				(font
@@
 		)
 		(property "Footprint" "Connector_PinHeader_2.54mm:PinHeader_1x01_P2.54mm_Vertical"
-			(at 158.75 50.8 0)
+			(at 142.24 38.1 0)
 			(effects
 				(font
@@
 		)
 		(property "Datasheet" "~"
-			(at 158.75 50.8 0)
+			(at 142.24 38.1 0)
 			(effects
 				(font
@@
 		)
 		(property "Description" ""
-			(at 153.67 50.8 0)
+			(at 137.16 38.1 0)
 			(effects
 				(font
@@
 		)
 		(property "Mouser Part Number" ""
-			(at 153.67 50.8 0)
+			(at 137.16 38.1 0)
 			(effects
 				(font

Commit message: New layouts for RF board, clock board, and attenuator board are done
Parts:
- removed C48, C51: 10uF 50V, Capacitor_SMD:C_1206_3216Metric, symbol Device:C
- added C14, C3: 10uF 50V, Capacitor_SMD:C_1206_3216Metric, symbol Device:C
- added L7: FB, Resistor_SMD:R_1206_3216Metric, symbol Device:L
- added R24, R28, R53, R55, R66, R67: 0, Resistor_SMD:R_1206_3216Metric, symbol Device:R
- JP2: now left out of the parts list
- R15, R19: value 500R -> 10k
- R52: value 2k2 -> 1k1
Connections:
- net +5V: now also L7.1; no longer C12.2, C13.2, R14.1
- net GND: now also C32.1, C35.1, C36.1, C42.1, C14.1, C3.1
- net at R38.1: now also R53.1; no longer C42.2
- net at J5.R, TP9.1: now also R66.2; no longer C35.2
- net at J5.T, TP14.1: now also R67.2
- net at C33.1, R25.2, R32.1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: now also R24.2; no longer C32.1
- net at C65.1, L9.1, R50.2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: now also C36.2
- net at R27.1: now also R24.1; no longer C32.2
- net at R43.1: now also R55.1
- net at C23.2, C25.1, C7.2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: now also C14.2
- net at C30.2, L5.2, U4.16 (VCC): now also C42.2
- net at C26.1, L2.1, U107.8 (V+): now also C32.2
- net at C46.1, R36.2, R46.1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: now also R53.2; no longer C42.1
- net at C64.1, L8.1, U6.8 (V+): now also C35.2
- net at R30.1: now also R66.1; no longer C35.1
- net at R41.2, U8.7: now also R55.2
- net at R44.1: now also R67.1
- net at R29.2, U6.7: now also R28.2; no longer C36.1
- net at R33.1: now also R28.1; no longer C36.2
- net at C6.2, L1.2, U1.16 (VCC): now also C3.2
- new net: C12.2, C13.2, L7.2, R14.1
Other:
- moved on the sheet: C18, C6, C61, L1, L2, L3

Commit message: Changed transmit chain direction on schematic to match RF board
Connections:
- net CW: now reaches C62.2, U12.4 (CLK6)
- net TX90: now reaches R35.1, U4.2 (S1)
- net RX0: now reaches R42.1, U12.12 (CLK0)
- net RX90: now reaches R40.1, U12.11 (CLK1)
- net TX0: now reaches R37.1, U4.14 (S0)
Other:
- note added: "<- RF TRANSMIT CHAIN"
- note removed: "RF TRANSMIT CHAIN ->"
- moved on the sheet: C30, C31, C33, C34, C35, C36, C37, C38, C39, C40, C41, C42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

Commit message: RF board updated to reverse the direction of the transmit chain, making routing easier and less prone to noise.
Parts:
- C1, C11, C12, C14, C3, C32, C35, C36, C39, C41, C42, C57, C60, C67, C71: LCSC (none) -> C13585; PN (none) -> C1206C106K4PACTU
- C10, C17, C28, C37, C4, C54: LCSC (none) -> C1846; PN (none) -> C1206C103K5RAC7210
- C13, C16, C18, C20, C22, C23, C25, C26, C27, C29, C30, C31, C40, C43, C45, C47, C53, C55, C56, C58, C59, C6, C61, C62, C63, C64, C65, C68, C7, C70, C72, C73, C80: LCSC (none) -> C24497; PN (none) -> C1206C104K5RACTU
- C15, C2, C24, C9: LCSC (none) -> C1848; PN (none) -> CL31B105KBHNNNE
- C19, C8: LCSC (none) -> C527293; PN (none) -> C1206C181J5GAC7800
- C21, C5: LCSC (none) -> C1884; PN (none) -> CL31C101JGFNNNE
- C33, C46: LCSC (none) -> C326631; PN (none) -> GRM3195C1H222JA01D
- C34, C38, C44, C50: LCSC (none) -> C1857; PN (none) -> 12065C204KAT4A
- C69: PN (none) -> ECA-1EM471
- G1, G2, G3, G4, G5, G6, JP4, TP1, TP10, TP11, TP12, TP13, TP14, TP17, TP18, TP2, TP3, TP4, TP5, TP6, TP7, TP8, TP9: now not fitted
- J1, J5: PN (none) -> SJ1-3515N
- J2, J6: Mouser Part Number 712-CONSMA001-G -> (none); PN (none) -> CONSMA001-G
- L1, L2, L3, L5, L6, L7, L8, L9: LCSC (none) -> C74486; PN (none) -> HZ1206E601R-10
- L10, L4: LCSC (none) -> C395022; PN (none) -> LQM31PN1R5M00L
- L11, L12, L13: LCSC (none) -> C5753503; PN (none) -> IFSC2020DEER100M01
- Q1: PN (none) -> BS170
- R1, R13: LCSC (none) -> C17944; PN (none) -> ERA-8AEB202V
- R10, R11, R17, R18, R2, R3, R5, R6: LCSC (none) -> C26033; PN (none) -> ERJ-8ENF5101V
- R12, R15, R19, R20, R21, R23, R25, R29, R30, R32, R36, R39, R41, R44, R46, R47, R7, R9: LCSC (none) -> C17902; PN (none) -> CR1206-FX-1002ELF
- R14: LCSC (none) -> C205349; PN (none) -> CRCW120636R5FKEA
- R16, R22, R4, R54, R8: LCSC (none) -> C17901; PN (none) -> CR1206-FX-1000ELF
- R24, R28, R35, R37, R40, R42, R53, R55, R64, R65, R66, R67: LCSC (none) -> C17888; PN (none) -> 1206S4J0000TDE
- R26, R31, R34, R45, R49, R50, R51, R60, R61, R62, R63: LCSC (none) -> C17948; PN (none) -> RT1206FRE072K2L
- R27, R33, R38, R43: LCSC (none) -> C2984401; PN (none) -> CRCW120649R9FKEAC
- R48, R73: LCSC (none) -> C17900; PN (none) -> CRCW1206100KFKEAC
- R52: LCSC (none) -> C17889; PN (none) -> CR1206-FX-1101ELF
- R56: value 1k8 -> 1k6; LCSC (none) -> C17896; PN (none) -> ERJ-8ENF1601V
- R57: LCSC (none) -> C17930; PN (none) -> CR1206-FX-3300ELF
- R58: LCSC (none) -> C17992; PN (none) -> CR1206-FX-5102ELF
- R59: value 1k2 -> 1k1; LCSC (none) -> C17889; PN (none) -> CR1206-FX-1101ELF
- TR1: LCSC (none) -> C2683432; PN (none) -> ADT1-1+
- TR2: LCSC (none) -> C5223988; PN (none) -> ADT2-1T+
- U1, U4: LCSC (none) -> C543079; PN (none) -> SN74CBTLV3253DR
- U10, U5: LCSC (none) -> C8207; PN (none) -> SN74LVC1G04DCKR
- U106: LCSC (none) -> C207971; PN (none) -> AD8599ARZ-REEL
- U107: LCSC (none) -> C2057330; PN (none) -> OPA2209AIDR
- U13: LCSC (none) -> C6937326; PN (none) -> MAR-3SM+
- U14: LCSC (none) -> C725349; PN (none) -> LM7805CT
- U15: LCSC (none) -> C201726; PN (none) -> LM1117T-3.3/NOPB
- U16: LCSC (none) -> C1850238; PN (none) -> LM358BIDR
- U17: LCSC (none) -> C183332; PN (none) -> LM317LIDR
- U2: LCSC (none) -> C3192212; PN (none) -> PSA-8A+
- U21: LCSC (none) -> C47023; PN (none) -> MCP23017-E/SO
- U6, U8: LCSC (none) -> C2057560; PN (none) -> MC33078DR
- U7, U9: LCSC (none) -> C3304462; PN (none) -> MASWSS0179TR-3000
Connections:
- net RX0: now also R40.1, U12.11 (CLK1); no longer R42.1, U12.12 (CLK0)
- net RX90: now also R42.1, U12.12 (CLK0); no longer R40.1, U12.11 (CLK1)
- net TX0: now also R35.2, U12.1 (CLK4); no longer R37.1, U4.14 (S0)
- net TX90: now also R37.2, U12.2 (CLK5); no longer R35.1, U4.2 (S1)
- new net: R35.1, U4.2 (S1)
- new net: R37.1, U4.14 (S0)
Other:
- moved on the sheet: C53, C58, C63, J6, U10, U3, U9
