File: T41_V012_Files/T41_V012_PCBs/T41_V012_PCBs_KiCad/T41-RF-board-DualClock-daughterboard/DualClockLO.kicad_pcb (KiCad board)
At the start: 4 copper layers, 30 x 25.3 mm, 24 parts, among them J1 qwiic, J2 pin header, J3 pin header, J4 pin header, J5 OEBSSEN, Y1 ECS-TX053-S3, Y2 25MHz, Y3 Si5351A-B-GM

Commit message: New layouts for RF board, clock board, and attenuator board are done
Parts:
- Y2: moved to F.Cu
- moved Y2 16.4 mm to (138.2, 93.7), turned to 0 degrees
- moved J2 10.1 mm to (141.0, 79.8), turned to -90 degrees
- moved C1 8.30 mm to (140.2, 98.8), turned to 0 degrees
- moved H1 5.79 mm to (146.1, 79.8)
- moved H2 5.79 mm to (146.1, 100.1)
- moved L1 5.04 mm to (140.2, 100.6)
- moved J1 4.77 mm to (144.8, 86.9)
- moved G1 4.60 mm to (140.2, 86.9), turned to 90 degrees
- moved Y1 4.07 mm to (134.4, 99.8), turned to 180 degrees
- moved R2 3.27 mm to (134.9, 87.4), turned to 90 degrees
- moved R1 2.87 mm to (134.9, 84.3)
- moved C2 2.51 mm to (127.0, 93.7), turned to -90 degrees
Routing:
- net Net-(Y3-XB): track 6.78 -> 24.9 mm, vias 1 -> 0
- net /SDA: track 23.0 -> 30.2 mm
- net /SCL: track 21.2 -> 27.4 mm, vias 0 -> 1
- net +3V3: track 13.6 -> 8.10 mm, vias 6 -> 8
- net Net-(Y1-OUT): track 4.53 -> 9.23 mm
- net GND: track 18.2 -> 19.9 mm, vias 36 -> 59
- net Net-(Y3-XA): track 11.3 -> 12.9 mm, vias 1 -> 0
- net Net-(Y1-VDD): track 3.78 -> 4.80 mm
Other:
- board size 30 x 25.3 mm -> 35.1 x 25.3 mm

Commit message: Changed transmit chain direction on schematic to match RF board
Parts:
- moved C1 1.78 mm to (140.2, 100.6)
- moved L1 1.78 mm to (140.2, 98.8)
Changed lines of the file:
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@@
 	(footprint "Inductor_SMD:L_0603_1608Metric"
 		(layer "F.Cu")
-		(at 140.233501 100.584)
+		(at 140.208 98.806)
 		(descr "Inductor SMD 0603 (1608 Metric), square (rectangular) end terminal, IPC-7351 nominal, (Body size source: http://www.tortai-tech.com/upload/download/2011102023233369053.pdf), generated with kicad-footprint-generator")
 		(tags "inductor")
 		(property "Reference" "L1"
-			(at 2.514499 0.254 0)
+			(at 2.413 0 0)
 			(layer "F.SilkS")
 			(effects
@@
 	(footprint "Capacitor_SMD:C_0603_1608Metric"
 		(layer "F.Cu")
-		(at 140.208 98.806)
+		(at 140.233501 100.584)
 		(descr "Capacitor SMD 0603 (1608 Metric), square (rectangular) end terminal, IPC-7351 nominal, (Body size source: IPC-SM-782 page 76, https://www.pcb-3d.com/wordpress/wp-content/uploads/ipc-sm-782a_amendment_1_and_2.pdf), generated with kicad-footprint-generator")
 		(tags "capacitor")
@@
 	)
 	(segment
-		(start 140.983 98.806)
-		(end 141.732 98.806)
-		(width 0.5)
-		(layer "F.Cu")
-		(net 2)
-	)
-	(segment
 		(start 118.999 81.407)
 		(end 118.999 82.156)
@@
 	)
 	(segment
+		(start 141.008501 100.584)
+		(end 141.732 100.584)
+		(width 0.5)
+		(layer "F.Cu")
+		(net 2)
+	)
+	(segment
 		(start 137.638 98.522)
 		(end 137.668 98.552)
@@
 	)
 	(via
-		(at 141.732 98.806)
-		(size 0.6)
-		(drill 0.3)
-		(layers "F.Cu" "B.Cu")
-		(net 2)
-	)
-	(via
 		(at 139.7 83.058)
 		(size 0.6)
@@
 	)
 	(via
+		(at 141.732 100.584)
+		(size 0.6)
+		(drill 0.3)
+		(layers "F.Cu" "B.Cu")
+		(net 2)
+	)
+	(via
 		(at 141.224 88.392)
 		(size 0.6)
@@
 	)
 	(segment
-		(start 141.021002 100.584)
-		(end 141.732 100.584)
-		(width 0.5)
-		(layer "F.Cu")
-		(net 6)
-	)
-	(segment
 		(start 142.78 87.368)
 		(end 141.232 87.368)
@@
 	)
 	(segment
+		(start 140.995501 98.806)
+		(end 141.732 98.806)
+		(width 0.5)
+		(layer "F.Cu")
+		(net 6)
+	)
+	(segment
 		(start 141.232 87.368)
 		(end 141.224 87.376)
@@
 	)
 	(via
-		(at 141.732 100.584)
+		(at 114.935 91.567)
 		(size 0.6)
 		(drill 0.3)
@@
 	)
 	(via
-		(at 114.935 91.567)
+		(at 141.732 98.806)
 		(size 0.6)
 		(drill 0.3)
