File: T41_V012_Files/T41_V012_PCBs/T41_V012_PCBs_KiCad/T41-RF-board-DualClock-daughterboard/DualClockLO.kicad_sch (KiCad schematic)
At the start: 24 parts, among them J1 qwiic, J2 pin header, J3 pin header, J4 pin header, J5 OEBSSEN, Y1 ECS-TX053-S3, Y2 25MHz, Y3 Si5351A-B-GM

Commit message: RF board updated to reverse the direction of the transmit chain, making routing easier and less prone to noise.
Parts:
- C1, C2, C3, C4, C5: LCSC (none) -> C14663
- J1: LCSC (none) -> C160404; now left out of the parts list
- L1, L2, L3, L4: LCSC (none) -> C1002
- R1, R2: LCSC (none) -> C4190; PN (none) -> CRGP0603F2K2; now not fitted; now left out of the parts list
- Y1: LCSC (none) -> C18457614
- Y2: now not fitted
- Y3: LCSC (none) -> C22413806
Changed lines of the file:
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@@
 			)
 		)
+		(property "LCSC" ""
+			(at 168.91 110.49 0)
+			(effects
+				(font
+					(size 1.27 1.27)
+				)
+				(hide yes)
+			)
+		)
 		(pin "3"
 		)
@@
 			)
 		)
-		(property "Mouser Part Number" ""
-			(at 217.17 49.53 0)
+		(property "PN" "BMC-Q1JY0500H"
+			(at 217.17 49.53 90)
 			(effects
 				(font
@@
 			)
 		)
-		(property "PN" "BMC-Q1JY0500H"
+		(property "LCSC" "C1002"
 			(at 217.17 49.53 90)
 			(effects
@@
 			)
 		)
+		(property "LCSC" ""
+			(at 251.46 80.01 0)
+			(effects
+				(font
+					(size 1.27 1.27)
+				)
+				(hide yes)
+			)
+		)
 		(pin "3"
 		)
@@
 		(unit 1)
 		(exclude_from_sim no)
-		(in_bom yes)
+		(in_bom no)
 		(on_board yes)
 		(dnp no)
@@
 			)
 		)
+		(property "LCSC" "C160404"
+			(at 246.38 128.27 0)
+			(effects
+				(font
+					(size 1.27 1.27)
+				)
+				(hide yes)
+			)
+		)
 		(pin "3"
 		)
@@
 			)
 		)
+		(property "LCSC" ""
+			(at 266.7 99.06 0)
+			(effects
+				(font
+					(size 1.27 1.27)
+				)
+				(hide yes)
+			)
+		)
 		(pin "3"
 		)
@@
 			)
 		)
+		(property "LCSC" ""
+			(at 262.89 127 0)
+			(effects
+				(font
+					(size 1.27 1.27)
+				)
+				(hide yes)
+			)
+		)
 		(instances
 			(project ""
@@
 			)
 		)
-		(property "Mouser Part Number" ""
+		(property "PN" "ECS-TXO53-S3-33-250-BN-TR "
 			(at 135.89 72.39 0)
 			(effects
@@
 			)
 		)
-		(property "PN" "ECS-TXO53-S3-33-250-BN-TR "
+		(property "LCSC" "C18457614"
 			(at 135.89 72.39 0)
 			(effects
@@
 			)
 		)
-		(property "Mouser Part Number" ""
-			(at 213.36 62.23 0)
+		(property "PN" "BMC-Q1JY0500H"
+			(at 213.36 62.23 90)
 			(effects
 				(font
@@
 			)
 		)
-		(property "PN" "BMC-Q1JY0500H"
+		(property "LCSC" "C1002"
 			(at 213.36 62.23 90)
 			(effects
@@
 			)
 		)
-		(property "Mouser Part Number" ""
-			(at 198.12 58.42 0)
+		(property "PN" "CC0603KRX7R9BB104"
+			(at 198.12 58.42 90)
 			(effects
 				(font
@@
 			)
 		)
-		(property "PN" "CC0603KRX7R9BB104"
+		(property "LCSC" "C14663"
 			(at 198.12 58.42 90)
 			(effects
@@
 		(in_bom yes)
 		(on_board yes)
-		(dnp no)
+		(dnp yes)
 		(property "Reference" "Y2"
 			(at 160.02 81.3958 90)
@@
 			)
 		)
-		(property "Mouser Part Number" ""
-			(at 162.56 76.2 0)
+		(property "LCSC" ""
+			(at 162.56 76.2 90)
 			(effects
 				(font
@@
 			)
 		)
-		(property "Mouser Part Number" ""
-			(at 139.7 58.42 0)
+		(property "PN" "CC0603KRX7R9BB104"
+			(at 139.7 58.42 90)
 			(effects
 				(font
@@
 			)
 		)
-		(property "PN" "CC0603KRX7R9BB104"
+		(property "LCSC" "C14663"
 			(at 139.7 58.42 90)
 			(effects
@@
 			)
 		)
-		(property "Mouser Part Number" ""
-			(at 147.32 72.39 0)
+		(property "PN" "CC0603KRX7R9BB104"
+			(at 147.32 72.39 90)
 			(effects
 				(font
@@
 			)
 		)
-		(property "PN" "CC0603KRX7R9BB104"
+		(property "LCSC" "C14663"
 			(at 147.32 72.39 90)
 			(effects
@@
 			)
 		)
+		(property "LCSC" "C22413806"
+			(at 207.01 92.71 0)
+			(effects
+				(font
+					(size 1.27 1.27)
+				)
+				(hide yes)
+			)
+		)
 		(pin "9"
 		)
@@
 		(unit 1)
 		(exclude_from_sim no)
-		(in_bom yes)
+		(in_bom no)
 		(on_board yes)
-		(dnp no)
+		(dnp yes)
 		(fields_autoplaced yes)
 		(property "Reference" "R1"
@@
 			)
 		)
+		(property "LCSC" "C4190"
+			(at 163.83 93.98 0)
+			(effects
+				(font
+					(size 1.27 1.27)
+				)
+				(hide yes)
+			)
+		)
+		(property "PN" "CRGP0603F2K2"
+			(at 163.83 93.98 0)
+			(effects
+				(font
+					(size 1.27 1.27)
+				)
+				(hide yes)
+			)
+		)
 		(pin "2"
 		)
@@
 			)
 		)
-		(property "Mouser Part Number" ""
-			(at 220.98 53.34 0)
+		(property "PN" "CC0603KRX7R9BB104"
+			(at 220.98 53.34 90)
 			(effects
 				(font
@@
 			)
 		)
-		(property "PN" "CC0603KRX7R9BB104"
+		(property "LCSC" "C14663"
 			(at 220.98 53.34 90)
 			(effects
@@
 			)
 		)
+		(property "LCSC" ""
+			(at 176.53 90.17 0)
+			(effects
+				(font
+					(size 1.27 1.27)
+				)
+				(hide yes)
+			)
+		)
 		(pin "2"
 		)
@@
 			)
 		)
-		(property "Mouser Part Number" ""
+		(property "LCSC" ""
 			(at 186.69 90.17 0)
 			(effects
@@
 			)
 		)
+		(property "LCSC" ""
+			(at 140.97 143.51 0)
+			(effects
+				(font
+					(size 1.27 1.27)
+				)
+				(hide yes)
+			)
+		)
 		(instances
 			(project ""
@@
 			)
 		)
+		(property "LCSC" ""
+			(at 242.57 143.51 0)
+			(effects
+				(font
+					(size 1.27 1.27)
+				)
+				(hide yes)
+			)
+		)
 		(pin "3"
 		)
@@
 			)
 		)
-		(property "Mouser Part Number" ""
-			(at 201.93 46.99 0)
+		(property "PN" "BMC-Q1JY0500H"
+			(at 201.93 46.99 90)
 			(effects
 				(font
@@
 			)
 		)
-		(property "PN" "BMC-Q1JY0500H"
+		(property "LCSC" "C1002"
 			(at 201.93 46.99 90)
 			(effects
@@
 			)
 		)
-		(property "Mouser Part Number" ""
-			(at 133.35 54.61 0)
+		(property "PN" "BMC-Q1JY0500H"
+			(at 133.35 54.61 90)
 			(effects
 				(font
@@
 			)
 		)
-		(property "PN" "BMC-Q1JY0500H"
+		(property "LCSC" "C1002"
 			(at 133.35 54.61 90)
 			(effects
@@
 			)
 		)
-		(property "Mouser Part Number" ""
-			(at 217.17 66.04 0)
+		(property "PN" "CC0603KRX7R9BB104"
+			(at 217.17 66.04 90)
 			(effects
 				(font
@@
 			)
 		)
-		(property "PN" "CC0603KRX7R9BB104"
+		(property "LCSC" "C14663"
 			(at 217.17 66.04 90)
 			(effects
@@
 			)
 		)
+		(property "LCSC" ""
+			(at 140.97 149.86 0)
+			(effects
+				(font
+					(size 1.27 1.27)
+				)
+				(hide yes)
+			)
+		)
 		(instances
 			(project "DualClockLO"
@@
 		(unit 1)
 		(exclude_from_sim no)
-		(in_bom yes)
+		(in_bom no)
 		(on_board yes)
-		(dnp no)
+		(dnp yes)
 		(fields_autoplaced yes)
 		(property "Reference" "R2"
@@
 			(at 156.21 93.98 0)
 			(effects
+				(font
+					(size 1.27 1.27)
+				)
+				(hide yes)
+			)
+		)
+		(property "LCSC" "C4190"
+			(at 156.21 93.98 0)
+			(effects
+				(font
+					(size 1.27 1.27)
+				)
+				(hide yes)
+			)
+		)
+		(property "PN" "CRGP0603F2K2"
+			(at 156.21 93.98 0)
+			(effects
