File: T41_V012_Files/T41_V012_PCBs/T41_V012_PCBs_KiCad/T41-RF-board-Attenuator-daughterboard/T41-RF-board-Attenuator-daughterboard.kicad_sch (KiCad schematic)
At the start: 6 parts, among them J1 Conn 1, J2 Conn 2, U1 PE4312

Commit message: Updated titles for schematics and printed to PDF
Other:
- company: (none) -> Oliver King, KI3P
- title: (none) -> T41 RF Board Attenuator Daughterboard
Changed lines of the file:
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@@
 	(generator_version "9.0")
 	(paper "A4")
+	(title_block
+		(title "T41 RF Board Attenuator Daughterboard")
+		(date "2025-12-27")
+		(rev "1")
+		(company "Oliver King, KI3P")
+	)
 	(junction
 		(at 138.43 68.58)

Commit message: New layouts for RF board, clock board, and attenuator board are done
Parts:
- added C2: 10uF 50V, Capacitor_SMD:C_0603_1608Metric, symbol Device:C
- added L1: FB, Resistor_SMD:R_0603_1608Metric, symbol Device:L
- C1: footprint Capacitor_SMD:C_1206_3216Metric -> Capacitor_SMD:C_0603_1608Metric
- R1, R2: footprint Resistor_SMD:R_1206_3216Metric -> Resistor_SMD:R_0603_1608Metric
Connections:
- net +3V3: now also L1.1; no longer C1.2, U1.5 (LE), U1.6 (VDD), U1.9 (VDD)
- net GND: now also C2.1
- new net: C1.2, C2.2, L1.2, U1.5 (LE), U1.6 (VDD), U1.9 (VDD)

Commit message: RF board updated to reverse the direction of the transmit chain, making routing easier and less prone to noise.
Parts:
- C1: LCSC (none) -> C14663; PN (none) -> CC0603KRX7R9BB104
- C2: LCSC (none) -> C96446; PN (none) -> GXT188R61C106KE13D
- L1: LCSC (none) -> C1002; PN (none) -> BMC-Q1JY0500H
- R1, R2: LCSC (none) -> C25804; PN (none) -> CMP0603-FX-1002ELF
- U1: LCSC (none) -> C500480; PN (none) -> PE4312C-Z
Changed lines of the file:
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@@
 			)
 		)
-		(property "Mouser Part Number" ""
+		(property "LCSC" "C500480"
+			(at 135.89 96.52 0)
+			(effects
+				(font
+					(size 1.27 1.27)
+				)
+				(hide yes)
+			)
+		)
+		(property "PN" "PE4312C-Z"
 			(at 135.89 96.52 0)
 			(effects
@@
 			)
 		)
-		(property "Mouser Part Number" ""
-			(at 147.32 73.66 0)
+		(property "LCSC" "C14663"
+			(at 147.32 73.66 90)
+			(effects
+				(font
+					(size 1.27 1.27)
+				)
+				(hide yes)
+			)
+		)
+		(property "PN" "CC0603KRX7R9BB104"
+			(at 147.32 73.66 90)
 			(effects
 				(font
@@
 			)
 		)
-		(property "Mouser Part Number" ""
+		(property "LCSC" "C1002"
+			(at 138.43 60.96 0)
+			(effects
+				(font
+					(size 1.27 1.27)
+				)
+				(hide yes)
+			)
+		)
+		(property "PN" "BMC-Q1JY0500H"
 			(at 138.43 60.96 0)
 			(effects
@@
 			)
 		)
-		(property "Mouser Part Number" ""
+		(property "LCSC" "C25804"
+			(at 120.65 109.22 0)
+			(effects
+				(font
+					(size 1.27 1.27)
+				)
+				(hide yes)
+			)
+		)
+		(property "PN" "CMP0603-FX-1002ELF"
 			(at 120.65 109.22 0)
 			(effects
@@
 			)
 		)
-		(property "Mouser Part Number" ""
+		(property "LCSC" "C25804"
+			(at 111.76 81.28 0)
+			(effects
+				(font
+					(size 1.27 1.27)
+				)
+				(hide yes)
+			)
+		)
+		(property "PN" "CMP0603-FX-1002ELF"
 			(at 111.76 81.28 0)
 			(effects
@@
 			)
 		)
-		(property "Mouser Part Number" ""
-			(at 157.48 73.66 0)
+		(property "LCSC" "C96446"
+			(at 157.48 73.66 90)
+			(effects
+				(font
+					(size 1.27 1.27)
+				)
+				(hide yes)
+			)
+		)
+		(property "PN" "GXT188R61C106KE13D"
+			(at 157.48 73.66 90)
 			(effects
 				(font
@@
 			)
 		)
+		(property "LCSC" ""
+			(at 173.99 93.98 0)
+			(effects
+				(font
+					(size 1.27 1.27)
+				)
+				(hide yes)
+			)
+		)
+		(property "PN" ""
+			(at 173.99 93.98 0)
+			(effects
+				(font
+					(size 1.27 1.27)
+				)
+				(hide yes)
+			)
+		)
 		(pin "3"
 		)
@@
 			(at 83.82 96.52 0)
 			(effects
+				(font
+					(size 1.27 1.27)
+				)
+				(hide yes)
+			)
+		)
+		(property "LCSC" ""
+			(at 83.82 96.52 0)
+			(effects
+				(font
+					(size 1.27 1.27)
+				)
+				(hide yes)
+			)
+		)
+		(property "PN" ""
+			(at 83.82 96.52 0)
+			(effects

Commit message: Files Update
Files Update
Parts:
- J1, J2: now not fitted
Changed lines of the file:
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@@
 		(in_bom yes)
 		(on_board yes)
-		(dnp no)
+		(dnp yes)
 		(fields_autoplaced yes)
 		(property "Reference" "J2"
@@
 		(in_bom yes)
 		(on_board yes)
-		(dnp no)
+		(dnp yes)
 		(fields_autoplaced yes)
 		(property "Reference" "J1"
