File: T41_V012_Files/T41_V012_PCBs/T41_V012_PCBs_KiCad/T41-RF-board-si5340Clock-daughterboard/T41-RF-board-si5340Clock-daughterboard.kicad_pcb (KiCad board)
At the start: 4 copper layers, 35.1 x 25.3 mm, 5 parts, among them J2 pin header, J3 pin header, J4 pin header

Commit message: File updates
file updates
Other:
- board text added: "*** TO BE REVISED ***"
Changed lines of the file:
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@@
 		(layer "Edge.Cuts")
+	)
+	(gr_text "*** TO BE REVISED ***"
+		(at 117.73 93.68 0)
+		(layer "F.Cu")
+		(effects
+			(font
+				(size 1.5 1.5)
+				(thickness 0.3)
+				(bold yes)
+			)
+			(justify left bottom)
+		)
+	)
+	(gr_text "*** TO BE REVISED ***"
+		(at 143.9 90.98 0)
+		(layer "B.Cu")
+		(effects
+			(font
+				(size 1.5 1.5)
+				(thickness 0.3)
+				(bold yes)
+			)
+			(justify left bottom mirror)
+		)
 	)
 	(gr_text "1"
