File: T41_V012_Files/T41_V012_PCBs/T41_V012_PCBs_KiCad/T41-RF-board-V012.8/T41-RF-board-V012.8.kicad_sch (KiCad schematic)
At the start: 210 parts, among them J1 IQ_Out, J2 RF_IN, J3 RFControl, J4 12-13.8V, J5 IQ_In, J6 RF_OUT, Q1 BS170, U1 74CBTLV3253DR, U10 SN74LVC1G04DCK, U106 AD8599, U107 OPA2209, U11 T41_Attenuator_Daughter, U12 T41_DualClock_Daughter, U13 MAR-3SM+, U14 LM7805CT, U15 LM1117T-3.3, U16 LM358B, U17 LM317L, U2 PSA-8A+, U21 MCP23017_SO, U3 T41_Attenuator_Daughter, U4 74CBTLV3253DR, U5 SN74LVC1G04DCK, U6 MC33078, U7 MASWSS0179, U8 MC33078, U9 MASWSS0179

Commit message: Update Files
Update Files
Parts:
- U11, U3: value T41_Attenuator_Daughter -> Attenuator Daughter Board (See Legend)
- U12: value T41_DualClock_Daughter -> Oscillator Daughter Board (See Legend)
Other:
- note added: "Attenuator Daughter Board Options ---------------------------- 1. Single PE4312 Attenuator Daughterboard 2. Dual PE4312 Attenuator Daughterboard"
- note added: "Oscillator Daughter Board Options ---------------------------- 1. si5351A-B-GM Oscillator Daughterboard 2. si5340 Oscillator Daughterboard"
Changed lines of the file:
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@@
 		(comment 3 "Change log: Added daughterboards")
 	)
+	(text "Attenuator Daughter Board Options\n----------------------------\n1.  Single PE4312 Attenuator Daughterboard\n2.  Dual PE4312 Attenuator Daughterboard"
+		(exclude_from_sim no)
+		(at 235.966 131.826 0)
+		(effects
+			(font
+				(size 1.27 1.27)
+				(color 255 0 0 1)
+			)
+			(justify left)
+		)
+	)
 	(text "RF output"
 		(exclude_from_sim no)
@@
 		)
 	)
+	(text "Oscillator Daughter Board Options\n----------------------------\n1.  si5351A-B-GM Oscillator Daughterboard\n2.  si5340 Oscillator Daughterboard"
+		(exclude_from_sim no)
+		(at 301.498 131.826 0)
+		(effects
+			(font
+				(size 1.27 1.27)
+				(color 255 0 0 1)
+			)
+			(justify left)
+		)
+	)
 	(text "CW Mode"
 		(exclude_from_sim no)
@@
 		)
 	)
+	(text_box "Oscillator"
+		(exclude_from_sim no)
+		(at 179.07 138.43 0)
+		(size 41.402 30.734)
+		(margins 0.9525 0.9525 0.9525 0.9525)
+		(stroke
+			(width 0.381)
+			(type dot)
+			(color 255 0 0 1)
+		)
+		(fill
+			(type none)
+		)
+		(effects
+			(font
+				(size 1.27 1.27)
+				(thickness 0.254)
+				(bold yes)
+			)
+			(justify right top)
+		)
+	)
 	(text_box "Auto calibrate switch"
 		(exclude_from_sim no)
@@
 		)
 	)
-	(text_box "Transmit RF gain control"
+	(text_box "Transmit RF Gain Control"
 		(exclude_from_sim no)
-		(at 80.01 201.93 0)
-		(size 43.18 34.29)
+		(at 82.042 200.914 0)
+		(size 37.846 35.56)
 		(margins 0.9525 0.9525 0.9525 0.9525)
 		(stroke
-			(width 0)
-			(type default)
+			(width 0.381)
+			(type dot)
+			(color 255 0 0 1)
 		)
 		(fill
@@
 	(text_box "Receive RF gain control"
 		(exclude_from_sim no)
-		(at 77.47 59.69 0)
-		(size 50.8 54.61)
+		(at 76.962 71.374 0)
+		(size 43.18 37.592)
 		(margins 0.9525 0.9525 0.9525 0.9525)
 		(stroke
-			(width 0)
-			(type default)
+			(width 0.381)
+			(type dot)
+			(color 255 0 0 1)
 		)
 		(fill
@@
 		(on_board yes)
 		(dnp no)
-		(fields_autoplaced yes)
 		(property "Reference" "U3"
-			(at 102.235 205.74 0)
+			(at 102.616 208.788 0)
 			(effects
 				(font
@@
 			)
 		)
-		(property "Value" "T41_Attenuator_Daughter"
-			(at 102.235 208.28 0)
+		(property "Value" "Attenuator Daughter Board (See Legend)"
+			(at 101.346 198.12 0)
 			(effects
 				(font
 					(size 1.27 1.27)
+					(color 255 0 0 1)
 				)
 			)
@@
 			)
 		)
-		(property "Value" "T41_DualClock_Daughter"
-			(at 223.774 162.052 90)
+		(property "Value" "Oscillator Daughter Board (See Legend)"
+			(at 218.694 136.652 90)
 			(effects
 				(font
 					(size 1.27 1.27)
+					(color 255 0 0 1)
 				)
 				(justify left)
@@
 		(on_board yes)
 		(dnp no)
-		(fields_autoplaced yes)
 		(property "Reference" "U11"
 			(at 100.965 78.74 0)
@@
 			)
 		)
-		(property "Value" "T41_Attenuator_Daughter"
-			(at 100.965 81.28 0)
+		(property "Value" "Attenuator Daughter Board (See Legend)"
+			(at 99.314 68.072 0)
 			(effects
 				(font
 					(size 1.27 1.27)
+					(color 255 0 0 1)
 				)
 			)
