File: T41_V012_Files/T41_V012_PCBs/T41_V012_PCBs_KiCad/T41-RF-board-V012.8/T41-RF-board-V012.8.kicad_pcb (KiCad board)
At the start: 4 copper layers, 100 x 100 mm, 209 parts, among them J1 IQ_Out, J2 RF_IN, J3 RFControl, J4 12-13.8V, J5 IQ_In, J6 RF_OUT, Q1 BS170, U1 74CBTLV3253DR, U10 SN74LVC1G04DCK, U106 AD8599, U107 OPA2209, U11 T41_Attenuator_Daughter, U12 T41_DualClock_Daughter, U13 MAR-3SM+, U14 LM7805CT, U15 LM1117T-3.3, U16 LM358B, U17 LM317L, U2 PSA-8A+, U21 MCP23017_SO, U3 T41_Attenuator_Daughter, U4 74CBTLV3253DR, U5 SN74LVC1G04DCK, U6 MC33078, U7 MASWSS0179, U8 MC33078, U9 MASWSS0179

Commit message: Upates
Updates
Connections:
- R35 pad 2: /TX0 -> /TX90
- R37 pad 2: /TX90 -> /TX0
- R40 pad 1: /RX0 -> /RX90
- R42 pad 1: /RX90 -> /RX0
- U12 pad 1: /TX0 -> /TX90
- U12 pad 11: /RX0 -> /RX90
- U12 pad 12: /RX90 -> /RX0
- U12 pad 2: /TX90 -> /TX0
Changed lines of the file:
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@@
 			(layers "F.Cu" "F.Mask" "F.Paste")
 			(roundrect_rratio 0.222222)
-			(net "/TX90")
+			(net "/TX0")
 			(pintype "passive")
 		)
@@
 			(layers "F.Cu" "F.Mask" "F.Paste")
 			(roundrect_rratio 0.222222)
-			(net "/RX0")
+			(net "/RX90")
 			(pintype "passive")
 		)
@@
 			(layer "F.CrtYd")
 		)
-		(fp_text user "RX90"
-			(at 0.508 -5.08 90)
+		(fp_text user "TX90"
+			(at 0.508 9.144 90)
 			(unlocked yes)
 			(layer "F.SilkS")
@@
 			)
 		)
-		(fp_text user "TX0"
-			(at 0.508 9.144 90)
+		(fp_text user "RX0"
+			(at 0.578 -5.952 90)
 			(unlocked yes)
 			(layer "F.SilkS")
@@
 			)
 		)
-		(fp_text user "RX0"
-			(at 3.048 -6.096 90)
+		(fp_text user "TX0"
+			(at 3.048 9.144 90)
 			(unlocked yes)
 			(layer "F.SilkS")
@@
 			)
 		)
-		(fp_text user "TX90"
-			(at 3.048 9.144 90)
+		(fp_text user "RX90"
+			(at 3.178 -5.002 90)
 			(unlocked yes)
 			(layer "F.SilkS")
@@
 			(layers "*.Cu" "*.Mask")
 			(remove_unused_layers no)
-			(net "/TX0")
+			(net "/TX90")
 			(pinfunction "CLK4")
 			(pintype "input")
@@
 			(layers "*.Cu" "*.Mask")
 			(remove_unused_layers no)
-			(net "/TX90")
+			(net "/TX0")
 			(pinfunction "CLK5")
 			(pintype "input")
@@
 			(layers "*.Cu" "*.Mask")
 			(remove_unused_layers no)
-			(net "/RX0")
+			(net "/RX90")
 			(pinfunction "CLK1")
 			(pintype "power_in")
@@
 			(layers "*.Cu" "*.Mask")
 			(remove_unused_layers no)
-			(net "/RX90")
+			(net "/RX0")
 			(pinfunction "CLK0")
 			(pintype "input")
@@
 			(layers "F.Cu" "F.Mask" "F.Paste")
 			(roundrect_rratio 0.222222)
-			(net "/RX90")
+			(net "/RX0")
 			(pintype "passive")
 		)
@@
 			(layers "F.Cu" "F.Mask" "F.Paste")
 			(roundrect_rratio 0.222222)
-			(net "/TX0")
+			(net "/TX90")
 			(pintype "passive")
 		)
@@
 		)
 	)
-	(gr_text "RX90"
+	(gr_text "RX0"
 		(at 81.9658 76.327 0)
 		(layer "F.SilkS")
@@
 		)
 	)
-	(gr_text "TX0"
+	(gr_text "TX90"
 		(at 82.804 104.8258 0)
 		(layer "F.SilkS")
@@
 		)
 	)
-	(gr_text "TX90"
+	(gr_text "TX0"
 		(at 90.7034 105.1052 0)
 		(layer "F.SilkS")
@@
 		)
 	)
-	(gr_text "RX0"
+	(gr_text "RX90"
 		(at 91.44 76.327 0)
 		(layer "F.SilkS")
@@
 	)
 	(segment
-		(start 89.662 104.8365)
-		(end 89.408 105.0905)
+		(start 87.122 104.7095)
+		(end 86.868 104.9635)
 		(width 0.2)
 		(layer "F.Cu")
@@
 	)
 	(segment
-		(start 89.662 102.362)
-		(end 89.662 104.8365)
+		(start 86.868 104.9635)
+		(end 86.868 105.0905)
+		(width 0.2)
+		(layer "F.Cu")
+		(net "/TX90")
+	)
+	(segment
+		(start 87.122 102.362)
+		(end 87.122 104.7095)
 		(width 0.2)
 		(layer "F.Cu")
@@
 		(width 0.25)
 		(layer "F.Cu")
-		(net "/RX0")
+		(net "/RX90")
 	)
 	(segment
@@
 		(width 0.25)
 		(layer "F.Cu")
-		(net "/RX0")
+		(net "/RX90")
 	)
 	(segment
@@
 	)
 	(segment
-		(start 87.122 104.7095)
-		(end 86.868 104.9635)
-		(width 0.2)
-		(layer "F.Cu")
-		(net "/TX0")
-	)
-	(segment
-		(start 86.868 104.9635)
-		(end 86.868 105.0905)
+		(start 89.662 104.8365)
+		(end 89.408 105.0905)
 		(width 0.2)
 		(layer "F.Cu")
@@
 	)
 	(segment
-		(start 87.122 102.362)
-		(end 87.122 104.7095)
+		(start 89.662 102.362)
+		(end 89.662 104.8365)
 		(width 0.2)
 		(layer "F.Cu")
@@
 		(width 0.25)
 		(layer "F.Cu")
-		(net "/RX90")
+		(net "/RX0")
 	)
 	(segment
