File: T41_V012_Files/T41_V012_PCBs/T41_V012_PCBs_KiCad/T41-si5351A-B-GM-Oscillator-daughterboard/T41-si5351A-B-GM-Oscillator-daughterboard.kicad_sch (KiCad schematic)
At the start: 27 parts, among them J1 qwiic, J2 pin header, J3 pin header, J4 pin header, J5 OEBSSEN, U1 Si5351A-B-GM, U2 ECS-TX053-S3, U3 ECS-TXO-2520-250-TR, U4 ECS-TXO-3225-100-TR

Commit message: Update Files
Update Files
Changed lines of the file:
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@@
 		)
 	)
-	(text_box "Option 1: 4-SMD 3.2 x 2.5"
+	(text_box "Option 3: 4-SMD 3.2 x 2.5"
 		(exclude_from_sim no)
 		(at 95.25 135.128 0)

Commit message: update files
Update files
Parts:
- U4: now fitted; now in the parts list
