File: T41_V012_Files/T41_V012_PCBs/T41_V012_PCBs_KiCad/T41-si5351A-B-GM-Oscillator-daughterboard/T41-si5351A-B-GM-Oscillator-daughterboard.kicad_sch (KiCad schematic)
At the start: 27 parts, among them J1 qwiic, J2 pin header, J3 pin header, J4 pin header, J5 OEBSSEN, U1 Si5351A-B-GM, U2 ECS-TX053-S3, U3 ECS-TXO-2520-250-TR, U4 ECS-TXO-3225-100-TR

Commit message: BOM Updates
BOM Updates
Parts:
- added J6: Conn_01x02_Socket, symbol Connector:Conn_01x02_Socket
Connections:
- net GND: now also J6.2 (Pin_2)
- net at C2.2, U2.6 (OUT), U3.3 (OUT)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: now also J6.1 (Pin_1)
Other:
- note added: "TXCO SIGNAL FOR DIVERSITY"
Changed lines of the file:
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@@
 		(company "WJ Schmidt - K9HZ")
+	)
+	(text "TXCO SIGNAL FOR DIVERSITY"
+		(exclude_from_sim no)
+		(at 157.48 58.166 0)
+		(effects
+			(font
+				(size 1.27 1.27)
+			)
+		)
 	)
 	(text_box "Option 1: 10-SMD 5.0 x 3.2"
@@
 	)
 	(junction
+		(at 156.21 74.93)
+		(diameter 0)
+		(color 0 0 0 0)
+	)
+	(junction
 		(at 237.49 123.19)
 		(diameter 0)
@@
 	(wire
 		(pts
+			(xy 158.75 66.04) (xy 158.75 68.58)
+		)
+		(stroke
+			(width 0)
+			(type default)
+		)
+	)
+	(wire
+		(pts
 			(xy 173.99 110.49) (xy 191.77 110.49)
 		)
@@
 	(wire
 		(pts
-			(xy 135.89 74.93) (xy 173.99 74.93)
+			(xy 135.89 74.93) (xy 156.21 74.93)
 		)
 		(stroke
@@
 	(wire
 		(pts
+			(xy 156.21 74.93) (xy 173.99 74.93)
+		)
+		(stroke
+			(width 0)
+			(type default)
+		)
+	)
+	(wire
+		(pts
 			(xy 156.21 100.33) (xy 191.77 100.33)
 		)
@@
 		(pts
 			(xy 222.25 85.09) (xy 242.57 85.09)
+		)
+		(stroke
+			(width 0)
+			(type default)
+		)
+	)
+	(wire
+		(pts
+			(xy 156.21 66.04) (xy 156.21 74.93)
 		)
 		(stroke
@@
 	)
 	(symbol
+		(lib_name "GND_1")
+		(lib_id "power:GND")
+		(at 158.75 68.58 0)
+		(unit 1)
+		(body_style 1)
+		(exclude_from_sim no)
+		(in_bom yes)
+		(on_board yes)
+		(in_pos_files yes)
+		(dnp no)
+		(fields_autoplaced yes)
+		(property "Reference" "#PWR022"
+			(at 158.75 74.93 0)
+			(hide yes)
+			(show_name no)
+			(do_not_autoplace no)
+			(effects
+				(font
+					(size 1.27 1.27)
+				)
+			)
+		)
+		(property "Value" "GND"
+			(at 158.75 73.66 0)
+			(show_name no)
+			(do_not_autoplace no)
+			(effects
+				(font
+					(size 1.27 1.27)
+				)
+			)
+		)
+		(property "Footprint" ""
+			(at 158.75 68.58 0)
+			(hide yes)
+			(show_name no)
+			(do_not_autoplace no)
+			(effects
+				(font
+					(size 1.27 1.27)
+				)
+			)
+		)
+		(property "Datasheet" ""
+			(at 158.75 68.58 0)
+			(hide yes)
+			(show_name no)
+			(do_not_autoplace no)
+			(effects
+				(font
+					(size 1.27 1.27)
+				)
+			)
+		)
+		(property "Description" "Power symbol creates a global label with name \"GND\" , ground"
+			(at 158.75 68.58 0)
+			(hide yes)
+			(show_name no)
+			(do_not_autoplace no)
+			(effects
+				(font
+					(size 1.27 1.27)
+				)
+			)
+		)
+		(pin "1"
+		)
+		(instances
+			(project "T41-si5351A-B-GM-Oscillator-daughterboard"
+				(path "/19e7ad66-8f4f-49d3-ad58-95c831b9d6b3"
+					(reference "#PWR022")
+					(unit 1)
+				)
+			)
+		)
+	)
+	(symbol
 		(lib_id "SparkFun-Qwiic:qwiic_Logo")
 		(at 262.89 127 0)
@@
 					(unit 1)
 				)
+			)
+		)
+	)
+	(symbol
+		(lib_id "Connector:Conn_01x02_Socket")
+		(at 156.21 60.96 90)
+		(unit 1)
+		(body_style 1)
+		(exclude_from_sim no)
+		(in_bom yes)
+		(on_board yes)
+		(in_pos_files yes)
+		(dnp no)
+		(fields_autoplaced yes)
+		(property "Reference" "J6"
+			(at 160.02 60.3249 90)
+			(show_name no)
+			(do_not_autoplace no)
+			(effects
+				(font
+					(size 1.27 1.27)
+				)
+				(justify right)
+			)
+		)
+		(property "Value" "Conn_01x02_Socket"
+			(at 160.02 62.8649 90)
+			(hide yes)
+			(show_name no)
+			(do_not_autoplace no)
+			(effects
+				(font
+					(size 1.27 1.27)
+				)
+				(justify right)
+			)
+		)
+		(property "Footprint" ""
+			(at 156.21 60.96 0)
+			(hide yes)
+			(show_name no)
+			(do_not_autoplace no)
+			(effects
+				(font
+					(size 1.27 1.27)
+				)
+			)
+		)
+		(property "Datasheet" ""
+			(at 156.21 60.96 0)
+			(hide yes)
+			(show_name no)
+			(do_not_autoplace no)
+			(effects
+				(font
+					(size 1.27 1.27)
+				)
+			)
+		)
+		(property "Description" "Generic connector, single row, 01x02, script generated"
+			(at 156.21 60.96 0)
+			(hide yes)
+			(show_name no)
+			(do_not_autoplace no)
+			(effects
+				(font
+					(size 1.27 1.27)
+				)
+			)
+		)
+		(pin "1"
+		)
+		(pin "2"
+		)
+		(instances
+			(project "T41-si5351A-B-GM-Oscillator-daughterboard"
+				(path "/19e7ad66-8f4f-49d3-ad58-95c831b9d6b3"
+					(reference "J6")
+					(unit 1)
+				)
