File: T41_V012_Files/T41_V012_PCBs/T41_V012_PCBs_KiCad/T41-si5351A-B-GM-Oscillator-daughterboard/T41-si5351A-B-GM-Oscillator-daughterboard.kicad_pcb (KiCad board)
At the start: 4 copper layers, 35.1 x 25.3 mm, 27 parts, among them J1 qwiic, J2 pin header, J3 pin header, J4 pin header, J5 OEBSSEN, U1 Si5351A-B-GM, U2 ECS-TX053-S3, U3 ECS-TXO-2520-250-TR, U4 ECSTXO3225120TR

Commit message: OSC Files Update
OSC Files Update
Parts:
- added J6: PinHeader_1x02_P2.54mm_Vertical, Connector_PinHeader_2.54mm:PinHeader_1x02_P2.54mm_Vertical, F.Cu at (129.1, 96.4)
- moved C2 1.01 mm to (127.1, 92.7)
Routing:
- net Net-(U2-OUT): track 18.9 -> 20.0 mm
- net Net-(U1-XA): track 7.79 -> 6.98 mm
- net GND: vias 67 -> 65
Other:
- board text added: "OSC"
- board text added: "Si5351A-B-GM OSC BOARD K9HZ 090626"
- board text removed: "Si5351A-B-GM OSC BOARD K9HZ 042426"
