File: T41_V012_Files/T41_V012_PCBs/T41_V012_PCBs_KiCad/T41-Single-PE4312-Attenuator-daughterboard/T41-Single-PE4312-Attenuator-daughterboard.kicad_sch (KiCad schematic)
At the start: 8 parts, among them J1 Conn 1, J2 Conn 2, U1 PE4312

Commit message: Update
Update
Other:
- company: Oliver King, KI3P -> Oliver King, KI3P/ Revised by WJ Schmidt, K9HZ

Commit message: Update
Update
Parts:
- renumbered C2 to C1, C1 to C2
Changed lines of the file:
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@@
 		(in_pos_files yes)
 		(dnp no)
-		(property "Reference" "C1"
+		(property "Reference" "C2"
 			(at 153.6233 73.66 90)
 			(show_name no)
@@
 			(project "T41-Single-PE4312-Attenuator-daughterboard"
 				(path "/4fb44e34-3372-47df-9694-9168f4fad0b1"
-					(reference "C1")
+					(reference "C2")
 					(unit 1)
 				)
@@
 		(in_pos_files yes)
 		(dnp no)
-		(property "Reference" "C2"
+		(property "Reference" "C1"
 			(at 163.7833 73.66 90)
 			(show_name no)
@@
 			(project "T41-Single-PE4312-Attenuator-daughterboard"
 				(path "/4fb44e34-3372-47df-9694-9168f4fad0b1"
-					(reference "C2")
-					(unit 1)
-				)
+					(reference "C1")
+					(unit 1)
+				)
